File: Encoder_TestBench/Hardware/EncoderTBPCB.brd (EAGLE design)
At the start: 51.7 x 81.3 mm, 18 parts, among them IC1 7805DT, U1 ATMEGA328P-PU

Commit message: Board Revised
Parts:
- removed SV1, SV2: (no value), con-lstb:MA05-1
- added X1, X2: C-GRID-05-15-91, con-molex:15-91-05
- moved R2 8.03 mm to (90.2, 33.0)
- moved JP1 3.81 mm to (55.9, 53.3)
Connections:
- net N$13: now also X1.1, X2.1; no longer SV1.1, SV2.1
- net N$14: now also X1.3, X2.3; no longer SV1.3, SV2.3
- net VDD: now also X1.2, X2.2; no longer SV1.2, SV2.2
- net VSS: now also X1.5, X2.5; no longer SV1.5, SV2.5
Routing:
- net VDD: track 123.0 -> 164.4 mm
- net N$13: track 56.7 -> 44.2 mm
- net N$14: track 49.3 -> 57.6 mm
- net N$11: track 46.7 -> 41.4 mm, vias 1 -> 0
- net N$19: track 47.0 -> 50.8 mm
- net N$9: track 50.4 -> 47.7 mm
- net N$18: track 18.9 -> 20.4 mm
- net VSS: track 271.4 -> 270.2 mm
- net N$1: track 46.0 -> 45.5 mm
- net N$10: track 39.8 -> 39.7 mm, vias 1 -> 0

Commit message: Port Updated
Parts:
- removed U$1: LCD-HD447804-HOLES16X2-4-HOLES, HD44780LCD:LCD-16X2-4HOLES
- removed X2: C-GRID-05-15-91, con-molex:15-91-05
- added JP2: (no value), pinhead:1X16
- moved JP1 21.6 mm to (57.1, 31.8)
- moved X1 21.6 mm to (53.3, 14.0)
- moved G1 20.3 mm to (55.9, 47.0)
Connections:
- net N$1: now also JP2.6; no longer U$1.6
- net N$13: no longer X2.1
- net N$14: no longer X2.3
- net N$2: now also JP2.15; no longer U$1.15
- net N$4: now also JP2.14; no longer U$1.14
- net N$5: now also JP2.13; no longer U$1.13
- net N$6: now also JP2.12; no longer U$1.12
- net N$7: now also JP2.11; no longer U$1.11
- net N$9: now also JP2.4; no longer U$1.4
- net VDD: now also JP2.2; no longer U$1.2, X2.2
- net VO: now also JP2.3; no longer U$1.3
- net VSS: now also JP2.1, JP2.16, JP2.5; no longer U$1.1, U$1.16, U$1.5, X2.5
Routing:
- net VDD: track 164.4 -> 127.2 mm
- net N$14: track 57.6 -> 26.9 mm
- net N$19: track 50.8 -> 28.3 mm
- net N$9: track 47.7 -> 67.5 mm
- net N$13: track 44.2 -> 28.9 mm
- net N$15: track 11.2 -> 22.0 mm
- net N$1: track 45.5 -> 56.1 mm
- net N$18: track 20.4 -> 26.4 mm
- net VSS: track 270.2 -> 265.6 mm
