File: Testbench/Motor_Shield_Testbench/Board Design/MotorShieldTestbench_ro.brd (EAGLE design)
At the start: 60 x 67 mm, 49 parts, among them IC2 74LS04D, IC3 74AC74D, IC4 74AC74D, U1 ATMEGA2560AU, U10 +12v, U2 FT232RL, U3 ATTINY85-20SU, U4 ATTINY85-20SU, U6 SN74LVC2G157DCTR, U7 SN74LVC2G157DCTR, U8 SN74LVC2G157DCTR, U9 SN74LVC2G157DCTR, X4 2510-, X5 2510-, X6 MINI-USB_4P-32005-101

Commit message: minor improvements
Parts:
- moved R1 9.91 mm to (39.2, 5.75), turned to 270 degrees
- moved R15 9.18 mm to (48.5, 62.8), turned to 180 degrees
- moved R14 4.30 mm to (51.0, 60.8), turned to 180 degrees
- moved R6 2.51 mm to (32.0, 39.0)
- moved SV3 2.50 mm to (48.2, 30.2)
- moved R2 2.47 mm to (39.2, 9.50)
- moved X4 1.50 mm to (54.0, 11.5)
- moved X5 1.50 mm to (45.0, 11.5)
- moved C7 1.00 mm to (34.0, 61.5), turned to 90 degrees
Connections:
- net LE1: now also U1.4
- net LE2: now also U1.5
- net RDIR: now also U1.85; no longer U1.77
- net RE1: now also U1.45
- net RE2: now also U1.46
Routing:
- net RE2: track 9.82 -> 106.8 mm, vias 0 -> 4
- net RE1: track 8.34 -> 82.7 mm, vias 0 -> 2
- net LE1: track 6.51 -> 76.5 mm, vias 0 -> 4
- net LE2: track 6.75 -> 69.0 mm, vias 0 -> 4
- net +5V: track 102.8 -> 134.5 mm, vias 5 -> 18
- net SCL: track 40.6 -> 54.2 mm, vias 4 -> 2
- net RDIR: track 64.9 -> 77.8 mm, vias 1 -> 0
- net RSPEED: track 23.5 -> 12.1 mm
- net RSPEEDH: track 50.3 -> 60.2 mm
- net LSPEEDH: track 49.4 -> 55.2 mm
- net LSPEED: track 18.6 -> 12.9 mm
- net SDA: track 39.6 -> 44.8 mm, vias 2 -> 0
- net RESET: track 52.2 -> 54.8 mm, vias 4 -> 2
- net OA2: track 28.0 -> 25.6 mm
- net OA1: track 26.1 -> 23.7 mm
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