File: Testbench/Motor_Shield_Testbench/Board Design/MotorShieldTestbench_ro.sch (EAGLE design)
At the start: 49 parts, among them IC2 74LS04D, IC3 74AC74D, IC4 74AC74D, U1 ATMEGA2560AU, U10 +12v, U2 FT232RL, U3 ATTINY85-20SU, U4 ATTINY85-20SU, U6 SN74LVC2G157DCTR, U7 SN74LVC2G157DCTR, U8 SN74LVC2G157DCTR, U9 SN74LVC2G157DCTR, X4 2510-, X5 2510-, X6 MINI-USB_4P-32005-101

Commit message: minor improvements
Connections:
- net LE1: now also U1.(XCK0/AIN0)PE2
- net LE2: now also U1.(OC3A/AIN1)PE3
- net RDIR: now also U1.PK4(ADC12/PCINT20); no longer U1.(AD1)PA1
- net RE1: now also U1.(RXD1/INT2)PD2
- net RE2: now also U1.(TXD1/INT3)PD3
Changed lines of the file:
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@@
 <label x="198.12" y="38.1" size="1.778" layer="95"/>
+</segment>
+<segment>
+<pinref part="U1" gate="1" pin="(RXD1/INT2)PD2"/>
+<wire x1="337.82" y1="22.86" x2="347.98" y2="22.86" width="0.1524" layer="91"/>
+<label x="337.82" y="22.86" size="1.778" layer="95"/>
 </segment>
 </net>
@@
 <label x="198.12" y="7.62" size="1.778" layer="95"/>
 </segment>
+<segment>
+<pinref part="U1" gate="1" pin="(TXD1/INT3)PD3"/>
+<wire x1="337.82" y1="25.4" x2="347.98" y2="25.4" width="0.1524" layer="91"/>
+<label x="337.82" y="25.4" size="1.778" layer="95"/>
+</segment>
 </net>
 <net name="LE1" class="0">
@@
 <wire x1="198.12" y1="99.06" x2="205.74" y2="99.06" width="0.1524" layer="91"/>
 <label x="198.12" y="99.06" size="1.778" layer="95"/>
+</segment>
+<segment>
+<pinref part="U1" gate="1" pin="(XCK0/AIN0)PE2"/>
+<wire x1="337.82" y1="0" x2="347.98" y2="0" width="0.1524" layer="91"/>
+<label x="337.82" y="0" size="1.778" layer="95"/>
 </segment>
 </net>
@@
 <label x="198.12" y="68.58" size="1.778" layer="95"/>
 </segment>
+<segment>
+<pinref part="U1" gate="1" pin="(OC3A/AIN1)PE3"/>
+<wire x1="337.82" y1="2.54" x2="347.98" y2="2.54" width="0.1524" layer="91"/>
+<label x="337.82" y="2.54" size="1.778" layer="95"/>
+</segment>
 </net>
 <net name="RDIR" class="0">
@@
 </segment>
 <segment>
-<pinref part="U1" gate="1" pin="(AD1)PA1"/>
-<wire x1="337.82" y1="88.9" x2="347.98" y2="88.9" width="0.1524" layer="91"/>
-<label x="337.82" y="88.9" size="1.778" layer="95"/>
+<pinref part="U1" gate="1" pin="PK4(ADC12/PCINT20)"/>
+<wire x1="266.7" y1="10.16" x2="256.54" y2="10.16" width="0.1524" layer="91"/>
+<label x="256.54" y="10.16" size="1.778" layer="95"/>
 </segment>
 </net>
