File: Testbench/Motor_Shield_Testbench/Board Design/MotorShieldTestbench.sch (EAGLE design)
At the start: 46 parts, among them U1 ATMEGA2560AU, U2 ATMEGA8U2-AU, U3 ATTINY85-20SU, U4 ATTINY85-20SU, X1 MINI-USB-32005-301

Commit message: board design v. unknown
Parts:
- removed B1: ARDUINO_UNO_R3_SHIELD_ICSP, SparkFun-Boards:ARDUINO_UNO_R3_SHIELD_ICSP
- removed C10, C11, C12: 0.1uF, SparkFun-Capacitors:0.1UF-0603-25V-5%
- removed C15, C16: 22uF, SparkFun-Capacitors:22UF-0805-6.3V-20%
- removed FF1, FF2: 74HC74N, 74xx-eu:74HC74N
- removed NOT_GATES: 74LS04N, 74xx-eu:74LS04N
- added H1: MOUNT-PAD-ROUND2.8, holes:MOUNT-PAD-ROUND2.8
- added H2: MOUNT-PAD-SQUARE2.8, holes:MOUNT-PAD-SQUARE2.8
- added IC1: 7805T, linear:7805T
- added IC2: 74LS04D, 74xx-eu:74LS04D
- added IC3, IC4: 74AC74D, 74xx-eu:74AC74D
- added LED4: (no value), eagle-ltspice:LED_E
- added R16: 1k, SparkFun-Resistors:1KOHM-0603-1/10W-1%
- added SV1, SV2: (no value), con-lstb:MA03-2
- added X2, X3: C-GRID-05-15-91, con-molex:C-GRID-05-15-91
- added X4, X5: 2510-, con-3m:2510-
- C8: value 22pF -> 10uF; device SparkFun-Capacitors:22PF-0603-50V-5% -> SparkFun-Capacitors:10UF-0603-6.3V-20%
- C9: value 0.1uF -> 10uF; device SparkFun-Capacitors:0.1UF-0603-25V-5% -> SparkFun-Capacitors:10UF-0603-6.3V-20%
- R1, R2, R3, R4: device SparkFun-Resistors:10KOHM-HORIZ-1/4W-5% -> SparkFun-Resistors:10KOHM-0603-1/10W-1%
Connections:
- removed net N$12: B1.D1, U1.(RXD0/PCIN8)PE0
- removed net N$25: C2.2, Q3.2, U1.XTAL2
- removed net N$28: B1.D0, U1.(TXD0)PE1
- new net N$30: LED4.A, R16.2
- new net N$51: H1.MOUNT, IC1.VI
- new net N$52: LED4.C, U1.(AD0)PA0
- new net N$53: SV1.5, U1.RESET
- new net N$54: SV1.1, U1.(MISO/PCINT3)PB3
- new net N$55: SV1.3, U1.(MOSI/PCINT2)PB2
- new net N$58: R7.2, SV2.5, U2.(~RESET)_(PC1_/_DW)
- new net N$59: SV2.4, U2.PB2
- new net N$60: SV2.1, U2.PB3
- new net N$61: SV2.3, U2.PB1
- new net N$63: C1.2, Q3.1, R5.2, R6.1
- net +5V: now also IC1.VO, IC2P.VCC, IC3P.VCC, IC4P.VCC, R16.1, SV1.2, SV2.2, X2-4.S, X3-4.S, X4-1.KL, X4-2.KL, X4-5.KL, X4-7.KL, X5-1.KL, X5-2.KL, X5-5.KL, X5-7.KL; no longer B1.VIN, C10.1, C11.1, C12.1, C9.1, FF1P.VCC, FF2P.VCC, NOT_GATESP.VCC
- net GND: now also H2.MOUNT, IC1.GND, IC2P.GND, IC3P.GND, IC4P.GND, SV1.6, SV2.6, X2-1.S, X3-1.S, X4-10.KL, X4-9.KL, X5-10.KL, X5-9.KL; no longer B1.GND@0, C10.2, C11.2, C12.2, C15.2, C16.2, FF1P.GND, FF2P.GND, NOT_GATESP.GND, R6.1, R6.2
- net N$1: now also IC3A.!Q, IC3A.D; no longer FF1A.!Q, FF1A.D
- net N$10: now also IC3A.CLR, IC3A.PRE, IC3B.CLR, IC3B.PRE; no longer FF1A.CLR, FF1A.PRE, FF1B.CLR, FF1B.PRE
- net N$11: now also IC2B.I, IC4A.CLK; no longer FF2A.CLK, NOT_GATESB.I
- net N$13: now also IC2A.I, IC3A.CLK; no longer FF1A.CLK, NOT_GATESA.I
- net N$14: now also IC2B.O, IC4B.CLK; no longer FF2B.CLK, NOT_GATESB.O
- net N$15: now also X2-3.S; no longer B1.*D3
- net N$16: now also X2-5.S; no longer B1.*D5
- net N$17: now also X3-3.S; no longer B1.D2
- net N$18: now also X3-5.S; no longer B1.D4
- net N$2: now also IC3A.Q; no longer FF1A.Q
- net N$23: now also X5-8.KL; no longer B1.D7
- net N$24: now also C2.2, Q3.2, R6.2, U1.XTAL2; no longer C1.2, Q3.1, R5.2
- net N$26: now also SV1.4, U1.(SCK/PCINT1)PB1; no longer C8.1, R7.2, U1.RESET
- net N$27: now also IC2A.O, IC3B.CLK; no longer FF1B.CLK, NOT_GATESA.O
- net N$29: now also X4-8.KL; no longer B1.*D9
- net N$3: now also IC3B.Q; no longer FF1B.Q
- net N$31: now also X4-6.KL; no longer B1.*D10
- net N$4: now also IC3B.!Q, IC3B.D; no longer FF1B.!Q, FF1B.D
- net N$48: now also C8.1; no longer C15.1
- net N$49: now also X5-6.KL; no longer B1.*D6
- net N$5: now also IC4A.!Q, IC4A.D; no longer FF2A.!Q, FF2A.D
- net N$50: now also C9.1; no longer C16.1
- net N$6: now also IC4B.!Q, IC4B.D; no longer FF2B.!Q, FF2B.D
- net N$7: now also IC4A.Q; no longer FF2A.Q
- net N$8: now also IC4B.Q; no longer FF2B.Q
- net N$9: now also IC4A.CLR, IC4A.PRE, IC4B.CLR, IC4B.PRE; no longer FF2A.CLR, FF2A.PRE, FF2B.CLR, FF2B.PRE
Other:
- moved on the sheet: C8, C9, R7

Commit message: board ready for design review
Parts:
- removed C13: 22pF, SparkFun-Capacitors:22PF-0603-50V-5%
- removed C14: 1.0uF, SparkFun-Capacitors:1.0UF-0603-16V-10%
- removed IC1: 7805T, linear:7805T
- removed LED4: (no value), eagle-ltspice:LED_E
- removed Q2: (no value), special:XTAL/S
- removed R10, R11, R12, R16: 1k, SparkFun-Resistors:1KOHM-0603-1/10W-1%
- removed SV2: (no value), con-lstb:MA03-2
- removed X1: MINI-USB-32005-301, con-cypressindustries:MINI-USB-32005-301
- added C10: 0.1uF, SparkFun-Capacitors:0.1UF-0402-16V-10%
- added C11: 0.1uF, SparkFun-Capacitors:0.1UF-0603-25V-(+80/-20%)
- added S1: MOMENTARY-SWITCH-SPST-SMD-5.2-REDUNDANT, SparkFun-Switches:MOMENTARY-SWITCH-SPST-SMD-5.2-REDUNDANT
- added SV3: (no value), con-lstb:MA06-2
- added U5: (no value), SparkFun-IC-Power:V_REG_78XXSIDE
- added U6, U7, U8, U9: SN74LVC2G157DCTR, Texas Instruments_By_element14_Batch_1:SN74LVC2G157DCTR
- added X6: MINI-USB_4P-32005-101, con-cypressindustries:MINI-USB_4P-32005-101
- C3: value 22pF -> 10uF; device SparkFun-Capacitors:22PF-0603-50V-5% -> SparkFun-Capacitors:10UF-POLAR-0603-6.3V-20%(TANT)
- R7: value 10k -> 1k; device SparkFun-Resistors:10KOHM-0603-1/10W-1% -> SparkFun-Resistors:1KOHM-0603-1/10W-1%
- R8: value 22 -> 1k; device SparkFun-Resistors:22OHM-0603-1/10W-1% -> SparkFun-Resistors:1KOHM-0603-1/10W-1%
- R9: value 22 -> 10k; device SparkFun-Resistors:22OHM-0603-1/10W-1% -> SparkFun-Resistors:10KOHM-0603-1/10W-1%
- U2: value ATMEGA8U2-AU -> FT232RL; device Atmel_By_element14_Batch_1-00:ATMEGA8U2-AU -> SparkFun-IC-Comms:FT232RLSSOP
- renumbered X2 to LEFTENCODER, X3 to RIGHTENCODER
Connections:
- net N$19 renamed SCL
- net N$21 renamed SDA
- net N$23 renamed LDIR
- net N$26 renamed SCK
- net N$29 renamed RDIR
- net N$31 renamed RSPEEDH
- net N$48 renamed LSPEED
- net N$49 renamed LSPEEDH
- net N$50 renamed RSPEED
- net N$54 renamed MISO
- net N$55 renamed MOSI
- removed net N$13: IC2A.I, IC3A.CLK, U3.PB1
- removed net N$15: LEFTENCODER-3.S, MULTIPLEXERA.1Y
- removed net N$16: LEFTENCODER-5.S, MULTIPLEXERA.2Y
- removed net N$17: MULTIPLEXERA.3Y, RIGHTENCODER-3.S
- removed net N$18: MULTIPLEXERA.4Y, RIGHTENCODER-5.S
- removed net N$2: IC3A.Q, MULTIPLEXERA.1A, MULTIPLEXERA.2B
- removed net N$20: MULTIPLEXERA.!A!/B, U1.PL7
- removed net N$30: LED4.A, R16.2
- removed net N$32: C3.2, Q2.1, U2.XTAL1
- removed net N$34: R9.1, X1.2
- removed net N$35: R9.2, U2.D-
- removed net N$39: C14.1, U2.UCAP
- removed net N$40: R10.2, U2.PD7
- removed net N$41: U1.(RXD1/INT2)PD2, U2.PD2
- removed net N$42: U1.(TXD1/INT3)PD3, U2.PD3
- removed net N$43: LED1.A, R11.2
- removed net N$44: LED2.A, R12.2
- removed net N$45: LED1.C, U2.PD4
- removed net N$46: LED2.C, U2.PD5
- removed net N$51: H1.MOUNT, IC1.VI
- removed net N$52: LED4.C, U1.(AD0)PA0
- removed net N$53: SV1.5, U1.RESET
- removed net N$58: R7.2, SV2.5, U2.(~RESET)_(PC1_/_DW)
- removed net N$59: SV2.4, U2.PB2
- removed net N$60: SV2.1, U2.PB3
- removed net N$61: SV2.3, U2.PB1
- new net D+: U2.USBDP, X6.3
- new net D-: U2.USBDM, X6.2
- new net DTR: C11.1, U2.DTR
- new net LE1: LEFTENCODER-3.S, U6.Y
- new net LE2: LEFTENCODER-5.S, U7.Y
- new net LSELECT: IC2A.I, U1.PJ4(PCINT13), U6.~A/B
- new net LWAVE: IC2D.I, IC3A.CLK, U3.PB4
- new net LWAVE1: IC3A.Q, U6.A, U7.A
- new net LWAVE2: IC3B.Q, U6.B, U7.B
- new net N$12: U2.GND18
- new net OA1: SV3.8, U1.(A15)PC7
- new net OA2: SV3.6, U1.(A14)PC6
- new net OA3: SV3.4, U1.(A13)PC5
- new net OA4: SV3.2, U1.(A12)PC4
- new net OD1: SV3.7, U1.(OC0A/OC1C/PCINT7)PB7
- new net OD2: SV3.5, U1.PL3(OC5A)
- new net OD3: SV3.3, U1.PL4(OC5B)
- new net OD4: SV3.1, U1.PL5(OC5C)
- new net ORXM: SV3.9, U1.PJ0(RXD3/PCINT9)
- new net OTXM: SV3.10, U1.PJ1(TXD3/PCINT10)
- new net RE1: RIGHTENCODER-3.S, U9.Y
- new net RE2: RIGHTENCODER-5.S, U8.Y
- new net RESET: C11.2, R9.1, S1.2, SV1.5, U1.RESET, U2.RESET
- new net RSELECT: IC2B.I, U1.(AD3)PA3, U9.~A/B
- new net RWAVE: IC2E.I, IC4A.CLK, U4.PB4
- new net RWAVE1: IC4A.Q, U8.A, U9.A
- new net RWAVE2: IC4B.Q, U8.B, U9.B
- new net RXLED: LED2.C, U2.RXLED
- new net RXM: U1.(RXD1/INT2)PD2, U2.TXD
- new net STOP: U1.(OC3A/AIN1)PE3, U6.~G, U7.~G, U8.~G, U9.~G
- new net TXLED: LED1.C, U2.TXLED
- new net TXM: U1.(TXD1/INT3)PD3, U2.RXD
- net +5V: now also C10.1, C3.+, R7.2, R8.2, R9.2, SV3.12, U2.VCCIO, U5.OUT, U6.VCC, U7.VCC, U8.VCC, U9.VCC, X6.1; no longer IC1.VO, R11.1, R12.1, R16.1, R7.1, SV2.2, U2.AVCC, U2.UVCC, X1.1
- net GND: now also C10.2, C3.-, H1.MOUNT, S1.1, SV3.11, U2.CTS, U2.GND21, U2.TEST, U5.GND, U6.GND, U7.GND, U8.GND, U9.GND, X6.4; no longer C13.1, C14.2, C3.1, H2.MOUNT, IC1.GND, MULTIPLEXERA.G, R10.1, SV2.6, U2.GND, U2.UGND, X1.5
- net N$11: now also U2.AGND; no longer IC2B.I, IC4A.CLK, U4.PB1
- net N$14: now also IC2E.O; no longer IC2B.O
- net N$27: now also IC2D.O; no longer IC2A.O
- net N$3: now also IC2B.O, U8.~A/B; no longer IC3B.Q, MULTIPLEXERA.1B, MULTIPLEXERA.2A
- net N$33: now also H2.MOUNT, U5.IN; no longer C13.2, Q2.2, U2.(PC0)_XTAL2
- net N$37: now also LED1.A, R7.1; no longer R8.1, X1.3
- net N$38: now also LED2.A, R8.1; no longer R8.2, U2.D+
- net N$7: now also U2.GND7; no longer IC4A.Q, MULTIPLEXERA.3A, MULTIPLEXERA.4A
- net N$8: now also IC2A.O, U7.~A/B; no longer IC4B.Q, MULTIPLEXERA.3B, MULTIPLEXERA.4B
Other:
- moved on the sheet: H1, H2, IC2A, IC2B, IC2P, IC3P, IC4P, LED1, LED2, LED3, MULTIPLEXERP, R1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

Commit message: completed board v1
Parts:
- removed MULTIPLEXER: 74LS257D, 74xx-eu:74LS257D
- removed U5: (no value), SparkFun-IC-Power:V_REG_78XXSIDE
- added U10: +12v, SparkFun-IC-Power:V_REG_78XX7812
Connections:
- removed net N$11: U2.AGND
- removed net N$12: U2.GND18
- removed net N$7: U2.GND7
- net +5V: now also U10.OUT; no longer MULTIPLEXERP.VCC, U5.OUT
- net GND: now also U10.GND, U2.AGND, U2.GND18, U2.GND7; no longer MULTIPLEXERP.GND, U5.GND
- net LDIR: now also U1.(AD2)PA2; no longer U1.PH6(OC2B)
- net LSELECT: now also U1.PL1(ICP5); no longer U1.PJ4(PCINT13)
- net LSPEED: now also U1.PK7(ADC15/PCINT23); no longer U1.(A9)PC1
- net N$33: now also U10.IN; no longer U5.IN
- net OD1: now also U1.(AD7)PA7; no longer U1.(OC0A/OC1C/PCINT7)PB7
- net OD2: now also U1.(AD6)PA6; no longer U1.PL3(OC5A)
- net OD3: now also U1.(AD5)PA5; no longer U1.PL4(OC5B)
- net OD4: now also U1.(AD4)PA4; no longer U1.PL5(OC5C)
- net RDIR: now also U1.(AD1)PA1; no longer U1.(SS/PCINT0)PB0
- net RSELECT: now also U1.PL2(T5); no longer U1.(AD3)PA3
- net RSPEED: now also U1.PK6(ADC14/PCINT22); no longer U1.(A8)PC0
- net RXM: now also U1.(RXD0/PCIN8)PE0; no longer U1.(RXD1/INT2)PD2
- net STOP: now also U1.PL0(ICP4); no longer U1.(OC3A/AIN1)PE3
- net TXM: now also U1.(TXD0)PE1; no longer U1.(TXD1/INT3)PD3

Commit message: complete board v1
Connections:
- net LDIR: now also U1.PK6(ADC14/PCINT22); no longer U1.(AD2)PA2
- net RSPEED: now also U1.PK5(ADC13/PCINT21); no longer U1.PK6(ADC14/PCINT22)
Changed lines of the file:
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@@
 </segment>
 <segment>
-<pinref part="U1" gate="1" pin="PK6(ADC14/PCINT22)"/>
-<wire x1="266.7" y1="15.24" x2="256.54" y2="15.24" width="0.1524" layer="91"/>
-<label x="256.54" y="15.24" size="1.778" layer="95"/>
+<pinref part="U1" gate="1" pin="PK5(ADC13/PCINT21)"/>
+<wire x1="266.7" y1="12.7" x2="256.54" y2="12.7" width="0.1524" layer="91"/>
+<label x="256.54" y="12.7" size="1.778" layer="95"/>
 </segment>
 </net>
@@
 </segment>
 <segment>
-<pinref part="U1" gate="1" pin="(AD2)PA2"/>
-<wire x1="337.82" y1="91.44" x2="347.98" y2="91.44" width="0.1524" layer="91"/>
-<label x="337.82" y="91.44" size="1.778" layer="95"/>
+<pinref part="U1" gate="1" pin="PK6(ADC14/PCINT22)"/>
+<wire x1="266.7" y1="15.24" x2="256.54" y2="15.24" width="0.1524" layer="91"/>
+<label x="256.54" y="15.24" size="1.778" layer="95"/>
 </segment>
 </net>

Commit message: minor improvements
Connections:
- net LE1: now also U1.(XCK0/AIN0)PE2
- net LE2: now also U1.(OC3A/AIN1)PE3
- net LSELECT: now also IC2F.I; no longer IC2A.I
- net LWAVE: now also IC2E.I; no longer IC2D.I
- net N$14: now also IC2B.O; no longer IC2E.O
- net N$27: now also IC2E.O; no longer IC2D.O
- net N$3: now also IC2A.O; no longer IC2B.O
- net N$8: now also IC2F.O; no longer IC2A.O
- net RDIR: now also U1.PK4(ADC12/PCINT20); no longer U1.(AD1)PA1
- net RE1: now also U1.(RXD1/INT2)PD2
- net RE2: now also U1.(TXD1/INT3)PD3
- net RSELECT: now also IC2A.I; no longer IC2B.I
- net RWAVE: now also IC2B.I; no longer IC2E.I
Other:
- moved on the sheet: IC2A, IC2B, IC2E
Changed lines of the file:
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@@
 <instance part="GND23" gate="1" x="490.22" y="-2.54"/>
 <instance part="P+22" gate="1" x="502.92" y="17.78"/>
-<instance part="IC2" gate="D" x="30.48" y="76.2" rot="R270"/>
-<instance part="IC2" gate="E" x="30.48" y="15.24" rot="R270"/>
 <instance part="U6" gate="A" x="180.34" y="93.98"/>
 <instance part="U7" gate="A" x="180.34" y="63.5"/>
@@
 <instance part="P+16" gate="1" x="152.4" y="111.76"/>
 <instance part="GND6" gate="1" x="149.86" y="-22.86"/>
-<instance part="IC2" gate="A" x="124.46" y="45.72" rot="R90"/>
-<instance part="IC2" gate="B" x="124.46" y="-15.24" rot="R90"/>
 <instance part="P+23" gate="1" x="462.28" y="132.08"/>
 <instance part="GND16" gate="1" x="462.28" y="99.06"/>
@@
 <instance part="GND26" gate="1" x="261.62" y="55.88"/>
 <instance part="U10" gate="G$1" x="490.22" y="10.16"/>
+<instance part="IC2" gate="F" x="124.46" y="45.72" rot="R90"/>
+<instance part="IC2" gate="A" x="124.46" y="-15.24" rot="R90"/>
+<instance part="IC2" gate="B" x="30.48" y="15.24" rot="R270"/>
+<instance part="IC2" gate="E" x="30.48" y="76.2" rot="R270"/>
 </instances>
 <busses>
@@
 <net name="N$27" class="0">
 <segment>
-<wire x1="30.48" y1="66.04" x2="30.48" y2="63.5" width="0.1524" layer="91"/>
 <wire x1="63.5" y1="63.5" x2="30.48" y2="63.5" width="0.1524" layer="91"/>
 <pinref part="IC3" gate="B" pin="CLK"/>
-<pinref part="IC2" gate="D" pin="O"/>
+<wire x1="30.48" y1="63.5" x2="30.48" y2="66.04" width="0.1524" layer="91"/>
+<pinref part="IC2" gate="E" pin="O"/>
 </segment>
 </net>
 <net name="N$14" class="0">
 <segment>
-<wire x1="30.48" y1="5.08" x2="30.48" y2="2.54" width="0.1524" layer="91"/>
 <wire x1="63.5" y1="2.54" x2="30.48" y2="2.54" width="0.1524" layer="91"/>
 <pinref part="IC4" gate="B" pin="CLK"/>
-<pinref part="IC2" gate="E" pin="O"/>
+<pinref part="IC2" gate="B" pin="O"/>
+<wire x1="30.48" y1="5.08" x2="30.48" y2="2.54" width="0.1524" layer="91"/>
 </segment>
 </net>
@@
 <label x="198.12" y="38.1" size="1.778" layer="95"/>
 </segment>
+<segment>
+<pinref part="U1" gate="1" pin="(RXD1/INT2)PD2"/>
+<wire x1="337.82" y1="22.86" x2="347.98" y2="22.86" width="0.1524" layer="91"/>
+<label x="337.82" y="22.86" size="1.778" layer="95"/>
+</segment>
 </net>
 <net name="RE2" class="0">
@@
 <label x="198.12" y="7.62" size="1.778" layer="95"/>
 </segment>
+<segment>
+<pinref part="U1" gate="1" pin="(TXD1/INT3)PD3"/>
+<wire x1="337.82" y1="25.4" x2="347.98" y2="25.4" width="0.1524" layer="91"/>
+<label x="337.82" y="25.4" size="1.778" layer="95"/>
+</segment>
 </net>
 <net name="LE1" class="0">
@@
 <label x="198.12" y="99.06" size="1.778" layer="95"/>
 </segment>
+<segment>
+<pinref part="U1" gate="1" pin="(XCK0/AIN0)PE2"/>
+<wire x1="337.82" y1="0" x2="347.98" y2="0" width="0.1524" layer="91"/>
+<label x="337.82" y="0" size="1.778" layer="95"/>
+</segment>
 </net>
 <net name="LE2" class="0">
@@
 <label x="198.12" y="68.58" size="1.778" layer="95"/>
 </segment>
+<segment>
+<pinref part="U1" gate="1" pin="(OC3A/AIN1)PE3"/>
+<wire x1="337.82" y1="2.54" x2="347.98" y2="2.54" width="0.1524" layer="91"/>
+<label x="337.82" y="2.54" size="1.778" layer="95"/>
+</segment>
 </net>
 <net name="RDIR" class="0">
@@
 </segment>
 <segment>
-<pinref part="U1" gate="1" pin="(AD1)PA1"/>
-<wire x1="337.82" y1="88.9" x2="347.98" y2="88.9" width="0.1524" layer="91"/>
-<label x="337.82" y="88.9" size="1.778" layer="95"/>
+<pinref part="U1" gate="1" pin="PK4(ADC12/PCINT20)"/>
+<wire x1="266.7" y1="10.16" x2="256.54" y2="10.16" width="0.1524" layer="91"/>
+<label x="256.54" y="10.16" size="1.778" layer="95"/>
 </segment>
 </net>
@@
 </segment>
 <segment>
-<wire x1="63.5" y1="86.36" x2="30.48" y2="86.36" width="0.1524" layer="91"/>
 <pinref part="IC3" gate="A" pin="CLK"/>
-<pinref part="IC2" gate="D" pin="I"/>
-<wire x1="30.48" y1="86.36" x2="17.78" y2="86.36" width="0.1524" layer="91"/>
+<label x="15.24" y="86.36" size="1.778" layer="95"/>
+<wire x1="17.78" y1="86.36" x2="30.48" y2="86.36" width="0.1524" layer="91"/>
+<pinref part="IC2" gate="E" pin="I"/>
+<wire x1="30.48" y1="86.36" x2="63.5" y2="86.36" width="0.1524" layer="91"/>
 <junction x="30.48" y="86.36"/>
-<label x="15.24" y="86.36" size="1.778" layer="95"/>
 </segment>
 </net>
@@
 <wire x1="63.5" y1="25.4" x2="30.48" y2="25.4" width="0.1524" layer="91"/>
 <pinref part="IC4" gate="A" pin="CLK"/>
-<pinref part="IC2" gate="E" pin="I"/>
 <wire x1="30.48" y1="25.4" x2="17.78" y2="25.4" width="0.1524" layer="91"/>
+<label x="15.24" y="25.4" size="1.778" layer="95"/>
+<pinref part="IC2" gate="B" pin="I"/>
 <junction x="30.48" y="25.4"/>
-<label x="15.24" y="25.4" size="1.778" layer="95"/>
 </segment>
 </net>
@@
 <net name="RSELECT" class="0">
 <segment>
-<pinref part="IC2" gate="B" pin="I"/>
-<wire x1="124.46" y1="-25.4" x2="124.46" y2="-30.48" width="0.1524" layer="91"/>
-<wire x1="124.46" y1="-30.48" x2="119.38" y2="-30.48" width="0.1524" layer="91"/>
 <wire x1="119.38" y1="-30.48" x2="111.76" y2="-30.48" width="0.1524" layer="91"/>
 <wire x1="111.76" y1="-30.48" x2="111.76" y2="25.4" width="0.1524" layer="91"/>
@@
 <wire x1="119.38" y1="-30.48" x2="119.38" y2="-33.02" width="0.1524" layer="91"/>
 <junction x="119.38" y="-30.48"/>
+<wire x1="119.38" y1="-30.48" x2="124.46" y2="-30.48" width="0.1524" layer="91"/>
+<pinref part="IC2" gate="A" pin="I"/>
+<wire x1="124.46" y1="-30.48" x2="124.46" y2="-25.4" width="0.1524" layer="91"/>
 </segment>
 <segment>
@@
 <net name="LSELECT" class="0">
 <segment>
-<pinref part="IC2" gate="A" pin="I"/>
-<wire x1="124.46" y1="35.56" x2="124.46" y2="33.02" width="0.1524" layer="91"/>
 <wire x1="124.46" y1="33.02" x2="119.38" y2="33.02" width="0.1524" layer="91"/>
 <wire x1="119.38" y1="33.02" x2="111.76" y2="33.02" width="0.1524" layer="91"/>
@@
 <wire x1="119.38" y1="33.02" x2="119.38" y2="30.48" width="0.1524" layer="91"/>
 <junction x="119.38" y="33.02"/>
+<pinref part="IC2" gate="F" pin="I"/>
+<wire x1="124.46" y1="33.02" x2="124.46" y2="35.56" width="0.1524" layer="91"/>
 </segment>
 <segment>
@@
 <net name="N$3" class="0">
 <segment>
-<pinref part="IC2" gate="B" pin="O"/>
 <pinref part="U8" gate="A" pin="~A/B"/>
+<pinref part="IC2" gate="A" pin="O"/>
 <wire x1="124.46" y1="-5.08" x2="162.56" y2="-5.08" width="0.1524" layer="91"/>
 </segment>
@@
 <net name="N$8" class="0">
 <segment>
-<pinref part="IC2" gate="A" pin="O"/>
 <pinref part="U7" gate="A" pin="~A/B"/>
+<pinref part="IC2" gate="F" pin="O"/>
 <wire x1="124.46" y1="55.88" x2="162.56" y2="55.88" width="0.1524" layer="91"/>
 </segment>
