File: Shields/Motor_Shield/MotorShield.brd (EAGLE design)
At the start: 40.8 x 54.5 mm, 38 parts, among them U1 ATMEGA328P_TQFP, U3 FT232RL, X1 2510-, X2 2510-, X3 C-GRID-05-15-91, X4 C-GRID-05-15-91, X5 MINI-USB_4P-32005-101, Y1 16MHz

Commit message: motor and light board
Parts:
- removed C5, C6: 0.1uF, SparkFun-Capacitors:0603
- removed C7: 10uF, SparkFun-Capacitors:0603-POLAR
- removed D1, D2: (no value), SparkFun-LED:LED-0603
- removed R15: 1k, SparkFun-Resistors:0603
- removed SV1: (no value), con-lstb:MA03-2
- removed U1: ATMEGA328P_TQFP, SparkFun-IC-Microcontroller:TQFP32-08
- removed U3: FT232RL, SparkFun-IC-Comms:SSOP28DB
- removed X5: MINI-USB_4P-32005-101, con-cypressindustries:32005-101
- removed Y1: 16MHz, SparkFun-Clocks:HC49US
- added C10, C11: 10pF, SparkFun-Capacitors:0603
- added C8, C9: 27pF, SparkFun-Capacitors:0603
- added JP1: (no value), jumper:JP2
- added U2: STM32F103RBT6, ST Microelctronics_By_element14_Batch_1:QFP50P1200X1200X160-64N
- added Y2: 8MHz, SparkFun-Clocks:CRYSTAL-SMD-5X3.2-4PAD
- added Y3: 32.768kHz, SparkFun-Clocks:CRYSTAL-SMD-3.2X1.5MM
- C3, C4: value 22pF -> 0.1uF
- R1: value 1M -> 10k
- R14: value 1k -> 10k
- S1: value MOMENTARY-SWITCH-SPST-SMD-5.2-REDUNDANT -> button
- moved R1 78.7 mm to (-6.00, -19.0), turned to 0 degrees
- moved C1 77.8 mm to (-6.00, -5.00), turned to 0 degrees
- moved C2 72.8 mm to (-6.00, -8.50), turned to 0 degrees
- moved R14 71.5 mm to (-6.00, -22.5), turned to 0 degrees
- moved C3 68.2 mm to (-6.00, -12.0), turned to 0 degrees
- moved C4 67.5 mm to (-6.00, -15.5), turned to 0 degrees
Connections:
- removed net DTR: C6.1, U3.2
- removed net N$10: U3.16, X5.2
- removed net N$11: U3.15, X5.3
- removed net N$14: D1.A, R14.1
- removed net N$15: D2.A, R15.1
- removed net N$16: D1.C, U3.23
- removed net N$17: D2.C, U3.22
- removed net N$3: C3.2, R1.2, U1.7, Y1.2
- removed net N$4: C4.2, R1.1, U1.8, Y1.1
- removed net RXM: U1.30, U3.1
- removed net TXM: U1.31, U3.5
- new net +3.3V: C1.1, C2.1, C3.1, C4.1, U2.1, U2.13, U2.19, U2.32, U2.48, U2.64
- new net +5V: JP1.1, R1.2, R14.2
- new net N$12: C8.1, U2.5, Y2.3
- new net N$13: C9.1, U2.6, Y2.1
- new net N$19: C11.1, U2.4, Y3.P$1
- new net N$20: C10.1, U2.3, Y3.P$2
- new net SCL: R14.1, U2.29
- new net SDA: R1.1, U2.30
- new net USBDM: U2.44
- new net USBDP: U2.45
- net GND: now also C10.2, C11.2, C3.2, C4.2, C8.2, C9.2, JP1.3, U2.12, U2.18, U2.31, U2.47, U2.63; no longer C3.1, C4.1, C5.2, C7.-, SV1.1, U1.21, U1.3, U1.5, U3.11, U3.18, U3.21, U3.25, U3.26, U3.7, X5.4
- net LDIR: no longer U1.9
- net LDISABLEI: no longer U1.11
- net LEA: no longer U1.26
- net LEB: no longer U1.25
- net LSPEED: no longer U1.10
- net MISO: now also U2.22; no longer SV1.6, U1.16
- net MOSI: now also U2.23; no longer SV1.3, U1.15
- net N$2: now also JP1.2, U2.60; no longer C1.1, U1.20
- net RDIR: no longer U1.13
- net RDISABLEI: no longer U1.12
- net REA: no longer U1.27
- net REB: no longer U1.28
- net RESET: now also U2.7; no longer C6.2, SV1.2, U1.29
- net RSPEED: no longer U1.14
- net SCK: now also U2.21; no longer SV1.4, U1.17
- net VCC: no longer C2.1, C5.1, C7.+, R14.2, R15.2, SV1.5, U1.18, U1.4, U1.6, U3.20, U3.4, X5.1
Routing:
- net RXM: track 30.0 -> 0.00 mm
- net GND: track 57.1 -> 27.7 mm, vias 20 -> 8
- net N$11: track 26.7 -> 0.00 mm
- net N$10: track 24.5 -> 0.00 mm
- net TXM: track 20.7 -> 0.00 mm
- net DTR: track 15.6 -> 0.00 mm, vias 2 -> 0
- net RESET: track 45.2 -> 29.9 mm
- net N$4: track 13.4 -> 0.00 mm
- net N$3: track 12.0 -> 0.00 mm
- net N$17: track 12.0 -> 0.00 mm
- net MISO: track 8.98 -> 0.00 mm
- net N$16: track 8.45 -> 0.00 mm
- net SCK: track 7.09 -> 0.00 mm
- net MOSI: track 5.58 -> 0.00 mm
- net LDIR: track 6.01 -> 3.18 mm
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