File: Motor and Light/MotorAndLightmBed.sch (EAGLE design)
At the start: 131 parts, among them J6 6_PIN_SERIAL_CABLEPTH, J8 1981568-1, Q1 BSS84, Q3 BC846ASMD, Q4 220mA/50V/3.5Ω, Q5 220mA/50V/3.5Ω, Q6 220mA/50V/3.5Ω, Q7 220mA/50V/3.5Ω, U1 9DoF IMU, U2 LPC1768FBD100, X1 2510-, X2 2510-, X3 C-GRID-05-15-91, X4 C-GRID-05-15-91, X5 C-GRID-02-70553, X6 SI-50170, Y1 32.768kHz, Y2 OSCILLATORSMD-5X3-50MHz, Y3 OSCILLATORSMD-5X3-12MHz

Commit message: Bad Update After Review
Parts:
- removed D8: (no value), SparkFun-LED:LED0603
- removed J8: 1981568-1, DigiKey:1981568-1
- removed Q7: 220mA/50V/3.5Ω, SparkFun-DiscreteSemi:MOSFET-NCH-BSS138
- removed R57, R58: 200, SparkFun-Resistors:200OHM-0603-1/10W-1%
- removed R60, R61, R65: 2700, SparkFun-Resistors:3.9KOHM-0603-1/10W-1%
- removed R63: 536, SparkFun-Resistors:3.9KOHM-0603-1/10W-1%
- removed R68, R69, R70, R73: 10k, SparkFun-Resistors:10KOHM-0603-1/10W-1%
- added D2: (no value), SparkFun-LED:LED0603
- added J7: (no value), SparkFun-Connectors:CONN_025MM
- added Q2: BC846ASMD, transistor-npn:BC846ASMD
- added R12, R13: 49.9, rcl:R-US_R0603
- added R20: 10k, SparkFun-Resistors:10KOHM-0603-1/10W-1%
- added R21: 4.87k, rcl:R-US_R0603
- added R22: 100k, SparkFun-Resistors:100KOHM-0603-1/10W-1%
- added R23: 150, SparkFun-Resistors:150OHM-0603-1/10W-1%
- added R36: 2700, SparkFun-Resistors:2.55KOHM-0603-1/10W-1%
- added R37, R38: 200, SparkFun-Resistors:200OHM-0603-1/10W-1%
- added R42: 2700, SparkFun-Resistors:3.9KOHM-0603-1/10W-1%
- C1, C2: value 18pF -> 0.1uF; device SparkFun-Capacitors:18PF-0603-50V-5% -> SparkFun-Capacitors:0.1UF-0603-25V-(+80/-20%)
- C10, C11: value 18pF -> 0.1uF; device SparkFun-Capacitors:18PF-0603-50V-5% -> SparkFun-Capacitors:0.1UF-0603-25V-5%
- C12: value 1nF -> 0.1uF; device SparkFun-Capacitors:1.0NF/1000PF-0603-50V-10% -> SparkFun-Capacitors:0.1UF-0603-25V-5%
- C13: value 0.1uF -> 10uF; device SparkFun-Capacitors:0.1UF-0603-25V-(+80/-20%) -> SparkFun-Capacitors:10UF-POLAR-0603-6.3V-20%(TANT)
- C14, C27, C28, C29: device SparkFun-Capacitors:0.1UF-0603-25V-(+80/-20%) -> SparkFun-Capacitors:0.1UF-0603-25V-5%
- C15: value 0.1uF -> 10uF; device SparkFun-Capacitors:0.1UF-0603-25V-5% -> SparkFun-Capacitors:10UF-POLAR-0603-6.3V-20%(TANT)
- C16, C17, C18, C19, C20, C24, C25: device SparkFun-Capacitors:0.1UF-0603-25V-5% -> SparkFun-Capacitors:0.1UF-0603-25V-(+80/-20%)
- C22: value 10uF -> 0.1uF; device SparkFun-Capacitors:10UF-POLAR-0603-6.3V-20%(TANT) -> SparkFun-Capacitors:0.1UF-0603-25V-(+80/-20%)
- C3: value 100pF -> 18pF; device SparkFun-Capacitors:100PF-0603-50V-5% -> SparkFun-Capacitors:18PF-0603-50V-5%
- C4, C5, C6: value 0.1uF -> 18pF; device SparkFun-Capacitors:0.1UF-0603-25V-(+80/-20%) -> SparkFun-Capacitors:18PF-0603-50V-5%
- C7: value 0.1uF -> 100pF; device SparkFun-Capacitors:0.1UF-0603-25V-(+80/-20%) -> SparkFun-Capacitors:100PF-0603-50V-5%
- C8: value 0.1uF -> 1000pF; device SparkFun-Capacitors:0.1UF-0603-25V-(+80/-20%) -> SparkFun-Capacitors:1.0NF/1000PF-0603-50V-10%
- C9: value 10uF -> 0.1uF; device SparkFun-Capacitors:10UF-POLAR-0603-6.3V-20%(TANT) -> SparkFun-Capacitors:0.1UF-0603-25V-5%
- J1: value (none) -> 1981568-1; device SparkFun-Connectors:CONN_12LOCK_LONGPADS -> DigiKey:1981568-1
- J2: device SparkFun-Connectors:CONN_025MM -> SparkFun-Connectors:CONN_05X2SHD
- J3: value (none) -> 6_PIN_SERIAL_CABLEPTH; device SparkFun-Connectors:CONN_025MM -> SparkFun-Connectors:6_PIN_SERIAL_CABLEPTH
- J4: device SparkFun-Retired:CONN_02POLAR -> SparkFun-Connectors:CONN_12LOCK_LONGPADS
- J5: device SparkFun-Connectors:CONN_05X2SHD -> SparkFun-Retired:CONN_02POLAR
- J6: value 6_PIN_SERIAL_CABLEPTH -> (none); device SparkFun-Connectors:6_PIN_SERIAL_CABLEPTH -> SparkFun-Connectors:CONN_025MM
- Q3: value BC846ASMD -> 220mA/50V/3.5Ω; device transistor-npn:BC846ASMD -> SparkFun-DiscreteSemi:MOSFET-NCH-BSS138
- R1: value 1.5k -> 33; device SparkFun-Resistors:1.5KOHM-0603-1/10W-1% -> SparkFun-Resistors:33OHM-0603-1/10W-1%
- R10, R9: value 10k -> 1k; device SparkFun-Resistors:10KOHM-0603-1/10W-1% -> SparkFun-Resistors:1KOHM-0603-1/10W-1%
- R15: value 47k -> 49.9; device SparkFun-Resistors:47KOHM-0603-1/10W-1% -> rcl:R-US_R0603
- R16, R17, R18: value 49.9 -> 10k; device rcl:R-US_R0603 -> SparkFun-Resistors:10KOHM-0603-1/10W-1%
- R19: value 4.87k -> 10k; device rcl:R-US_R0603 -> SparkFun-Resistors:10KOHM-0603-1/10W-1%
- R2: value 1k -> 33; device SparkFun-Resistors:1KOHM-0603-1/10W-1% -> SparkFun-Resistors:33OHM-0603-1/10W-1%
- R24: value 2.2k -> 150; device SparkFun-Resistors:2.2KOHM-0603-1/10W-1% -> SparkFun-Resistors:150OHM-0603-1/10W-1%
- R25: value 10k -> 2.2k; device SparkFun-Resistors:10KOHM-0603-1/10W-1% -> SparkFun-Resistors:2.2KOHM-0603-1/10W-1%
- R26: value 10k -> 2700; device SparkFun-Resistors:10KOHM-0603-1/10W-1% -> SparkFun-Resistors:3.9KOHM-0603-1/10W-1%
- R27: value 10k -> 2700; device SparkFun-Resistors:10KOHM-0603-1/10W-1% -> SparkFun-Resistors:2.55KOHM-0603-1/10W-1%
- R28: value 10k -> 200; device SparkFun-Resistors:10KOHM-0603-1/10W-1% -> SparkFun-Resistors:200OHM-0603-1/10W-1%
- R29: value 100k -> 200; device SparkFun-Resistors:100KOHM-0603-1/10W-1% -> SparkFun-Resistors:200OHM-0603-1/10W-1%
- R3: value 2700 -> 1.5k; device SparkFun-Resistors:3.9KOHM-0603-1/10W-1% -> SparkFun-Resistors:1.5KOHM-0603-1/10W-1%
- R30: value 33 -> 2700; device SparkFun-Resistors:33OHM-0603-1/10W-1% -> SparkFun-Resistors:3.9KOHM-0603-1/10W-1%
- R31: value 33 -> 200; device SparkFun-Resistors:33OHM-0603-1/10W-1% -> SparkFun-Resistors:200OHM-0603-1/10W-1%
- R32: value 150 -> 200; device SparkFun-Resistors:150OHM-0603-1/10W-1% -> SparkFun-Resistors:200OHM-0603-1/10W-1%
- R33: value 150 -> 2700; device SparkFun-Resistors:150OHM-0603-1/10W-1% -> SparkFun-Resistors:3.9KOHM-0603-1/10W-1%
- R46: value 2700 -> 536; device SparkFun-Resistors:2.55KOHM-0603-1/10W-1% -> SparkFun-Resistors:3.9KOHM-0603-1/10W-1%
- R47, R48: value 2700 -> 200; device SparkFun-Resistors:2.55KOHM-0603-1/10W-1% -> SparkFun-Resistors:200OHM-0603-1/10W-1%
- R49: value 200 -> 2700; device SparkFun-Resistors:200OHM-0603-1/10W-1% -> SparkFun-Resistors:2.55KOHM-0603-1/10W-1%
- R50, R51, R54, R55: value 200 -> 10k; device SparkFun-Resistors:200OHM-0603-1/10W-1% -> SparkFun-Resistors:10KOHM-0603-1/10W-1%
- R52: value 200 -> 2700; device SparkFun-Resistors:200OHM-0603-1/10W-1% -> SparkFun-Resistors:3.9KOHM-0603-1/10W-1%
- R6: value 2700 -> 47k; device SparkFun-Resistors:3.9KOHM-0603-1/10W-1% -> SparkFun-Resistors:47KOHM-0603-1/10W-1%
- R7: value 1k -> 10k; device SparkFun-Resistors:1KOHM-0603-1/10W-1% -> SparkFun-Resistors:10KOHM-0603-1/10W-1%
- T1: device transistor:-PNP-TO220V -> transistor:-NPN-TO220V
- T10: device transistor:-NPN-TO220V -> transistor:-PNP-TO220V
- X3: value C-GRID-05-15-91 -> SI-50170; device con-molex:C-GRID-05-15-91 -> con-stewart:SI-50170
- X5: value C-GRID-02-70553 -> C-GRID-05-15-91; device con-molex:C-GRID-02-70553 -> con-molex:C-GRID-05-15-91
- X6: value SI-50170 -> C-GRID-02-70553; device con-stewart:SI-50170 -> con-molex:C-GRID-02-70553
- Y2: value OSCILLATORSMD-5X3-50MHz -> OSCILLATORSMD-5X3-12MHz
- Y3: value OSCILLATORSMD-5X3-12MHz -> OSCILLATORSMD-5X3-50MHz
- renumbered C47 to C30, D10 to D3, D7 to D4, D9 to D1, OK3 to OK2, R56 to R41, R59 to R34, R62 to R35, R64 to R43, R66 to R45, R67 to R39, R71 to R44, R72 to R40, U$2 to MU1
Connections:
- removed net TRST: U2.!TRST
- net +12V: now also J6.1, R30.2, R32.2, R53.2, T2.E, T5.E, T8.E; no longer J2.1, R55.2, R57.2, R6.2, T1.E, T7.E, T9.E
- net +24V: now also J7.1, R33.2; no longer J3.1, R65.2
- net +3V3: now also C1.1, C10.2, C11.1, C15.+, C17.2, C19.1, C21.+, C22.1, C23.1, C25.1, C27.1, C29.2, C9.2, Q3.G, R11.2, R12.1, R13.2, R20.1, R22.2, R50.2, R51.2, R52.2, R6.2, X3.RCT, X3.TCT, Y2.EN; no longer C13.1, C15.2, C16.2, C20.2, C22.+, C23.2, C28.1, C29.1, C5.1, C6.1, C7.1, C8.1, C9.+, Q7.G, R16.2, R17.1, R24.2, R27.2, R28.1, R29.2, R61.2, R68.2, R70.2, X6.RCT, X6.TCT, Y3.EN
- net +5V: now also J1.1, R54.2, R55.2; no longer J8.1, R69.2, R73.2
- net 12MHZ: now also C7.1, Y2.OUT; no longer C3.1, Y3.OUT
- net 1S1: now also R28.1; no longer R49.1
- net 1S1O: now also J4.4, T3.E; no longer J1.4, T2.E
- net 1S2: now also R37.1; no longer R51.1
- net 1S2O: now also J4.5, T6.E; no longer J1.5, T4.E
- net 1S3: now also R47.1; no longer R53.1
- net 1S3O: now also J4.6, T9.E; no longer J1.6, T6.E
- net 2S1: now also R29.1; no longer R50.1
- net 2S1O: now also J4.10, T4.E; no longer J1.10, T3.E
- net 2S2: now also R38.1; no longer R52.1
- net 2S2O: now also J4.11, T7.E; no longer J1.11, T5.E
- net 2S3: now also R48.1; no longer R54.1
- net 2S3O: now also J4.12, T10.E; no longer J1.12, T8.E
- net 50MHZ: now also Y3.OUT; no longer Y2.OUT
- net BATTIN: now also R46.2; no longer R63.2
- net BLUE: now also J4.1, R36.1; no longer J1.1, R47.1
- net ESTOP: now also R42.2, X6-1.S, X6-2.S; no longer R3.2, X5-1.S
- net ETH_LED1: now also R23.2, X3.A; no longer R32.2, X6.A
- net ETH_LED2: now also R24.2, X3.A1; no longer R33.2, X6.A1
- net ETH_OSC_EN: now also Y3.EN; no longer Y2.EN
- net GND: now also C1.2, C10.1, C13.-, C14.1, C15.-, C16.2, C2.2, C20.2, C22.2, C23.2, C29.1, C3.2, C4.1, C5.1, C9.1, D2.C, J1.5, J2.3, J2.5, J2.9, J3.6, J6.2, J7.2, Q2.E, R21.2, R31.1, R42.1, R46.1, T1.E, T10.C, X3.C, X3.C1, X3.S1, X3.S2, X5-1.S; no longer C1.1, C10.2, C13.2, C14.2, C15.1, C16.1, C2.1, C20.1, C22.-, C23.1, C29.2, C4.2, C5.2, C7.2, C9.-, D8.C, J2.2, J3.2, J5.3, J5.5, J5.9, J6.6, J8.5, Q3.E, R26.2, R3.1, R58.1, R63.1, S1.2, S1.3, T1.C, T10.E, X3-1.S, X6.C, X6.C1, X6.S1, X6.S2
- net GREEN: now also J4.2, R49.1; no longer J1.2, R48.1
- net LALI: now also R7.2; no longer R8.2
- net LBLI: now also R16.2; no longer R11.2
- net LDIR: now also R9.1; no longer R5.1
- net LEA: now also Q3.D, X4-3.S; no longer Q4.D, X3-3.S
- net LEA3: now also Q3.S; no longer Q4.S
- net LEB: now also Q4.D, X4-5.S; no longer Q6.D, X3-5.S
- net LEB3: now also Q4.S; no longer Q6.S
- net LGND: now also R16.1, R7.1; no longer R11.1, R8.1
- net LPC_D+: now also J1.3, R1.1; no longer J8.3, R30.1
- net LPC_D-: now also J1.2, R2.1; no longer J8.2, R31.1
- net LSPEED: now also R4.1; no longer R2.1
- net N$1: now also R4.2; no longer R2.2
- net N$10: now also C7.2; no longer C3.2
- net N$11: now also R23.1; no longer R32.1
- net N$13: now also C2.1; no longer C14.1
- net N$14: now also R21.1; no longer R19.1
- net N$15: now also R24.1; no longer R33.1
- net N$16: now also R25.1; no longer R24.1
- net N$2: now also C4.2; no longer C1.2
- net N$24: now also J5.1, J5.2, R30.1, T1.C; no longer J4.1, R6.1, T10.C
- net N$3: now also C5.2; no longer C2.2
- net N$34: now also R27.2, R32.1, T2.B; no longer R46.2, R55.1, T1.B
- net N$36: now also R36.2, T5.B; no longer R47.2, T9.B
- net N$38: now also R49.2, R53.1, T8.B; no longer R48.2, R57.1, T7.B
- net N$4: now also R3.1; no longer R1.1
- net N$40: now also R47.2, T9.B; no longer R53.2, T6.B
- net N$41: now also R37.2, T6.B; no longer R51.2, T4.B
- net N$42: now also R28.2, T3.B; no longer R49.2, T2.B
- net N$43: now also R29.2, T4.B; no longer R50.2, T3.B
- net N$44: now also R38.2, T7.B; no longer R52.2, T5.B
- net N$45: now also R48.2, T10.B; no longer R54.2, T8.B
- net N$46: now also R26.2; no longer R60.2
- net N$47: now also D2.A, R26.1; no longer D5.A, R60.1
- net N$49: now also Q2.B, R31.2; no longer Q3.B, R58.2
- net N$50: now also D5.A; no longer D6.A
- net N$51: now also Q2.C, R33.1; no longer Q3.C, R65.1
- net N$54: now also D6.A, R52.1; no longer D8.A, R61.1
- net N$6: now also R5.2; no longer R4.2
- net N$7: now also R10.2; no longer R7.2
- net N$9: now also R9.2; no longer R5.2
- net NRESET: now also C16.1, C8.1, J2.10, R22.1, R6.1; no longer C12.1, C27.1, J5.10, R15.1, R29.1
- net PFBOUT: now also C12.1, C13.+, C14.2, C28.1; no longer C17.2, C19.1, C21.+, C25.1
- net RALI: now also R8.2; no longer R10.2
- net RBLI: now also R17.2; no longer R9.2
- net RD+: now also R13.1, X3.RD+; no longer R16.1, X6.RD+
- net RD-: now also R12.2, X3.RD-; no longer R14.2, X6.RD-
- net RDIR: now also R10.1; no longer R7.1
- net REA: now also R54.1, X5-3.S; no longer R69.1, X4-3.S
- net REA3: now also R50.1; no longer R68.1
- net REB: now also Q6.D, R55.1, X5-5.S; no longer Q7.D, R73.1, X4-5.S
- net REB3: now also Q6.S, R51.1; no longer Q7.S, R70.1
- net RED: now also J4.3, R27.1; no longer J1.3, R46.1
- net RGND: now also R17.1, R8.1; no longer R10.1, R9.1
- net RSPEED: now also R5.1; no longer R4.1
- net RTCK: now also J2.7, R11.1; no longer J5.7, R25.1
- net SLIGHT: now also T1.B; no longer T10.B
- net TCLK: now also J2.4, R19.1; no longer J5.4, R26.1
- net TD+: now also R15.1, X3.TD+; no longer R18.1, X6.TD+
- net TD-: now also R14.2, X3.TD-; no longer R17.2, X6.TD-
- net TDI: now also J2.8, R20.2; no longer J5.8, R28.2
- net TDO: now also J2.6; no longer J5.6
- net TGT_RXD: now also J3.3; no longer J6.3
- net TGT_TXD: now also J3.2; no longer J6.2
- net TMS: now also J2.2, R18.1; no longer J5.2, R27.1
- net USB_D+: now also C3.1, R3.2; no longer C10.1, R30.2
- net USB_D-: now also C6.1, R2.2; no longer C11.1, R31.2
- net VCC: now also X5-4.S; no longer X3-4.S
- net VDDA: now also C20.1; no longer C4.1
Other:
- note added: "Current limiting R"
- note added: "Pin 13 Connected to +3V3 to make PCB compatible with LPC2368"
- moved on the sheet: C1, C10, C11, C12, C14, C16, C17, C18, C19, C2, C20, C21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
