File: Motor and Light/MotorBoard.sch (EAGLE design)
At the start: 132 parts, among them J1 1981568-1, J2 Programming Port, J3 6_PIN_SERIAL_CABLEPTH, J4 Under Glow, J5 Safety Light, J6 12V, J7 24V, Q1 BSS84, Q2 BC846ASMD, Q3 220mA/50V/3.5Ω, Q4 220mA/50V/3.5Ω, Q5 220mA/50V/3.5Ω, Q6 220mA/50V/3.5Ω, T1 TIP41A, T10 TIP41A, T2 TIP41A, T3 TIP41A, T4 TIP41A, T5 TIP41A, T6 TIP41A, T7 TIP41A, T8 TIP41A, T9 TIP41A, U1 9DoF IMU, U2 LPC1768FBD100, U3 DP83848JSQ/NOPB, X1 2510-, X2 2510-, X3 SI-50170, X4 C-GRID-05-15-91, X5 C-GRID-05-15-91, X6 C-GRID-02-70553, Y1 32.768kHz, Y2 OSCILLATORSMD-5X3-12MHz, Y3 OSCILLATORSMD-5X3-50MHz

Commit message: Schematics Beautified
Other:
- note added: "12MHz Oscillator"
- note added: "12V 24V Jack"
- note added: "50MHz Oscillator"
- note added: "9Dof IMU"
- note added: "???"
- note added: "E-Stop"
- note added: "Encoder Ports"
- note added: "Ethernet Chip"
- note added: "Ethernet Jack"
- note added: "Inverter"
- note added: "OSMC Ports"
- note added: "Optoisolator"
- note added: "Power"
- note added: "Safety Light"
- note added: "Serial and USB"
- note added: "THE mbed chip"
- note added: "Transistor Array"
- note added: "Under Glow"
- note added: "Voltage Regulator"
- note removed: "Get NPN Transistors"
- note removed: "This is Wrong"
- note removed: "need to verify this"
