File: Motor and Light/MotorBoardDev.sch (EAGLE design)
At the start: 83 parts, among them J1 Under Glow, J2 Safety Light, J3 12V, J4 24V, Q1 TIP42C, Q10 TIP42C, Q11 TIP42C, Q15 TIP41C, Q16 TIP41C, Q2 220mA/50V/3.5Ω, Q3 TIP42C, Q4 TIP42C, Q5 TIP42C, Q6 TIP42C, Q7 220mA/50V/3.5Ω, Q8 220mA/50V/3.5Ω, Q9 220mA/50V/3.5Ω, T1 NCP1117DT50GOS-ND, T2 TIP41A, T3 NCP1117DT33GOS-ND, U2 9DoF IMU, X1 C-GRID-05-15-91, X2 C-GRID-05-15-91, X3 MINI-USB_SHIELD5P4-32005-400, X4 C-GRID-02-70553, X5 SI-50170, X7 2510-, X8 2510-

Commit message: Somehoe the branch still exists
Parts:
- added D5: BLUE, SparkFun-LED:LED-BLUE0603
- added U1: TXB0104DR, MotorBoardDev:TXB0104DR
- D3: value WHITE -> Yellow; device SparkFun-LED:LED-WHITE0603 -> SparkFun-LED:LED-YELLOW0603
- R10: value 200 -> 4.7k
- R16: value 200 -> 500
- R25, R27, R28, R29: value 10k -> 4.7k
Connections:
- net D+ renamed D_P
- net D- renamed D_N
- net RD+ renamed RD_P
- net RD- renamed RD_N
- net TD+ renamed TD_P
- net TD- renamed TD_N
- removed net ID: X3G$1.4
- new net N$7: J2.2, T2.E
- net BLUE: no longer A1.P$21
- net ESTOP: now also A1.P$22; no longer A1.P$24
- net GND: now also D5.C; no longer J1.4, J1.8, J1.9, J2.2
- net GREEN: no longer A1.P$22
- net INDICATOR_LED: now also D5.A
- net LDIR: now also A1.P$24; no longer A1.P$26
- net LSPEED: now also A1.P$23; no longer A1.P$25
- net N$1: no longer T2.E
- net RDIR: now also A1.P$26; no longer A1.P$28
- net RED: no longer A1.P$23
- net RSPEED: now also A1.P$25; no longer A1.P$27
Other:
- note added: "#S#O control which bar lights up RGB control the color of the entire stripe"
- note added: "(By OSMC Schematics"
- note added: "30Ω"
- note added: "Add disable"
- note added: "Also make sure this is the chip we want"
- note added: "Buck converter"
- note added: "Check layout package"
- note added: "If have space add Optoisolator for HI lines"
- note added: "Label them on the board"
- note added: "Level shifting"
- note added: "Make them bigger"
- note added: "Motor stuff go to PWM"
- note added: "Power distribution load switch"
- note added: "Put it bak on"
- note added: "RGB are currently not connected to the mbed"
- note added: "Rename those as LSPEED and LDIR"
- note added: "TXB0104DR"
- note added: "Use I2C pullup resistance"
- note added: "Use Neopixels"
- note added: "Use quad-line 12V inverter"
- note added: "also goes for this"
- note added: "do the same for safety light"
- note added: "fix this"
- note added: "get a SMD?"
- note added: "go from 5v to 3v3 not 12V"
- note added: "make absolute voltage 3V"
- note added: "not anymore"
- note removed: "Also logical shifters"
- note removed: "How it works?"
- note removed: "ID set to floating to identify the board as a slave"
- note removed: "Overkill?"
- note removed: "RGB control pin underglow thrown to PWM"
- note removed: "all of Speed control thrown to PWM"
- note removed: "pull up resistor position changed, it'll no longer short L/R+12V to L/R GND"
- moved on the sheet: C3, C4, Q15, Q16, R18, R19, R2, R3, R4, T2, U2
