File: estop/Eagle Files/RJ_IGVC_Estop.sch (EAGLE design)
At the start: 18 parts, among them IC1 LDL1117S33R, U4 ATMEGA328P-AUR, X1 2X3SHROUDED, X2 1751248, X3 1751248

Commit message: Finished board
Connections:
- net +5V renamed +3.3V
Changed lines of the file:
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@@
 <?xml version="1.0" encoding="utf-8"?>
 <!DOCTYPE eagle SYSTEM "eagle.dtd">
-<eagle version="8.5.2">
+<eagle version="8.3.2">
 <drawing>
 <settings>
@@
 </classes>
 <parts>
-<part name="SUPPLY34" library="supply2" library_urn="urn:adsk.eagle:library:372" deviceset="+5V" device=""/>
+<part name="SUPPLY34" library="supply1" library_urn="urn:adsk.eagle:library:371" deviceset="+3V3" device=""/>
 <part name="SUPPLY35" library="supply2" library_urn="urn:adsk.eagle:library:372" deviceset="GND" device=""/>
 <part name="SUPPLY21" library="supply2" library_urn="urn:adsk.eagle:library:372" deviceset="GND" device=""/>
-<part name="SUPPLY23" library="supply2" library_urn="urn:adsk.eagle:library:372" deviceset="+5V" device=""/>
+<part name="SUPPLY23" library="supply1" library_urn="urn:adsk.eagle:library:371" deviceset="+3V3" device=""/>
 <part name="R2" library="rcl" library_urn="urn:adsk.eagle:library:334" deviceset="R-US_" device="R0603" package3d_urn="urn:adsk.eagle:package:23555/2" value="10k"/>
 <part name="C7" library="rcl" library_urn="urn:adsk.eagle:library:334" deviceset="C-US" device="C0603" package3d_urn="urn:adsk.eagle:package:23616/2" value="4.7uF"/>
-<part name="SUPPLY22" library="supply2" library_urn="urn:adsk.eagle:library:372" deviceset="+5V" device=""/>
-<part name="SUPPLY27" library="supply2" library_urn="urn:adsk.eagle:library:372" deviceset="+5V" device=""/>
+<part name="SUPPLY22" library="supply1" library_urn="urn:adsk.eagle:library:371" deviceset="+3V3" device=""/>
+<part name="SUPPLY27" library="supply1" library_urn="urn:adsk.eagle:library:371" deviceset="+3V3" device=""/>
 <part name="SUPPLY28" library="supply2" library_urn="urn:adsk.eagle:library:372" deviceset="GND" device=""/>
 <part name="SUPPLY6" library="supply2" library_urn="urn:adsk.eagle:library:372" deviceset="GND" device=""/>
 <part name="C3" library="rcl" library_urn="urn:adsk.eagle:library:334" deviceset="C-US" device="C0603" package3d_urn="urn:adsk.eagle:package:23616/2" value="0.1uF"/>
 <part name="C2" library="rcl" library_urn="urn:adsk.eagle:library:334" deviceset="C-US" device="C0603" package3d_urn="urn:adsk.eagle:package:23616/2" value="0.1uF"/>
-<part name="SUPPLY5" library="supply2" library_urn="urn:adsk.eagle:library:372" deviceset="+5V" device=""/>
+<part name="SUPPLY5" library="supply1" library_urn="urn:adsk.eagle:library:371" deviceset="+3V3" device=""/>
 <part name="X1" library="lcd-buzzer" deviceset="2X3SHROUDED" device=""/>
 <part name="U4" library="lcd-buzzer" deviceset="ATMEGA328P-*" device="AUR"/>
@@
 <part name="R5" library="resistor" library_urn="urn:adsk.eagle:library:348" deviceset="R-US_" device="R0603" package3d_urn="urn:adsk.eagle:package:26057/1" value="300"/>
 <part name="SUPPLY2" library="supply2" library_urn="urn:adsk.eagle:library:372" deviceset="GND" device=""/>
-<part name="SUPPLY3" library="supply2" library_urn="urn:adsk.eagle:library:372" deviceset="+5V" device=""/>
+<part name="SUPPLY3" library="supply1" library_urn="urn:adsk.eagle:library:371" deviceset="+3V3" device=""/>
 <part name="FRAME2" library="RoboJackets-Frames" deviceset="FRAME_A_L" device=""/>
 <part name="X2" library="con-phoenix-350" library_urn="urn:adsk.eagle:library:174" deviceset="1751248" device="" package3d_urn="urn:adsk.eagle:package:9395/1"/>
@@
 <part name="JP1" library="pinhead" library_urn="urn:adsk.eagle:library:325" deviceset="PINHD-2X4" device="" package3d_urn="urn:adsk.eagle:package:22461/2"/>
 <part name="SUPPLY4" library="supply2" library_urn="urn:adsk.eagle:library:372" deviceset="GND" device=""/>
-<part name="SUPPLY7" library="supply2" library_urn="urn:adsk.eagle:library:372" deviceset="+5V" device=""/>
+<part name="SUPPLY7" library="supply1" library_urn="urn:adsk.eagle:library:371" deviceset="+3V3" device=""/>
 <part name="X3" library="con-phoenix-350" library_urn="urn:adsk.eagle:library:174" deviceset="1751248" device="" package3d_urn="urn:adsk.eagle:package:9395/1"/>
-<part name="SUPPLY8" library="supply2" library_urn="urn:adsk.eagle:library:372" deviceset="+5V" device=""/>
+<part name="SUPPLY8" library="supply1" library_urn="urn:adsk.eagle:library:371" deviceset="+3V3" device=""/>
 <part name="R1" library="resistor" library_urn="urn:adsk.eagle:library:348" deviceset="R-US_" device="R0603" package3d_urn="urn:adsk.eagle:package:26057/1" value="300"/>
 <part name="SUPPLY9" library="supply2" library_urn="urn:adsk.eagle:library:372" deviceset="GND" device=""/>
@@
 </plain>
 <instances>
-<instance part="SUPPLY34" gate="+5V" x="43.18" y="124.46"/>
+<instance part="SUPPLY34" gate="G$1" x="43.18" y="124.46"/>
 <instance part="SUPPLY35" gate="GND" x="43.18" y="99.06"/>
 <instance part="SUPPLY21" gate="GND" x="76.2" y="22.86"/>
-<instance part="SUPPLY23" gate="+5V" x="83.82" y="20.32"/>
+<instance part="SUPPLY23" gate="G$1" x="83.82" y="20.32"/>
 <instance part="R2" gate="G$1" x="76.2" y="53.34" rot="R90"/>
 <instance part="C7" gate="G$1" x="43.18" y="114.3"/>
-<instance part="SUPPLY22" gate="+5V" x="76.2" y="63.5"/>
-<instance part="SUPPLY27" gate="+5V" x="67.31" y="177.8"/>
+<instance part="SUPPLY22" gate="G$1" x="76.2" y="63.5"/>
+<instance part="SUPPLY27" gate="G$1" x="67.31" y="177.8"/>
 <instance part="SUPPLY28" gate="GND" x="67.31" y="162.56"/>
 <instance part="SUPPLY6" gate="GND" x="-40.64" y="38.1"/>
 <instance part="C3" gate="G$1" x="-40.64" y="52.07"/>
 <instance part="C2" gate="G$1" x="-50.8" y="52.07"/>
-<instance part="SUPPLY5" gate="+5V" x="-40.64" y="60.96"/>
+<instance part="SUPPLY5" gate="G$1" x="-40.64" y="60.96"/>
 <instance part="X1" gate="G$1" x="53.34" y="170.18"/>
 <instance part="U4" gate="G$1" x="27.94" y="35.56"/>
@@
 <instance part="R5" gate="G$1" x="154.94" y="63.5" rot="R180"/>
 <instance part="SUPPLY2" gate="GND" x="162.56" y="58.42"/>
-<instance part="SUPPLY3" gate="+5V" x="132.08" y="68.58"/>
+<instance part="SUPPLY3" gate="G$1" x="132.08" y="68.58"/>
 <instance part="FRAME2" gate="G$1" x="-71.12" y="-5.08"/>
 <instance part="FRAME2" gate="G$2" x="101.6" y="-5.08"/>
@@
 <instance part="JP1" gate="A" x="-35.56" y="170.18"/>
 <instance part="SUPPLY4" gate="GND" x="-21.59" y="165.1"/>
-<instance part="SUPPLY7" gate="+5V" x="-52.07" y="162.56"/>
+<instance part="SUPPLY7" gate="G$1" x="-52.07" y="162.56"/>
 <instance part="X3" gate="-1" x="144.78" y="182.88"/>
 <instance part="X3" gate="-2" x="144.78" y="162.56"/>
-<instance part="SUPPLY8" gate="+5V" x="113.03" y="185.42"/>
+<instance part="SUPPLY8" gate="G$1" x="113.03" y="185.42"/>
 <instance part="R1" gate="G$1" x="124.46" y="182.88"/>
 <instance part="SUPPLY9" gate="GND" x="128.27" y="160.02"/>
@@
 </busses>
 <nets>
-<net name="+5V" class="0">
-<segment>
-<pinref part="SUPPLY34" gate="+5V" pin="+5V"/>
+<net name="+3.3V" class="0">
+<segment>
+<pinref part="SUPPLY34" gate="G$1" pin="+3V3"/>
 <wire x1="43.18" y1="116.84" x2="43.18" y2="119.38" width="0.1524" layer="91"/>
 <pinref part="C7" gate="G$1" pin="1"/>
@@
 </segment>
 <segment>
-<pinref part="SUPPLY22" gate="+5V" pin="+5V"/>
+<pinref part="SUPPLY22" gate="G$1" pin="+3V3"/>
 <pinref part="R2" gate="G$1" pin="2"/>
 <wire x1="76.2" y1="60.96" x2="76.2" y2="58.42" width="0.1524" layer="91"/>
 </segment>
 <segment>
-<pinref part="SUPPLY23" gate="+5V" pin="+5V"/>
+<pinref part="SUPPLY23" gate="G$1" pin="+3V3"/>
 <wire x1="68.58" y1="17.78" x2="83.82" y2="17.78" width="0.1524" layer="91"/>
 <pinref part="U4" gate="G$1" pin="AVCC"/>
 </segment>
 <segment>
-<pinref part="SUPPLY27" gate="+5V" pin="+5V"/>
+<pinref part="SUPPLY27" gate="G$1" pin="+3V3"/>
 <wire x1="63.5" y1="172.72" x2="67.31" y2="172.72" width="0.1524" layer="91"/>
 <wire x1="67.31" y1="172.72" x2="67.31" y2="175.26" width="0.1524" layer="91"/>
@@
 <segment>
 <pinref part="C2" gate="G$1" pin="1"/>
-<pinref part="SUPPLY5" gate="+5V" pin="+5V"/>
+<pinref part="SUPPLY5" gate="G$1" pin="+3V3"/>
 <wire x1="-50.8" y1="54.61" x2="-50.8" y2="58.42" width="0.1524" layer="91"/>
 <wire x1="-50.8" y1="58.42" x2="-40.64" y2="58.42" width="0.1524" layer="91"/>
@@
 <pinref part="D2" gate="G$1" pin="A"/>
 <wire x1="139.7" y1="63.5" x2="132.08" y2="63.5" width="0.1524" layer="91"/>
-<pinref part="SUPPLY3" gate="+5V" pin="+5V"/>
+<pinref part="SUPPLY3" gate="G$1" pin="+3V3"/>
 <wire x1="132.08" y1="66.04" x2="132.08" y2="63.5" width="0.1524" layer="91"/>
 </segment>
@@
 <pinref part="JP1" gate="A" pin="7"/>
 <wire x1="-38.1" y1="167.64" x2="-45.72" y2="167.64" width="0.1524" layer="91"/>
-<pinref part="SUPPLY7" gate="+5V" pin="+5V"/>
+<pinref part="SUPPLY7" gate="G$1" pin="+3V3"/>
 <wire x1="-45.72" y1="167.64" x2="-45.72" y2="160.02" width="0.1524" layer="91"/>
 <wire x1="-45.72" y1="160.02" x2="-52.07" y2="160.02" width="0.1524" layer="91"/>
@@
 <segment>
 <pinref part="R1" gate="G$1" pin="1"/>
-<pinref part="SUPPLY8" gate="+5V" pin="+5V"/>
+<pinref part="SUPPLY8" gate="G$1" pin="+3V3"/>
 <wire x1="119.38" y1="182.88" x2="113.03" y2="182.88" width="0.1524" layer="91"/>
 </segment>

Commit message: Add files via upload
revisions from day of design review
Parts:
- removed D1: Blue, SparkFun-LED:LED-YELLOW0603
- removed IC1: LDL1117S33R, LDL1117S33R:LDL1117S33R
- added C4: 0.1uF, rcl:C-USC0603
- added JP2: (no value), pinhead:PINHD-1X3
- added R10: 750, resistor:R-US_R0603
- added R9: 4.7k, resistor:R-US_R0603
- added U$1: TRANSISTOR, transistor:TRANSISTOR
- added U1: LD1086D2M33TR, transistor:LD1086D2M33TR
- added X4, X5: 1751248, con-phoenix-350:1751248
- C1: value 1uF -> 10uF; device rcl:C-USC0603 -> rcl:C-USC1206
- C7: value 4.7uF -> 10uF; device rcl:C-USC0603 -> rcl:C-USC1206
- R1, R3: value 300 -> 10k
Connections:
- removed net IN/OUT: D1.A, R1.2, U4.(PCINT0/CLKO/ICP1)_PB0, X3-1.K
- new net +3V3: D2.A
- new net IN: R1.2, R10.1, R9.2, U4.(PCINT0/CLKO/ICP1)_PB0, X3-1.K
- new net N$6: R9.1, X4-1.K
- new net N$7: JP2.3, U4.PC2_(ADC2/PCINT10)
- new net N$8: JP2.2, U4.PC3_(ADC3/PCINT11)
- new net N$9: C4.1, U4.AREF
- new net OUT: R3.1, U$1.G, U4.(PCINT1/OC1A)_PB1
- net +3.3V: now also U1.OUTPUT; no longer D2.A, IC1.VOUT(1), IC1.VOUT(2)
- net GND: now also C4.2, JP2.1, R10.2, U$1.S, U1.GROUND, X4-2.K; no longer IC1.GND
- net N$1: now also U$1.D, X5-2.K; no longer D1.C, R3.1
- net V_IN: now also U1.INPUT, X5-1.K; no longer IC1.VIN
Other:
- note added: "24V Button IN"
- note added: "24V OUT"
- note added: "3.3V Button IN"
- note added: "Import Symbol"
- note added: "LED"
- note removed: "In/Out"
- moved on the sheet: C1, C2, C3, C6, C7, D2, JP1, R1, R2, R3, R5, S3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

Commit message: board v1
Parts:
- added D1, D3: Green, SparkFun-LED:LED-YELLOW0603
- added R4, R6: 300, resistor:R-US_R0603
Connections:
- new net BUTTON_LED: D1.A, U4.(PCINT21/OC0B/T1)_PD5
- new net N$3: D1.C, R4.2
- new net N$4: D3.C, R6.2
- new net WIRELESS_LED: D3.A, U4.(PCINT22/OC0A/AIN0)_PD6
- net GND: now also R4.1, R6.1
Other:
- note added: "Button LED"
- note added: "Wireless LED"
Changed lines of the file:
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@@
 <?xml version="1.0" encoding="utf-8"?>
 <!DOCTYPE eagle SYSTEM "eagle.dtd">
-<eagle version="8.5.2">
+<eagle version="8.6.0">
 <drawing>
 <settings>
@@
 <part name="JP2" library="pinhead" library_urn="urn:adsk.eagle:library:325" deviceset="PINHD-1X3" device="" package3d_urn="urn:adsk.eagle:package:22458/2"/>
 <part name="R3" library="resistor" library_urn="urn:adsk.eagle:library:348" deviceset="R-US_" device="R0603" package3d_urn="urn:adsk.eagle:package:26057/1" value="10k"/>
+<part name="D3" library="SparkFun-LED" deviceset="LED-YELLOW" device="0603" value="Green"/>
+<part name="R6" library="resistor" library_urn="urn:adsk.eagle:library:348" deviceset="R-US_" device="R0603" package3d_urn="urn:adsk.eagle:package:26057/1" value="300"/>
+<part name="SUPPLY13" library="supply2" library_urn="urn:adsk.eagle:library:372" deviceset="GND" device=""/>
+<part name="D1" library="SparkFun-LED" deviceset="LED-YELLOW" device="0603" value="Green"/>
+<part name="R4" library="resistor" library_urn="urn:adsk.eagle:library:348" deviceset="R-US_" device="R0603" package3d_urn="urn:adsk.eagle:package:26057/1" value="300"/>
+<part name="SUPPLY1" library="supply2" library_urn="urn:adsk.eagle:library:372" deviceset="GND" device=""/>
 </parts>
 <sheets>
@@
 <text x="617.22" y="381" size="1.016" layer="103">Import Symbol</text>
 <text x="345.44" y="271.78" size="1.016" layer="103">LED</text>
+<wire x1="462.28" y1="254" x2="462.28" y2="215.9" width="0.1524" layer="103" style="shortdash"/>
+<wire x1="462.28" y1="215.9" x2="419.1" y2="215.9" width="0.1524" layer="103" style="shortdash"/>
+<wire x1="419.1" y1="215.9" x2="419.1" y2="254" width="0.1524" layer="103" style="shortdash"/>
+<wire x1="419.1" y1="254" x2="462.28" y2="254" width="0.1524" layer="103" style="shortdash"/>
+<text x="421.64" y="246.38" size="3.81" layer="103" font="vector">Button LED</text>
+<wire x1="510.54" y1="297.18" x2="510.54" y2="259.08" width="0.1524" layer="103" style="shortdash"/>
+<wire x1="510.54" y1="259.08" x2="467.36" y2="259.08" width="0.1524" layer="103" style="shortdash"/>
+<wire x1="467.36" y1="259.08" x2="467.36" y2="297.18" width="0.1524" layer="103" style="shortdash"/>
+<wire x1="467.36" y1="297.18" x2="510.54" y2="297.18" width="0.1524" layer="103" style="shortdash"/>
+<text x="469.9" y="289.56" size="3.81" layer="103" font="vector">Wireless LED</text>
 </plain>
 <instances>
@@
 <instance part="JP2" gate="A" x="403.86" y="251.46"/>
 <instance part="R3" gate="G$1" x="594.36" y="381" rot="R270"/>
+<instance part="D3" gate="G$1" x="487.68" y="276.86" smashed="yes" rot="MR0">
+<attribute name="NAME" x="494.792" y="275.209" size="1.778" layer="95" font="vector" rot="MR0"/>
+<attribute name="VALUE" x="485.775" y="272.288" size="1.778" layer="96" font="vector" rot="MR90" align="top-left"/>
+</instance>
+<instance part="R6" gate="G$1" x="497.84" y="269.24" rot="R180"/>
+<instance part="SUPPLY13" gate="GND" x="505.46" y="264.16"/>
+<instance part="D1" gate="G$1" x="439.42" y="233.68" smashed="yes" rot="MR0">
+<attribute name="NAME" x="446.532" y="232.029" size="1.778" layer="95" font="vector" rot="MR0"/>
+<attribute name="VALUE" x="437.515" y="229.108" size="1.778" layer="96" font="vector" rot="MR90" align="top-left"/>
+</instance>
+<instance part="R4" gate="G$1" x="449.58" y="226.06" rot="R180"/>
+<instance part="SUPPLY1" gate="GND" x="457.2" y="220.98"/>
 </instances>
 <busses>
@@
 <wire x1="603.25" y1="386.08" x2="609.6" y2="386.08" width="0.1524" layer="91"/>
 </segment>
+<segment>
+<pinref part="SUPPLY13" gate="GND" pin="GND"/>
+<pinref part="R6" gate="G$1" pin="1"/>
+<wire x1="505.46" y1="266.7" x2="505.46" y2="269.24" width="0.1524" layer="91"/>
+<wire x1="505.46" y1="269.24" x2="502.92" y2="269.24" width="0.1524" layer="91"/>
+</segment>
+<segment>
+<pinref part="SUPPLY1" gate="GND" pin="GND"/>
+<pinref part="R4" gate="G$1" pin="1"/>
+<wire x1="457.2" y1="223.52" x2="457.2" y2="226.06" width="0.1524" layer="91"/>
+<wire x1="457.2" y1="226.06" x2="454.66" y2="226.06" width="0.1524" layer="91"/>
+</segment>
 </net>
 <net name="MISO" class="0">
@@
 </segment>
 </net>
+<net name="BUTTON_LED" class="0">
+<segment>
+<pinref part="U4" gate="G$1" pin="(PCINT21/OC0B/T1)_PD5"/>
+<wire x1="309.88" y1="246.38" x2="304.8" y2="246.38" width="0.1524" layer="91"/>
+<label x="304.8" y="246.38" size="1.27" layer="95" rot="R180" xref="yes"/>
+</segment>
+<segment>
+<pinref part="D1" gate="G$1" pin="A"/>
+<wire x1="439.42" y1="236.22" x2="439.42" y2="238.76" width="0.1524" layer="91"/>
+<wire x1="439.42" y1="238.76" x2="436.88" y2="238.76" width="0.1524" layer="91"/>
+<label x="436.88" y="238.76" size="1.27" layer="95" rot="R180" xref="yes"/>
+</segment>
+</net>
+<net name="WIRELESS_LED" class="0">
+<segment>
+<pinref part="U4" gate="G$1" pin="(PCINT22/OC0A/AIN0)_PD6"/>
+<wire x1="309.88" y1="243.84" x2="304.8" y2="243.84" width="0.1524" layer="91"/>
+<label x="304.8" y="243.84" size="1.27" layer="95" rot="R180" xref="yes"/>
+</segment>
+<segment>
+<pinref part="D3" gate="G$1" pin="A"/>
+<wire x1="487.68" y1="279.4" x2="487.68" y2="281.94" width="0.1524" layer="91"/>
+<wire x1="487.68" y1="281.94" x2="485.14" y2="281.94" width="0.1524" layer="91"/>
+<label x="485.14" y="281.94" size="1.27" layer="95" rot="R180" xref="yes"/>
+</segment>
+</net>
+<net name="N$4" class="0">
+<segment>
+<pinref part="D3" gate="G$1" pin="C"/>
+<wire x1="487.68" y1="271.78" x2="487.68" y2="269.24" width="0.1524" layer="91"/>
+<pinref part="R6" gate="G$1" pin="2"/>
+<wire x1="487.68" y1="269.24" x2="492.76" y2="269.24" width="0.1524" layer="91"/>
+</segment>
+</net>
+<net name="N$3" class="0">
+<segment>
+<pinref part="D1" gate="G$1" pin="C"/>
+<wire x1="439.42" y1="228.6" x2="439.42" y2="226.06" width="0.1524" layer="91"/>
+<pinref part="R4" gate="G$1" pin="2"/>
+<wire x1="439.42" y1="226.06" x2="444.5" y2="226.06" width="0.1524" layer="91"/>
+</segment>
+</net>
