File: logic/Eagle Files/logic.sch (EAGLE design)
At the start: 67 parts, among them J1 Under Glow, J2 B2PS-VH(LF)(SN), J3 B2PS-VH(LF)(SN), J4 B2PS-VH(LF)(SN), J5 B2PS-VH(LF)(SN), J6 B2PS-VH(LF)(SN), Q4 STT4P3LLH6, Q5 RRH100P03GZETB, T1 R-78E5.0-1.0, U1 9DoF IMU, U4 TLV70233DBVR, U5 TC4427ACOA713, U6 TC4427ACOA713, U7 TC4427ACOA713, X1 MINI-USB_SHIELD5P4-32005-400, X2 C-GRID-05-15-91, X3 2510-, X4 2510-, X5 C-GRID-05-15-91, X6 C-GRID-02-70553, X7 SI-50170

Commit message: added more power and removed old circuits
Parts:
- removed J1: Under Glow, SparkFun-Connectors:CONN_12LOCK_LONGPADS
- removed J5: B2PS-VH(LF)(SN), RoboJackets-Connectors:B2PS-VH(LF)(SN)
- removed OK1, OK2: MOCD208M, optocoupler:MOCD208M
- removed Q5: RRH100P03GZETB, MotorBoardDev:RRH100P03GZETB
- removed R10, R5, R9: 30, rcl:R-US_R0603
- removed R12, R13, R6, R7: 4.7k, rcl:R-US_R0603
- removed R14, R15: 1k, rcl:R-US_R0603
- removed R26: 2.7k, rcl:R-US_R0603
- removed U5, U6, U7: TC4427ACOA713, MotorBoardDev:TC4427ACOA713
- removed X3, X4: 2510-, con-3m:2510-
- removed X6: C-GRID-02-70553, con-molex:C-GRID-02-70553
- added C13, C15, C17, C19: 0.1uF, rcl:C-USC0603
- added C14, C16: 1nF, rcl:C-USC0603
- added C18, C20: 10uF, rcl:C-USC0805
- added R3: 1k, rcl:R-US_R0603
- added U$19, U$22: ACS711, IGVC-Sensor:ACS711
- added U$20, U$21, U$24: FUSE_HOLDER, IGVC-Misc:FUSE_HOLDER
- added U$23: MIS29301-12, IGVC-Regulator:MIS29301-12
- added U$25: BUK9226, IGVC-Discrete:BUK9226
- added U$26, U$27, U$28: S10M-TP, IGVC-Discrete:S10M-TP
- R4: value 30 -> 1k
Connections:
- removed net BLUE_3V3: A1.P$16, U5.IN_B
- removed net BLUE_OUT: J1.1, U5.!OUT_B
- removed net FRONT_HDR: Q5.D, X6-1.S
- removed net FRONT_LIGHT: R26.1, U5.!OUT_A
- removed net FRONT_LIGHT_3V3: A1.P$17, U5.IN_A
- removed net FRONT_R: Q5.G, R26.2
- removed net GREEN_3V3: A1.P$15, U6.IN_A
- removed net GREEN_OUT: J1.2, U6.!OUT_A
- removed net L+12V: R12.2, R6.2, X3-1.KL, X3-2.KL, X3-5.KL, X3-7.KL
- removed net LALI: OK1A.COL, R6.1, X3-6.KL
- removed net LALI_CTRL: A1.P$21, R4.1
- removed net LBLI: OK1B.COL, R12.1, X3-8.KL
- removed net LBLI_CTRL: A1.P$22, R9.1
- removed net LDISABLE: R14.2, X3-4.KL
- removed net LGND: OK1A.EMIT, OK1B.EMIT, R14.1, X3-10.KL, X3-9.KL
- removed net R+12V: R13.2, R7.2, X4-1.KL, X4-2.KL, X4-5.KL, X4-7.KL
- removed net RALI: OK2A.COL, R7.1, X4-6.KL
- removed net RALI_CTRL: A1.P$23, R5.1
- removed net RBLI: OK2B.COL, R13.1, X4-8.KL
- removed net RBLI_CTRL: A1.P$24, R10.1
- removed net RDISABLE: R15.2, X4-4.KL
- removed net RED_3V3: A1.P$14, U6.IN_B
- removed net RED_OUT: J1.3, U6.!OUT_B
- removed net RGND: OK2A.EMIT, OK2B.EMIT, R15.1, X4-10.KL, X4-9.KL
- removed net R_OK3A: OK1A.A, R4.2
- removed net R_OK3B: OK1B.A, R9.2
- removed net R_OK4A: OK2A.A, R5.2
- removed net R_OK4B: OK2B.A, R10.2
- new net +12V_FAN: U$22.IP-
- new net +12V_FAN_CURRSENSE: U$22.IP+, U$24.2
- new net +12V_FAN_FUSE: C18.1, U$23.OUT, U$24.1
- new net +12V_SAFETY_FUSE: C20.1, U$18.OUT, U$20.1
- new net +24V_FLOOD_CURRSENSE: U$19.IP+, U$21.2
- new net +24V_FLOOD_FUSE: U$21.1, U$25.S
- new net +24V_FLOOD_LIGHT: U$19.IP-
- new net DIODE_TO_INTER: U$27.C
- new net DIODE_TO_RED: U$26.C
- new net FAN_EN: U$23.EN
- new net FAN_FLG: U$23.FLG
- new net FLOOD_LIGHT_EN: U$25.G
- new net N$5: C14.1, U$19.VIOUT
- new net N$6: R3.1, U$19.!FAULT
- new net N$7: C16.1, U$22.VIOUT
- new net N$8: R4.1, U$22.!FAULT
- new net SOLENOID_TO_DIODE: U$27.A
- new net SOLENOID_TRIG: U$28.C
- new net SOLENOID_TRIG_GND: U$28.A
- net +12V: no longer Q5.S, U5.VDD, U6.VDD, U7.VDD
- net +12V_SAFETY_CURRSENSE: now also U$20.2; no longer U$18.OUT
- net +24V: now also C17.1, C19.1, U$23.IN, U$25.D, U$26.A
- net +3V3: now also C13.1, C15.1, R3.2, R4.2, U$19.VCC, U$22.VCC
- net ESTOP: no longer J5.2
- net GND: now also C13.2, C14.2, C15.2, C16.2, C17.2, C18.2, C19.2, C20.2, U$19.GND, U$22.GND, U$23.GND; no longer J1.10, J1.11, J1.12, J1.4, J1.5, J1.6, J5.1, OK1A.C, OK1B.C, OK2A.C, OK2B.C, U5.GND, U6.GND, U7.GND, X6-2.S
- net SAFETY_LIGHT: no longer U7.!OUT_B
- net SAFETY_LIGHT_3V3: no longer U7.IN_B
Other:
- note added: "Fan Power Distribution"
- note added: "Flood Light Power"
- note added: "Fuses"
- note added: "Mast Connector: - DIODE_TO_RED - DIODE_TO_INTER - GREEN_TO_WIRELESS"
- note added: "Solenoid Connector: - SOLENOID_TRIG - ESTOP - +3V3"
- note removed: "#S#O control which bar lights up RGB control the color of the entire stripe"
- note removed: "Also LGND"
- note removed: "DO the rest"
- note removed: "Estop Stuatus"
- note removed: "Flood Light"
- note removed: "Gate driver"
- note removed: "If have space add Optoisolator for HI lines"
- note removed: "Input Current 200mA Voltage 5V \therefore R = 25Ω ish"
- note removed: "No we dont"
- note removed: "OSMC Headers"
- note removed: "Optoisolators"
- note removed: "Review the connection of DISABLE even tho it physically works"
- note removed: "Therefore #S#O control pin dont need to be PWM"
- note removed: "Third pin points to Battery voltage level, something we already have, see battery sensor/Status Light, so not using it"
- note removed: "Underglow"
- note removed: "Underglow Header"
- note removed: "mk it clear for datapin"

Commit message: added new imu
Parts:
- added C21, C22, C23: 0.1uF, rcl:C-USC0603
- added U2: ICM-20948, ICM-20948:ICM-20948
Connections:
- new net +1V8: C22.1, U2.NCS, U2.VDDIO
- new net IMU_INT: A1.P$11, U2.INT1
- new net N$9: C23.1, U2.REGOUT
- net +3V3: now also C21.1, U2.VDD
- net GND: now also C21.2, C22.2, C23.2, U2.AD0/SDO, U2.EXP_PAD, U2.FSYNC, U2.GND, U2.RESV_20
- net GYRO_INT: no longer A1.P$11
- net SCL: now also U2.SCL/SCLK
- net SDA: now also U2.SDA/SDI

Commit message: removed imu
Parts:
- removed C21, C22, C23: 0.1uF, rcl:C-USC0603
- removed U2: ICM-20948, ICM-20948:ICM-20948
Connections:
- removed net +1V8: C22.1, U2.NCS, U2.VDDIO
- removed net N$9: C23.1, U2.REGOUT
- net +3V3: no longer C21.1, U2.VDD
- net GND: no longer C21.2, C22.2, C23.2, U2.AD0/SDO, U2.EXP_PAD, U2.FSYNC, U2.GND, U2.RESV_20
- net IMU_INT: no longer U2.INT1
- net SCL: no longer U2.SCL/SCLK
- net SDA: no longer U2.SDA/SDI
Changed lines of the file:
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@@
 <part name="U$28" library="IGVC-Discrete" deviceset="S10M-TP" device=""/>
 <part name="P+20" library="supply1" library_urn="urn:adsk.eagle:library:371" deviceset="+24V" device=""/>
-<part name="FRAME8" library="RoboJackets-Frames" deviceset="FRAME_A_L" device=""/>
-<part name="U2" library="ICM-20948" deviceset="ICM-20948" device=""/>
-<part name="GND13" library="supply1" library_urn="urn:adsk.eagle:library:371" deviceset="GND" device=""/>
-<part name="+3V4" library="supply1" library_urn="urn:adsk.eagle:library:371" deviceset="+3V3" device="" value="+1V8"/>
-<part name="C21" library="rcl" library_urn="urn:adsk.eagle:library:334" deviceset="C-US" device="C0603" package3d_urn="urn:adsk.eagle:package:23616/2" value="0.1uF"/>
-<part name="C22" library="rcl" library_urn="urn:adsk.eagle:library:334" deviceset="C-US" device="C0603" package3d_urn="urn:adsk.eagle:package:23616/2" value="0.1uF"/>
-<part name="GND14" library="supply1" library_urn="urn:adsk.eagle:library:371" deviceset="GND" device=""/>
-<part name="GND22" library="supply1" library_urn="urn:adsk.eagle:library:371" deviceset="GND" device=""/>
-<part name="+3V5" library="supply1" library_urn="urn:adsk.eagle:library:371" deviceset="+3V3" device=""/>
-<part name="+3V6" library="supply1" library_urn="urn:adsk.eagle:library:371" deviceset="+3V3" device="" value="+1V8"/>
-<part name="C23" library="rcl" library_urn="urn:adsk.eagle:library:334" deviceset="C-US" device="C0603" package3d_urn="urn:adsk.eagle:package:23616/2" value="0.1uF"/>
-<part name="GND27" library="supply1" library_urn="urn:adsk.eagle:library:371" deviceset="GND" device=""/>
-<part name="GND31" library="supply1" library_urn="urn:adsk.eagle:library:371" deviceset="GND" device=""/>
 </parts>
 <sheets>
@@
 </segment>
 </net>
-</nets>
-</sheet>
-<sheet>
-<description>Sensors</description>
-<plain>
-<wire x1="7.62" y1="208.28" x2="109.22" y2="208.28" width="0.1524" layer="97" style="longdash"/>
-<wire x1="109.22" y1="208.28" x2="109.22" y2="127" width="0.1524" layer="97" style="longdash"/>
-<wire x1="109.22" y1="127" x2="7.62" y2="127" width="0.1524" layer="97" style="longdash"/>
-<wire x1="7.62" y1="127" x2="7.62" y2="208.28" width="0.1524" layer="97" style="longdash"/>
-<text x="101.6" y="129.54" size="1.778" layer="97" font="vector">IMU</text>
-</plain>
-<instances>
-<instance part="FRAME8" gate="G$1" x="0" y="0"/>
-<instance part="FRAME8" gate="G$2" x="172.72" y="0">
-<attribute name="LAST_DATE_TIME" x="185.42" y="1.27" size="2.54" layer="94" font="vector"/>
-<attribute name="SHEET" x="259.08" y="1.27" size="2.54" layer="94" font="vector"/>
-<attribute name="DRAWING_NAME" x="187.96" y="19.05" size="2.54" layer="94" font="vector"/>
-<attribute name="TEAM" x="173.99" y="34.29" size="3.048" layer="94" ratio="10" align="top-left"/>
-<attribute name="REVISION" x="245.11" y="6.35" size="2.54" layer="94"/>
-<attribute name="SCH_DESC" x="173.99" y="6.35" size="2.54" layer="94"/>
-</instance>
-<instance part="U2" gate="G$1" x="48.26" y="162.56">
-<attribute name="NAME" x="32.9945" y="180.8786" size="1.78096875" layer="95"/>
-<attribute name="VALUE" x="32.9985" y="142.2113" size="1.780509375" layer="96"/>
-</instance>
-<instance part="GND13" gate="1" x="22.86" y="144.78">
-<attribute name="VALUE" x="20.32" y="142.24" size="1.778" layer="96"/>
-</instance>
-<instance part="+3V4" gate="G$1" x="20.32" y="177.8">
-<attribute name="VALUE" x="17.78" y="172.72" size="1.778" layer="96" rot="R90"/>
-</instance>
-<instance part="C21" gate="G$1" x="93.98" y="187.96">
-<attribute name="NAME" x="94.996" y="188.595" size="1.778" layer="95"/>
-<attribute name="VALUE" x="94.996" y="183.769" size="1.778" layer="96"/>
-</instance>
-<instance part="C22" gate="G$1" x="83.82" y="187.96">
-<attribute name="NAME" x="84.836" y="188.595" size="1.778" layer="95"/>
-<attribute name="VALUE" x="84.836" y="183.769" size="1.778" layer="96"/>
-</instance>
-<instance part="GND14" gate="1" x="83.82" y="177.8">
-<attribute name="VALUE" x="81.28" y="175.26" size="1.778" layer="96"/>
-</instance>
-<instance part="GND22" gate="1" x="93.98" y="177.8">
-<attribute name="VALUE" x="91.44" y="175.26" size="1.778" layer="96"/>
-</instance>
-<instance part="+3V5" gate="G$1" x="71.12" y="200.66">
-<attribute name="VALUE" x="68.58" y="195.58" size="1.778" layer="96" rot="R90"/>
-</instance>
-<instance part="+3V6" gate="G$1" x="76.2" y="200.66">
-<attribute name="VALUE" x="78.74" y="200.66" size="1.778" layer="96" rot="R90"/>
-</instance>
-<instance part="C23" gate="G$1" x="96.52" y="154.94">
-<attribute name="NAME" x="97.536" y="155.575" size="1.778" layer="95"/>
-<attribute name="VALUE" x="97.536" y="150.749" size="1.778" layer="96"/>
-</instance>
-<instance part="GND27" gate="1" x="96.52" y="144.78">
-<attribute name="VALUE" x="93.98" y="142.24" size="1.778" layer="96"/>
-</instance>
-<instance part="GND31" gate="1" x="88.9" y="144.78">
-<attribute name="VALUE" x="86.36" y="142.24" size="1.778" layer="96"/>
-</instance>
-</instances>
-<busses>
-</busses>
-<nets>
-<net name="SCL" class="0">
-<segment>
-<pinref part="U2" gate="G$1" pin="SCL/SCLK"/>
-<wire x1="27.94" y1="162.56" x2="12.7" y2="162.56" width="0.1524" layer="91"/>
-<label x="12.7" y="162.56" size="1.778" layer="95"/>
-</segment>
-</net>
-<net name="SDA" class="0">
-<segment>
-<pinref part="U2" gate="G$1" pin="SDA/SDI"/>
-<wire x1="27.94" y1="157.48" x2="12.7" y2="157.48" width="0.1524" layer="91"/>
-<label x="12.7" y="157.48" size="1.778" layer="95"/>
-</segment>
-</net>
-<net name="GND" class="0">
-<segment>
-<pinref part="U2" gate="G$1" pin="AD0/SDO"/>
-<pinref part="GND13" gate="1" pin="GND"/>
-<wire x1="27.94" y1="160.02" x2="22.86" y2="160.02" width="0.1524" layer="91"/>
-<wire x1="22.86" y1="160.02" x2="22.86" y2="147.32" width="0.1524" layer="91"/>
-<pinref part="U2" gate="G$1" pin="FSYNC"/>
-<wire x1="27.94" y1="170.18" x2="22.86" y2="170.18" width="0.1524" layer="91"/>
-<junction x="22.86" y="160.02"/>
-<wire x1="22.86" y1="170.18" x2="22.86" y2="160.02" width="0.1524" layer="91"/>
-</segment>
-<segment>
-<pinref part="C22" gate="G$1" pin="2"/>
-<pinref part="GND14" gate="1" pin="GND"/>
-<wire x1="83.82" y1="182.88" x2="83.82" y2="180.34" width="0.1524" layer="91"/>
-</segment>
-<segment>
-<pinref part="C21" gate="G$1" pin="2"/>
-<pinref part="GND22" gate="1" pin="GND"/>
-<wire x1="93.98" y1="182.88" x2="93.98" y2="180.34" width="0.1524" layer="91"/>
-</segment>
-<segment>
-<pinref part="C23" gate="G$1" pin="2"/>
-<pinref part="GND27" gate="1" pin="GND"/>
-<wire x1="96.52" y1="149.86" x2="96.52" y2="147.32" width="0.1524" layer="91"/>
-</segment>
-<segment>
-<pinref part="U2" gate="G$1" pin="RESV_20"/>
-<pinref part="GND31" gate="1" pin="GND"/>
-<wire x1="68.58" y1="154.94" x2="88.9" y2="154.94" width="0.1524" layer="91"/>
-<wire x1="88.9" y1="154.94" x2="88.9" y2="149.86" width="0.1524" layer="91"/>
-<pinref part="U2" gate="G$1" pin="GND"/>
-<wire x1="88.9" y1="149.86" x2="88.9" y2="147.32" width="0.1524" layer="91"/>
-<wire x1="68.58" y1="149.86" x2="71.12" y2="149.86" width="0.1524" layer="91"/>
-<junction x="88.9" y="149.86"/>
-<pinref part="U2" gate="G$1" pin="EXP_PAD"/>
-<wire x1="71.12" y1="149.86" x2="88.9" y2="149.86" width="0.1524" layer="91"/>
-<wire x1="68.58" y1="147.32" x2="71.12" y2="147.32" width="0.1524" layer="91"/>
-<wire x1="71.12" y1="147.32" x2="71.12" y2="149.86" width="0.1524" layer="91"/>
-<junction x="71.12" y="149.86"/>
-</segment>
-</net>
-<net name="+1V8" class="0">
-<segment>
-<pinref part="U2" gate="G$1" pin="NCS"/>
-<pinref part="+3V4" gate="G$1" pin="+3V3"/>
-<wire x1="27.94" y1="154.94" x2="20.32" y2="154.94" width="0.1524" layer="91"/>
-<wire x1="20.32" y1="154.94" x2="20.32" y2="175.26" width="0.1524" layer="91"/>
-</segment>
-<segment>
-<wire x1="76.2" y1="175.26" x2="76.2" y2="193.04" width="0.1524" layer="91"/>
-<pinref part="C22" gate="G$1" pin="1"/>
-<wire x1="76.2" y1="193.04" x2="76.2" y2="198.12" width="0.1524" layer="91"/>
-<wire x1="83.82" y1="190.5" x2="83.82" y2="193.04" width="0.1524" layer="91"/>
-<wire x1="83.82" y1="193.04" x2="76.2" y2="193.04" width="0.1524" layer="91"/>
-<junction x="76.2" y="193.04"/>
-<pinref part="+3V6" gate="G$1" pin="+3V3"/>
-<pinref part="U2" gate="G$1" pin="VDDIO"/>
-<wire x1="68.58" y1="175.26" x2="76.2" y2="175.26" width="0.1524" layer="91"/>
-</segment>
-</net>
-<net name="+3V3" class="0">
-<segment>
-<wire x1="71.12" y1="177.8" x2="71.12" y2="195.58" width="0.1524" layer="91"/>
-<pinref part="C21" gate="G$1" pin="1"/>
-<wire x1="71.12" y1="195.58" x2="71.12" y2="198.12" width="0.1524" layer="91"/>
-<wire x1="93.98" y1="190.5" x2="93.98" y2="195.58" width="0.1524" layer="91"/>
-<wire x1="93.98" y1="195.58" x2="71.12" y2="195.58" width="0.1524" layer="91"/>
-<junction x="71.12" y="195.58"/>
-<pinref part="+3V5" gate="G$1" pin="+3V3"/>
-<pinref part="U2" gate="G$1" pin="VDD"/>
-<wire x1="68.58" y1="177.8" x2="71.12" y2="177.8" width="0.1524" layer="91"/>
-</segment>
-</net>
-<net name="IMU_INT" class="0">
-<segment>
-<pinref part="U2" gate="G$1" pin="INT1"/>
-<wire x1="68.58" y1="167.64" x2="83.82" y2="167.64" width="0.1524" layer="91"/>
-<label x="78.74" y="167.64" size="1.778" layer="95"/>
-</segment>
-</net>
-<net name="N$9" class="0">
-<segment>
-<pinref part="U2" gate="G$1" pin="REGOUT"/>
-<wire x1="68.58" y1="162.56" x2="96.52" y2="162.56" width="0.1524" layer="91"/>
-<pinref part="C23" gate="G$1" pin="1"/>
-<wire x1="96.52" y1="162.56" x2="96.52" y2="157.48" width="0.1524" layer="91"/>
-</segment>
-</net>
