File: hotswap.sch (EAGLE design)
At the start: 10 parts, among them U1 LTC4416EMS#PBF, U2 641737-1, U3 641737-1, U4 641737-1

Commit message: Hotswap Design Review (Asha)
Parts:
- U2: value 641737-1 -> WALL
- U3: value 641737-1 -> BATTERY
- U4: value 641737-1 -> COMPUTER
Other:
- note added: "IGVC"
Changed lines of the file:
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@@
 <part name="VCC_BATT" library="supply1" library_urn="urn:adsk.eagle:library:371" deviceset="VCC" device="" value="VCC_BATT"/>
 <part name="VCC_WALL" library="supply1" library_urn="urn:adsk.eagle:library:371" deviceset="VCC" device="" value="VCC_WALL"/>
-<part name="U2" library="IGVC-Connector" deviceset="641737-1" device=""/>
+<part name="U2" library="IGVC-Connector" deviceset="641737-1" device="" value="WALL"/>
 <part name="VCC_COMP" library="supply1" library_urn="urn:adsk.eagle:library:371" deviceset="VCC" device="" value="VCC_COMP"/>
 <part name="GND2" library="supply1" library_urn="urn:adsk.eagle:library:371" deviceset="GND" device=""/>
-<part name="GND3" library="supply1" library_urn="urn:adsk.eagle:library:371" deviceset="GND" device=""/>
-<part name="U3" library="IGVC-Connector" deviceset="641737-1" device=""/>
-<part name="U4" library="IGVC-Connector" deviceset="641737-1" device=""/>
+<part name="U3" library="IGVC-Connector" deviceset="641737-1" device="" value="BATTERY"/>
+<part name="U4" library="IGVC-Connector" deviceset="641737-1" device="" value="COMPUTER"/>
 <part name="GND4" library="supply1" library_urn="urn:adsk.eagle:library:371" deviceset="GND" device=""/>
-<part name="GND5" library="supply1" library_urn="urn:adsk.eagle:library:371" deviceset="GND" device=""/>
 <part name="GND6" library="supply1" library_urn="urn:adsk.eagle:library:371" deviceset="GND" device=""/>
-<part name="GND7" library="supply1" library_urn="urn:adsk.eagle:library:371" deviceset="GND" device=""/>
+<part name="FRAME1" library="RoboJackets-Frames" deviceset="FRAME_A_L" device=""/>
 </parts>
 <sheets>
 <sheet>
 <plain>
+<text x="142.24" y="-40.64" size="1.778" layer="91">IGVC</text>
 </plain>
 <instances>
@@
 </instance>
 <instance part="U$3" gate="G$1" x="106.68" y="55.88" smashed="yes" rot="R90">
-<attribute name="NAME" x="104.14" y="62.23" size="1.778" layer="95" rot="R90"/>
-<attribute name="VALUE" x="106.68" y="62.23" size="1.778" layer="96" rot="R90"/>
+<attribute name="NAME" x="102.87" y="60.96" size="1.778" layer="95" rot="R180"/>
+<attribute name="VALUE" x="118.11" y="63.5" size="1.778" layer="96" rot="R180"/>
 </instance>
 <instance part="U$5" gate="G$1" x="93.98" y="15.24" smashed="yes" rot="R270">
-<attribute name="NAME" x="96.52" y="8.89" size="1.778" layer="95" rot="R270"/>
-<attribute name="VALUE" x="93.98" y="8.89" size="1.778" layer="96" rot="R270"/>
+<attribute name="NAME" x="90.17" y="17.78" size="1.778" layer="95"/>
+<attribute name="VALUE" x="87.63" y="7.62" size="1.778" layer="96"/>
 </instance>
 <instance part="R2E" gate="G$1" x="15.24" y="40.64" smashed="yes" rot="R90">
@@
 </instance>
 <instance part="U$4" gate="G$1" x="111.76" y="12.7" smashed="yes" rot="R180">
-<attribute name="NAME" x="105.41" y="10.16" size="1.778" layer="95" rot="R180"/>
-<attribute name="VALUE" x="105.41" y="12.7" size="1.778" layer="96" rot="R180"/>
+<attribute name="NAME" x="105.41" y="15.24" size="1.778" layer="95" rot="R180"/>
+<attribute name="VALUE" x="128.27" y="7.62" size="1.778" layer="96" rot="R180"/>
 </instance>
 <instance part="VCC_BATT" gate="VCC" x="55.88" y="12.7" smashed="yes" rot="R90">
-<attribute name="VALUE" x="58.42" y="10.16" size="1.778" layer="96" rot="R180"/>
+<attribute name="VALUE" x="55.88" y="10.16" size="1.778" layer="96" rot="R180"/>
 </instance>
 <instance part="VCC_WALL" gate="VCC" x="-5.08" y="58.42" smashed="yes" rot="R90">
@@
 </instance>
 <instance part="VCC_COMP" gate="VCC" x="134.62" y="33.02" smashed="yes" rot="R270">
-<attribute name="VALUE" x="132.08" y="35.56" size="1.778" layer="96"/>
+<attribute name="VALUE" x="134.62" y="38.1" size="1.778" layer="96"/>
 </instance>
 <instance part="GND2" gate="1" x="48.26" y="63.5" smashed="yes">
 <attribute name="VALUE" x="45.72" y="60.96" size="1.778" layer="96"/>
 </instance>
-<instance part="GND3" gate="1" x="55.88" y="63.5" smashed="yes">
-<attribute name="VALUE" x="53.34" y="60.96" size="1.778" layer="96"/>
-</instance>
 <instance part="U3" gate="A" x="58.42" y="0" smashed="yes">
 <attribute name="NAME" x="76.5556" y="9.1186" size="2.0828" layer="95" ratio="6" rot="SR0"/>
-<attribute name="VALUE" x="75.9206" y="6.5786" size="2.0828" layer="96" ratio="6" rot="SR0"/>
+<attribute name="VALUE" x="70.8406" y="6.5786" size="2.0828" layer="96" ratio="6" rot="SR0"/>
 </instance>
 <instance part="U4" gate="A" x="127" y="25.4" smashed="yes">
 <attribute name="NAME" x="145.1356" y="34.5186" size="2.0828" layer="95" ratio="6" rot="SR0"/>
-<attribute name="VALUE" x="144.5006" y="31.9786" size="2.0828" layer="96" ratio="6" rot="SR0"/>
+<attribute name="VALUE" x="139.4206" y="31.9786" size="2.0828" layer="96" ratio="6" rot="SR0"/>
 </instance>
 <instance part="GND4" gate="1" x="182.88" y="17.78" smashed="yes">
 <attribute name="VALUE" x="180.34" y="15.24" size="1.778" layer="96"/>
 </instance>
-<instance part="GND5" gate="1" x="187.96" y="17.78" smashed="yes">
-<attribute name="VALUE" x="185.42" y="15.24" size="1.778" layer="96"/>
-</instance>
 <instance part="GND6" gate="1" x="109.22" y="-7.62" smashed="yes">
 <attribute name="VALUE" x="106.68" y="-10.16" size="1.778" layer="96"/>
 </instance>
-<instance part="GND7" gate="1" x="114.3" y="-7.62" smashed="yes">
-<attribute name="VALUE" x="111.76" y="-10.16" size="1.778" layer="96"/>
+<instance part="FRAME1" gate="G$1" x="-48.26" y="-71.12" smashed="yes"/>
+<instance part="FRAME1" gate="G$2" x="124.46" y="-71.12" smashed="yes">
+<attribute name="LAST_DATE_TIME" x="137.16" y="-69.85" size="2.54" layer="94" font="vector"/>
+<attribute name="SHEET" x="210.82" y="-69.85" size="2.54" layer="94" font="vector"/>
+<attribute name="DRAWING_NAME" x="139.7" y="-52.07" size="2.54" layer="94" font="vector"/>
 </instance>
 </instances>
@@
 </segment>
 <segment>
+<pinref part="U2" gate="A" pin="4"/>
+<pinref part="GND2" gate="1" pin="GND"/>
+<wire x1="43.18" y1="71.12" x2="48.26" y2="71.12" width="0.1524" layer="91"/>
+<wire x1="48.26" y1="71.12" x2="48.26" y2="68.58" width="0.1524" layer="91"/>
 <pinref part="U2" gate="A" pin="3"/>
+<wire x1="48.26" y1="68.58" x2="48.26" y2="66.04" width="0.1524" layer="91"/>
 <wire x1="43.18" y1="68.58" x2="48.26" y2="68.58" width="0.1524" layer="91"/>
-<wire x1="48.26" y1="68.58" x2="48.26" y2="66.04" width="0.1524" layer="91"/>
-<pinref part="GND2" gate="1" pin="GND"/>
+<junction x="48.26" y="68.58"/>
 </segment>
 <segment>
-<pinref part="U2" gate="A" pin="4"/>
-<wire x1="43.18" y1="71.12" x2="55.88" y2="71.12" width="0.1524" layer="91"/>
-<wire x1="55.88" y1="71.12" x2="55.88" y2="66.04" width="0.1524" layer="91"/>
-<pinref part="GND3" gate="1" pin="GND"/>
+<pinref part="U3" gate="A" pin="4"/>
+<pinref part="GND6" gate="1" pin="GND"/>
+<wire x1="101.6" y1="0" x2="109.22" y2="0" width="0.1524" layer="91"/>
+<wire x1="109.22" y1="0" x2="109.22" y2="-2.54" width="0.1524" layer="91"/>
+<pinref part="U3" gate="A" pin="3"/>
+<wire x1="109.22" y1="-2.54" x2="109.22" y2="-5.08" width="0.1524" layer="91"/>
+<wire x1="101.6" y1="-2.54" x2="109.22" y2="-2.54" width="0.1524" layer="91"/>
+<junction x="109.22" y="-2.54"/>
 </segment>
 <segment>
 <pinref part="U4" gate="A" pin="3"/>
+<pinref part="GND4" gate="1" pin="GND"/>
 <wire x1="170.18" y1="22.86" x2="182.88" y2="22.86" width="0.1524" layer="91"/>
 <wire x1="182.88" y1="22.86" x2="182.88" y2="20.32" width="0.1524" layer="91"/>
-<pinref part="GND4" gate="1" pin="GND"/>
-</segment>
-<segment>
 <pinref part="U4" gate="A" pin="4"/>
-<wire x1="170.18" y1="25.4" x2="187.96" y2="25.4" width="0.1524" layer="91"/>
-<wire x1="187.96" y1="25.4" x2="187.96" y2="20.32" width="0.1524" layer="91"/>
-<pinref part="GND5" gate="1" pin="GND"/>
-</segment>
-<segment>
-<pinref part="U3" gate="A" pin="3"/>
-<wire x1="101.6" y1="-2.54" x2="109.22" y2="-2.54" width="0.1524" layer="91"/>
-<wire x1="109.22" y1="-2.54" x2="109.22" y2="-5.08" width="0.1524" layer="91"/>
-<pinref part="GND6" gate="1" pin="GND"/>
-</segment>
-<segment>
-<pinref part="U3" gate="A" pin="4"/>
-<wire x1="101.6" y1="0" x2="114.3" y2="0" width="0.1524" layer="91"/>
-<wire x1="114.3" y1="0" x2="114.3" y2="-5.08" width="0.1524" layer="91"/>
-<pinref part="GND7" gate="1" pin="GND"/>
+<wire x1="170.18" y1="25.4" x2="182.88" y2="25.4" width="0.1524" layer="91"/>
+<wire x1="182.88" y1="25.4" x2="182.88" y2="20.32" width="0.1524" layer="91"/>
+<junction x="182.88" y="20.32"/>
 </segment>
 </net>
