File: Diagnostic/eagle/Diagnostic.sch (EAGLE design)
At the start: 67 parts, among them J1 S7036-ND, J2 S7036-ND, J3 1175-1864-ND, J4 503182-1852, J5 277-1578-ND, Q1 16 MHz, Q2 16MHz, T2 LD1086D2M33TR, U1 ATMEGA2560AU, U2 BME280, U3 ATMEGA328P-AUR, U4 TXB0108PWR, U5 TPS565208DDCR, U6 TXB0108PWR, X1 B6B-EH-A(LF)(SN), X2 1751248, X3 NRF24L01, X5 1751248

Commit message: Started on the board
Parts:
- removed X2: 1751248, con-phoenix-350:1751248
Connections:
- removed net N$5: C10.1, C17.1, C26.1, U5.EN, U5.VIN, X5-1.K
- removed net V_IN: C16.1, T2.INPUT, X2-1.K
- net +12V: now also C10.1, C17.1, C26.1, U5.EN, U5.VIN, X5-1.K
- net +5V: now also C16.1, T2.INPUT
- net GND: no longer X2-2.K
Other:
- note added: "Bottom of Logic"
Changed lines of the file:
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@@
 <layers>
 <layer number="1" name="Top" color="4" fill="1" visible="no" active="no"/>
-<layer number="2" name="Route2" color="1" fill="3" visible="no" active="no"/>
-<layer number="3" name="Route3" color="4" fill="3" visible="no" active="no"/>
-<layer number="4" name="Route4" color="1" fill="4" visible="no" active="no"/>
-<layer number="5" name="Route5" color="4" fill="4" visible="no" active="no"/>
-<layer number="6" name="Route6" color="1" fill="8" visible="no" active="no"/>
-<layer number="7" name="Route7" color="4" fill="8" visible="no" active="no"/>
-<layer number="8" name="Route8" color="1" fill="2" visible="no" active="no"/>
-<layer number="9" name="Route9" color="4" fill="2" visible="no" active="no"/>
-<layer number="10" name="Route10" color="1" fill="7" visible="no" active="no"/>
-<layer number="11" name="Route11" color="4" fill="7" visible="no" active="no"/>
-<layer number="12" name="Route12" color="1" fill="5" visible="no" active="no"/>
-<layer number="13" name="Route13" color="4" fill="5" visible="no" active="no"/>
-<layer number="14" name="Route14" color="1" fill="6" visible="no" active="no"/>
-<layer number="15" name="Route15" color="4" fill="6" visible="no" active="no"/>
+<layer number="2" name="Route2" color="16" fill="1" visible="no" active="no"/>
+<layer number="3" name="Route3" color="17" fill="1" visible="no" active="no"/>
+<layer number="4" name="Route4" color="18" fill="1" visible="no" active="no"/>
+<layer number="5" name="Route5" color="19" fill="1" visible="no" active="no"/>
+<layer number="6" name="Route6" color="25" fill="1" visible="no" active="no"/>
+<layer number="7" name="Route7" color="26" fill="1" visible="no" active="no"/>
+<layer number="8" name="Route8" color="27" fill="1" visible="no" active="no"/>
+<layer number="9" name="Route9" color="28" fill="1" visible="no" active="no"/>
+<layer number="10" name="Route10" color="29" fill="1" visible="no" active="no"/>
+<layer number="11" name="Route11" color="30" fill="1" visible="no" active="no"/>
+<layer number="12" name="Route12" color="20" fill="1" visible="no" active="no"/>
+<layer number="13" name="Route13" color="21" fill="1" visible="no" active="no"/>
+<layer number="14" name="Route14" color="22" fill="1" visible="no" active="no"/>
+<layer number="15" name="Route15" color="23" fill="1" visible="no" active="no"/>
 <layer number="16" name="Bottom" color="1" fill="1" visible="no" active="no"/>
 <layer number="17" name="Pads" color="2" fill="1" visible="no" active="no"/>
 <layer number="18" name="Vias" color="2" fill="1" visible="no" active="no"/>
 <layer number="19" name="Unrouted" color="6" fill="1" visible="no" active="no"/>
-<layer number="20" name="Dimension" color="15" fill="1" visible="no" active="no"/>
+<layer number="20" name="Dimension" color="24" fill="1" visible="no" active="no"/>
 <layer number="21" name="tPlace" color="7" fill="1" visible="no" active="no"/>
 <layer number="22" name="bPlace" color="7" fill="1" visible="no" active="no"/>
@@
 <part name="GND24" library="supply1" library_urn="urn:adsk.eagle:library:371" deviceset="GND" device=""/>
 <part name="C15" library="rcl" library_urn="urn:adsk.eagle:library:334" deviceset="C-US" device="C1206" package3d_urn="urn:adsk.eagle:package:23618/2" value="10uF"/>
-<part name="X2" library="con-phoenix-350" library_urn="urn:adsk.eagle:library:174" deviceset="1751248" device="" package3d_urn="urn:adsk.eagle:package:9395/1"/>
 <part name="C16" library="rcl" library_urn="urn:adsk.eagle:library:334" deviceset="C-US" device="C1206" package3d_urn="urn:adsk.eagle:package:23618/2" value="10uF"/>
 <part name="T2" library="transistor" deviceset="LD1086D2M33TR" device=""/>
@@
 <part name="P+12" library="supply1" library_urn="urn:adsk.eagle:library:371" deviceset="+5V" device="" value="+5V"/>
 <part name="X3" library="IGVC-Connector" deviceset="NRF24L01+PA+LNA" device="" package3d_urn="urn:adsk.eagle:package:22461/2" value="NRF24L01"/>
+<part name="P+15" library="supply1" library_urn="urn:adsk.eagle:library:371" deviceset="+5V" device="" value="+5V"/>
 </parts>
 <sheets>
@@
 <text x="246.38" y="121.92" size="1.778" layer="97">+12V</text>
 <text x="162.56" y="66.04" size="1.778" layer="97">GND</text>
-<text x="246.38" y="114.3" size="1.778" layer="97">GND</text>
+<text x="119.38" y="91.44" size="1.778" layer="97">Bottom of Logic</text>
 </plain>
 <instances>
@@
 <attribute name="NAME" x="163.576" y="114.935" size="1.778" layer="95"/>
 <attribute name="VALUE" x="163.576" y="110.109" size="1.778" layer="96"/>
-</instance>
-<instance part="X2" gate="-1" x="238.76" y="119.38" smashed="yes">
-<attribute name="NAME" x="240.03" y="118.491" size="1.778" layer="95"/>
-<attribute name="VALUE" x="252.73" y="118.491" size="1.778" layer="96"/>
-</instance>
-<instance part="X2" gate="-2" x="238.76" y="111.76" smashed="yes">
-<attribute name="NAME" x="240.03" y="110.871" size="1.778" layer="95"/>
-<attribute name="VALUE" x="252.73" y="110.871" size="1.778" layer="96"/>
 </instance>
 <instance part="C16" gate="G$1" x="228.6" y="116.84" smashed="yes">
@@
 <attribute name="NAME" x="113.03" y="198.755" size="1.778" layer="95"/>
 <attribute name="VALUE" x="105.41" y="182.88" size="1.778" layer="96"/>
+</instance>
+<instance part="P+15" gate="1" x="236.22" y="121.92" smashed="yes">
+<attribute name="VALUE" x="238.76" y="124.46" size="1.778" layer="96" rot="R180"/>
 </instance>
 </instances>
@@
 <pinref part="P+12" gate="1" pin="+5V"/>
 </segment>
+<segment>
+<wire x1="236.22" y1="119.38" x2="228.6" y2="119.38" width="0.1524" layer="91"/>
+<pinref part="C16" gate="G$1" pin="1"/>
+<wire x1="220.98" y1="119.38" x2="228.6" y2="119.38" width="0.1524" layer="91"/>
+<junction x="228.6" y="119.38"/>
+<pinref part="T2" gate="A" pin="INPUT"/>
+<pinref part="P+15" gate="1" pin="+5V"/>
+</segment>
 </net>
 <net name="GND" class="0">
@@
 <wire x1="162.56" y1="104.14" x2="162.56" y2="101.6" width="0.1524" layer="91"/>
 <junction x="162.56" y="104.14"/>
-<pinref part="X2" gate="-2" pin="K"/>
 <wire x1="172.72" y1="104.14" x2="162.56" y2="104.14" width="0.1524" layer="91"/>
 <wire x1="223.52" y1="111.76" x2="228.6" y2="111.76" width="0.1524" layer="91"/>
-<wire x1="228.6" y1="111.76" x2="236.22" y2="111.76" width="0.1524" layer="91"/>
 <pinref part="C16" gate="G$1" pin="2"/>
-<junction x="228.6" y="111.76"/>
 <wire x1="223.52" y1="111.76" x2="223.52" y2="104.14" width="0.1524" layer="91"/>
 <wire x1="223.52" y1="104.14" x2="172.72" y2="104.14" width="0.1524" layer="91"/>
@@
 <pinref part="P+10" gate="1" pin="+5V"/>
 </segment>
+<segment>
+<pinref part="X5" gate="-1" pin="K"/>
+<pinref part="U5" gate="A" pin="VIN"/>
+<wire x1="177.8" y1="71.12" x2="185.42" y2="71.12" width="0.1524" layer="91"/>
+<pinref part="U5" gate="A" pin="EN"/>
+<wire x1="185.42" y1="71.12" x2="200.66" y2="71.12" width="0.1524" layer="91"/>
+<wire x1="203.2" y1="71.12" x2="203.2" y2="63.5" width="0.1524" layer="91"/>
+<wire x1="185.42" y1="71.12" x2="185.42" y2="63.5" width="0.1524" layer="91"/>
+<wire x1="185.42" y1="63.5" x2="193.04" y2="63.5" width="0.1524" layer="91"/>
+<pinref part="C10" gate="G$1" pin="1"/>
+<junction x="185.42" y="63.5"/>
+<pinref part="C17" gate="G$1" pin="1"/>
+<wire x1="203.2" y1="71.12" x2="200.66" y2="71.12" width="0.1524" layer="91"/>
+<junction x="203.2" y="71.12"/>
+<wire x1="200.66" y1="71.12" x2="200.66" y2="63.5" width="0.1524" layer="91"/>
+<junction x="200.66" y="71.12"/>
+<pinref part="C26" gate="G$1" pin="1"/>
+</segment>
 </net>
 <net name="+3V3" class="0">
@@
 </segment>
 </net>
-<net name="V_IN" class="0">
-<segment>
-<pinref part="X2" gate="-1" pin="K"/>
-<wire x1="236.22" y1="119.38" x2="228.6" y2="119.38" width="0.1524" layer="91"/>
-<pinref part="C16" gate="G$1" pin="1"/>
-<wire x1="220.98" y1="119.38" x2="228.6" y2="119.38" width="0.1524" layer="91"/>
-<junction x="228.6" y="119.38"/>
-<pinref part="T2" gate="A" pin="INPUT"/>
-</segment>
-</net>
 <net name="SS1_5V" class="0">
 <segment>
@@
 </segment>
 </net>
-<net name="N$5" class="0">
-<segment>
-<pinref part="X5" gate="-1" pin="K"/>
-<pinref part="U5" gate="A" pin="VIN"/>
-<wire x1="177.8" y1="71.12" x2="185.42" y2="71.12" width="0.1524" layer="91"/>
-<pinref part="U5" gate="A" pin="EN"/>
-<wire x1="185.42" y1="71.12" x2="200.66" y2="71.12" width="0.1524" layer="91"/>
-<wire x1="203.2" y1="71.12" x2="203.2" y2="63.5" width="0.1524" layer="91"/>
-<wire x1="185.42" y1="71.12" x2="185.42" y2="63.5" width="0.1524" layer="91"/>
-<wire x1="185.42" y1="63.5" x2="193.04" y2="63.5" width="0.1524" layer="91"/>
-<pinref part="C10" gate="G$1" pin="1"/>
-<junction x="185.42" y="63.5"/>
-<pinref part="C17" gate="G$1" pin="1"/>
-<wire x1="203.2" y1="71.12" x2="200.66" y2="71.12" width="0.1524" layer="91"/>
-<junction x="203.2" y="71.12"/>
-<wire x1="200.66" y1="71.12" x2="200.66" y2="63.5" width="0.1524" layer="91"/>
-<junction x="200.66" y="71.12"/>
-<pinref part="C26" gate="G$1" pin="1"/>
-</segment>
-</net>

Commit message: Working on the board
Connections:
- net +3V3: now also C15.1, T2.OUTPUT
- net +5V: no longer C15.1, T2.OUTPUT
Changed lines of the file:
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@@
-</segment>
-<segment>
-<wire x1="162.56" y1="116.84" x2="162.56" y2="119.38" width="0.1524" layer="91"/>
-<pinref part="C15" gate="G$1" pin="1"/>
-<wire x1="162.56" y1="119.38" x2="162.56" y2="121.92" width="0.1524" layer="91"/>
-<junction x="162.56" y="119.38"/>
-<pinref part="T2" gate="A" pin="OUTPUT"/>
-<wire x1="162.56" y1="119.38" x2="180.34" y2="119.38" width="0.1524" layer="91"/>
-<pinref part="P+5" gate="1" pin="+5V"/>
 </segment>
 <segment>
@@
 <junction x="302.26" y="200.66"/>
 </segment>
-</net>
+<segment>
+<wire x1="162.56" y1="116.84" x2="162.56" y2="119.38" width="0.1524" layer="91"/>
+<pinref part="C15" gate="G$1" pin="1"/>
+<wire x1="162.56" y1="119.38" x2="162.56" y2="121.92" width="0.1524" layer="91"/>
+<junction x="162.56" y="119.38"/>
+<pinref part="T2" gate="A" pin="OUTPUT"/>
+<wire x1="162.56" y1="119.38" x2="180.34" y2="119.38" width="0.1524" layer="91"/>
+<pinref part="P+5" gate="1" pin="+5V"/>
+</segment>
+</net>

Commit message: Finishing touches with board layout
Connections:
- net LOGIC_RX_3V3: now also U6.A2; no longer U4.A1
- net LOGIC_RX_5V: now also U6.B2; no longer U4.B1
- net LOGIC_TX_3V3: now also U6.A1; no longer U4.A2
- net LOGIC_TX_5V: now also U6.B1; no longer U4.B2
Changed lines of the file:
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@@
 <net name="LOGIC_TX_3V3" class="0">
-<segment>
-<pinref part="U4" gate="A" pin="A2"/>
-<label x="172.72" y="180.34" size="1.27" layer="95" rot="R180" xref="yes"/>
-<wire x1="180.34" y1="180.34" x2="172.72" y2="180.34" width="0.1524" layer="91"/>
-</segment>
 <segment>
 <label x="109.22" y="119.38" size="1.27" layer="95" rot="R180" xref="yes"/>
@@
 <pinref part="X1" gate="G$1" pin="X-4"/>
 </segment>
+<segment>
+<label x="299.72" y="185.42" size="1.27" layer="95" rot="R180" xref="yes"/>
+<wire x1="307.34" y1="185.42" x2="299.72" y2="185.42" width="0.1524" layer="91"/>
+<pinref part="U6" gate="A" pin="A1"/>
+</segment>
 </net>
 <net name="LOGIC_RX_3V3" class="0">
-<segment>
-<pinref part="U4" gate="A" pin="A1"/>
-<label x="172.72" y="185.42" size="1.27" layer="95" rot="R180" xref="yes"/>
-<wire x1="180.34" y1="185.42" x2="172.72" y2="185.42" width="0.1524" layer="91"/>
-</segment>
 <segment>
 <label x="109.22" y="116.84" size="1.27" layer="95" rot="R180" xref="yes"/>
@@
 <label x="109.22" y="116.84" size="1.27" layer="95" rot="R180" xref="yes"/>
 <pinref part="X1" gate="G$1" pin="X-5"/>
+</segment>
+<segment>
+<label x="299.72" y="180.34" size="1.27" layer="95" rot="R180" xref="yes"/>
+<wire x1="307.34" y1="180.34" x2="299.72" y2="180.34" width="0.1524" layer="91"/>
+<pinref part="U6" gate="A" pin="A2"/>
 </segment>
 </net>
@@
 <net name="LOGIC_RX_5V" class="0">
 <segment>
-<pinref part="U4" gate="A" pin="B1"/>
-<label x="243.84" y="185.42" size="1.27" layer="95" xref="yes"/>
-<wire x1="236.22" y1="185.42" x2="243.84" y2="185.42" width="0.1524" layer="91"/>
+<label x="370.84" y="180.34" size="1.27" layer="95" xref="yes"/>
+<wire x1="363.22" y1="180.34" x2="370.84" y2="180.34" width="0.1524" layer="91"/>
+<pinref part="U6" gate="A" pin="B2"/>
 </segment>
 </net>
 <net name="LOGIC_TX_5V" class="0">
 <segment>
-<pinref part="U4" gate="A" pin="B2"/>
-<label x="243.84" y="180.34" size="1.27" layer="95" xref="yes"/>
-<wire x1="236.22" y1="180.34" x2="243.84" y2="180.34" width="0.1524" layer="91"/>
+<label x="370.84" y="185.42" size="1.27" layer="95" xref="yes"/>
+<wire x1="363.22" y1="185.42" x2="370.84" y2="185.42" width="0.1524" layer="91"/>
+<pinref part="U6" gate="A" pin="B1"/>
 </segment>
 </net>

Commit message: Board functionally done, just need to make it look better
Connections:
- net +3V3: now also C3.1
- net +5V: no longer C3.1
Changed lines of the file:
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@@
-</segment>
-<segment>
-<wire x1="15.24" y1="203.2" x2="15.24" y2="198.12" width="0.1524" layer="91"/>
-<pinref part="+3V2" gate="1" pin="+5V"/>
-<pinref part="C3" gate="G$1" pin="1"/>
 </segment>
 <segment>
@@
 <pinref part="P+5" gate="1" pin="+5V"/>
 </segment>
-</net>
+<segment>
+<wire x1="15.24" y1="203.2" x2="15.24" y2="198.12" width="0.1524" layer="91"/>
+<pinref part="+3V2" gate="1" pin="+5V"/>
+<pinref part="C3" gate="G$1" pin="1"/>
+</segment>
+</net>
