File: core-boards/diagnostics-main/diagnostic-main.brd (EAGLE design)
At the start: 79.2 x 85 mm, 31 parts, among them J1 A118090TR-ND, J2 3M15451-ND, J3 B2PS-VH(LF)(SN), Q1 16 MHz, U1 ATMEGA2560-16AU, U2 296-38653-1-ND, U3 MCP2551T-I/SN, U4 LM1085ISX-5.0/NOPB, U5 LP2985IM5X-3.3/NOPB, U6 TXB0106PWR, X1 22-23-2031, X2 B6B-EH-A(LF)(SN), X5 22-23-2031, X8 WM4803-ND

Commit message: Small Design Review Changes
Connections:
- removed net LOGIC_RX: U1.64, X2.X-4
- removed net LOGIC_TX: U1.63, X2.X-3
- new net DIAG_RX: U1.63, X2.X-4
- new net DIAG_TX: U1.64, X2.X-3
- net CAN_RX: now also U3.1; no longer U3.4
- net CAN_TX: now also U3.4; no longer U3.1
Routing:
- net LOGIC_RX: track 61.8 -> 0.00 mm, vias 1 -> 0
- net DIAG_TX: track 0.00 -> 61.1 mm, vias 0 -> 1
- net LOGIC_TX: track 60.0 -> 0.00 mm, vias 1 -> 0
- net DIAG_RX: track 0.00 -> 57.5 mm, vias 0 -> 1
- net CAN_TX: track 7.81 -> 4.46 mm
- net CAN_RX: track 11.5 -> 8.68 mm
Changed lines of the file:
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@@
 <layer number="45" name="Holes" color="7" fill="1" visible="no" active="yes"/>
 <layer number="46" name="Milling" color="3" fill="1" visible="no" active="yes"/>
-<layer number="47" name="Measures" color="7" fill="1" visible="no" active="yes"/>
+<layer number="47" name="Measures" color="7" fill="1" visible="yes" active="yes"/>
 <layer number="48" name="Document" color="7" fill="1" visible="yes" active="yes"/>
 <layer number="49" name="Reference" color="7" fill="1" visible="yes" active="yes"/>
@@
 <via x="33.274" y="60.452" extent="1-16" drill="0.35"/>
 <wire x1="34.9146625" y1="60.4694" x2="33.2914" y2="60.4694" width="0.254" layer="1"/>
-<wire x1="70.358" y1="45.632" x2="70.446" y2="45.72" width="0.8128" layer="1"/>
 <wire x1="70.358" y1="45.632" x2="73.152" y2="45.632" width="0.8128" layer="1"/>
 <wire x1="73.152" y1="45.632" x2="75.946" y2="45.632" width="0.8128" layer="1"/>
@@
 <wire x1="11.03" y1="51.816" x2="10.414" y2="51.816" width="0.508" layer="1"/>
 <via x="10.414" y="51.816" extent="1-16" drill="0.35"/>
-<wire x1="10.414" y1="51.816" x2="10.414" y2="49.276" width="0.8128" layer="16"/>
+<wire x1="10.414" y1="51.816" x2="10.414" y2="49.276" width="0.508" layer="16"/>
 <via x="10.414" y="49.276" extent="1-16" drill="0.35"/>
 <wire x1="35.306" y1="38.78" x2="43.098" y2="38.78" width="0.8128" layer="16"/>
@@
 <via x="43.18" y="38.862" extent="1-16" drill="0.35"/>
 <wire x1="15.412" y1="57.938" x2="15.412" y2="56.306" width="0.508" layer="1"/>
-<wire x1="12.192" y1="54.7878" x2="10.414" y2="53.0098" width="0.8128" layer="1"/>
-<wire x1="10.414" y1="53.0098" x2="10.414" y2="51.816" width="0.8128" layer="1"/>
-<wire x1="15.412" y1="56.306" x2="13.8938" y2="54.7878" width="0.8128" layer="1"/>
-<wire x1="13.8938" y1="54.7878" x2="12.192" y2="54.7878" width="0.8128" layer="1"/>
+<wire x1="12.192" y1="54.7878" x2="10.414" y2="53.0098" width="0.508" layer="1"/>
+<wire x1="10.414" y1="53.0098" x2="10.414" y2="51.816" width="0.508" layer="1"/>
+<wire x1="15.412" y1="56.306" x2="13.8938" y2="54.7878" width="0.508" layer="1"/>
+<wire x1="13.8938" y1="54.7878" x2="12.192" y2="54.7878" width="0.508" layer="1"/>
+<wire x1="75.946" y1="47.332" x2="74.1045" y2="49.0728" width="0" layer="19" extent="1-1"/>
+<wire x1="44.108" y1="46.228" x2="74.1045" y2="49.0728" width="0" layer="19" extent="1-1"/>
+<wire x1="41.899" y1="46.2026" x2="44.108" y2="46.228" width="0" layer="19" extent="1-1"/>
+<wire x1="37.999" y1="46.2026" x2="41.899" y2="46.2026" width="0" layer="19" extent="1-1"/>
+<wire x1="43.18" y1="38.862" x2="44.108" y2="46.228" width="0" layer="19" extent="1-1"/>
+<wire x1="14.249" y1="46.73" x2="35.306" y2="38.78" width="0" layer="19" extent="1-1"/>
+<wire x1="14.644" y1="49.022" x2="14.249" y2="46.73" width="0" layer="19" extent="1-1"/>
+<wire x1="10.414" y1="49.276" x2="14.644" y2="49.022" width="0" layer="19" extent="1-1"/>
 </signal>
 <signal name="SCK3V3">
@@
 <wire x1="30.226" y1="85.09" x2="38.233475" y2="85.09" width="0.254" layer="1"/>
 </signal>
-<signal name="LOGIC_RX">
-<contactref element="X2" pad="X-4"/>
-<contactref element="U1" pad="64"/>
-<wire x1="50.038" y1="71.12" x2="52.07" y2="71.12" width="0.254" layer="1"/>
-<via x="52.07" y="71.12" extent="1-16" drill="0.35"/>
-<wire x1="62.5884" y1="57.8936125" x2="63.246" y2="57.2360125" width="0.254" layer="16"/>
-<wire x1="52.07" y1="71.12" x2="62.5884" y2="60.6016" width="0.254" layer="16"/>
-<wire x1="62.5884" y1="60.6016" x2="62.5884" y2="57.8936125" width="0.254" layer="16"/>
-<wire x1="63.246" y1="57.2360125" x2="63.246" y2="26.162" width="0.254" layer="16"/>
-<wire x1="69.944" y1="19.464" x2="69.944" y2="18.71" width="0.254" layer="16"/>
-<wire x1="63.246" y1="26.162" x2="69.944" y2="19.464" width="0.254" layer="16"/>
-</signal>
 <signal name="ENCODER2_SENSE">
 <contactref element="X2" pad="X-2"/>
@@
 <wire x1="62.484" y1="18.75" x2="62.444" y2="18.71" width="0.254" layer="16"/>
 </signal>
-<signal name="LOGIC_TX">
-<contactref element="X2" pad="X-3"/>
-<contactref element="U1" pad="63"/>
-<via x="52.07" y="70.104" extent="1-16" drill="0.35"/>
-<wire x1="62.8396" y1="57.067675" x2="62.182" y2="57.725275" width="0.254" layer="16"/>
-<wire x1="62.182" y1="59.992" x2="52.07" y2="70.104" width="0.254" layer="16"/>
-<wire x1="62.182" y1="57.725275" x2="62.182" y2="59.992" width="0.254" layer="16"/>
-<wire x1="52.07" y1="70.104" x2="51.562" y2="70.612" width="0.254" layer="1"/>
-<wire x1="51.562" y1="70.612" x2="50.038" y2="70.612" width="0.254" layer="1"/>
-<wire x1="62.8396" y1="57.067675" x2="62.8396" y2="25.8064" width="0.254" layer="16"/>
-<wire x1="67.444" y1="21.202" x2="67.444" y2="18.71" width="0.254" layer="16"/>
-<wire x1="62.8396" y1="25.8064" x2="67.444" y2="21.202" width="0.254" layer="16"/>
-</signal>
 <signal name="ESTOPCONNECTED">
 <contactref element="X1" pad="1"/>
@@
 <signal name="CAN_RX">
 <contactref element="U1" pad="45"/>
-<contactref element="U3" pad="4"/>
-<wire x1="52.2478" y1="55.753" x2="49.403" y2="55.753" width="0.254" layer="1"/>
 <wire x1="45.9232" y1="59.2328" x2="45.9232" y2="62.992" width="0.254" layer="1"/>
 <wire x1="49.403" y1="55.753" x2="45.9232" y2="59.2328" width="0.254" layer="1"/>
+<contactref element="U3" pad="1"/>
+<wire x1="49.403" y1="55.753" x2="52.2478" y2="59.563" width="0" layer="19" extent="1-1"/>
 </signal>
 <signal name="CAN_TX">
 <contactref element="U1" pad="46"/>
-<contactref element="U3" pad="1"/>
-<wire x1="52.2478" y1="59.563" x2="48.895" y2="59.563" width="0.254" layer="1"/>
 <wire x1="46.4058" y1="62.0522" x2="46.4058" y2="62.992" width="0.254" layer="1"/>
 <wire x1="48.895" y1="59.563" x2="46.4058" y2="62.0522" width="0.254" layer="1"/>
+<contactref element="U3" pad="4"/>
+<wire x1="52.2478" y1="55.753" x2="48.895" y2="59.563" width="0" layer="19" extent="1-1"/>
 </signal>
 <signal name="IRQ">
@@
 <wire x1="4.572" y1="96.012" x2="5.6896" y2="94.8944" width="0.254" layer="16"/>
 </signal>
+<signal name="DIAG_RX">
+<contactref element="X2" pad="X-4"/>
+<contactref element="U1" pad="63"/>
+<via x="52.07" y="70.104" extent="1-16" drill="0.35"/>
+<wire x1="62.8396" y1="57.067675" x2="62.182" y2="57.725275" width="0.254" layer="16"/>
+<wire x1="62.182" y1="59.992" x2="52.07" y2="70.104" width="0.254" layer="16"/>
+<wire x1="62.182" y1="57.725275" x2="62.182" y2="59.992" width="0.254" layer="16"/>
+<wire x1="52.07" y1="70.104" x2="51.562" y2="70.612" width="0.254" layer="1"/>
+<wire x1="51.562" y1="70.612" x2="50.038" y2="70.612" width="0.254" layer="1"/>
+<wire x1="62.8396" y1="57.067675" x2="62.8396" y2="25.8064" width="0.254" layer="16"/>
+<wire x1="62.8396" y1="25.8064" x2="67.444" y2="21.202" width="0.254" layer="16"/>
+<wire x1="67.444" y1="21.202" x2="69.944" y2="18.71" width="0" layer="19" extent="16-16"/>
+</signal>
+<signal name="DIAG_TX">
+<contactref element="X2" pad="X-3"/>
+<contactref element="U1" pad="64"/>
+<wire x1="50.038" y1="71.12" x2="52.07" y2="71.12" width="0.254" layer="1"/>
+<via x="52.07" y="71.12" extent="1-16" drill="0.35"/>
+<wire x1="62.5884" y1="57.8936125" x2="63.246" y2="57.2360125" width="0.254" layer="16"/>
+<wire x1="52.07" y1="71.12" x2="62.5884" y2="60.6016" width="0.254" layer="16"/>
+<wire x1="62.5884" y1="60.6016" x2="62.5884" y2="57.8936125" width="0.254" layer="16"/>
+<wire x1="63.246" y1="57.2360125" x2="63.246" y2="26.162" width="0.254" layer="16"/>
+<wire x1="63.246" y1="26.162" x2="69.944" y2="19.464" width="0.254" layer="16"/>
+<wire x1="67.444" y1="18.71" x2="69.944" y2="19.464" width="0" layer="19" extent="16-16"/>
+</signal>
 </signals>
