File: core-boards/diagnostics-main/diagnostic-main.sch (EAGLE design)
At the start: 31 parts, among them J1 A118090TR-ND, J2 3M15451-ND, J3 B2PS-VH(LF)(SN), Q1 16 MHz, U1 ATMEGA2560-16AU, U2 296-38653-1-ND, U3 MCP2551T-I/SN, U4 LM1085ISX-5.0/NOPB, U5 LP2985IM5X-3.3/NOPB, U6 TXB0106PWR, X1 22-23-2031, X2 B6B-EH-A(LF)(SN), X5 22-23-2031, X8 WM4803-ND

Commit message: Small Design Review Changes
Connections:
- removed net LOGIC_RX: U1.PJ1_(TXD3/PCINT10), X2.X-4
- removed net LOGIC_TX: U1.PJ0_(RXD3/PCINT9), X2.X-3
- new net DIAG_RX: U1.PJ0_(RXD3/PCINT9), X2.X-4
- new net DIAG_TX: U1.PJ1_(TXD3/PCINT10), X2.X-3
- net CAN_RX: now also U3.TXD; no longer U3.RXD
- net CAN_TX: now also U3.RXD; no longer U3.TXD
Other:
- note added: "ADD RADIO PART LABEL"
- note added: "Voltage Regulator (12v -> 5v @ 3A)"
- note removed: "Voltage Regulator (12v -> 3v3 @ 3A)"
Changed lines of the file:
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@@
 </segment>
 </net>
-<net name="LOGIC_TX" class="0">
+<net name="DIAG_RX" class="0">
 <segment>
 <wire x1="109.22" y1="71.12" x2="111.76" y2="71.12" width="0.1524" layer="91"/>
@@
 </segment>
 </net>
-<net name="LOGIC_RX" class="0">
+<net name="CAN_RX" class="0">
+<segment>
+<pinref part="U1" gate="A" pin="(RXD1/INT2)_PD2"/>
+<wire x1="17.78" y1="40.64" x2="15.24" y2="40.64" width="0.1524" layer="91"/>
+<label x="15.24" y="40.64" size="1.778" layer="95" rot="R180" xref="yes"/>
+</segment>
+</net>
+<net name="CAN_TX" class="0">
+<segment>
+<pinref part="U1" gate="A" pin="(TXD1/INT3)_PD3"/>
+<wire x1="17.78" y1="38.1" x2="15.24" y2="38.1" width="0.1524" layer="91"/>
+<label x="15.24" y="38.1" size="1.778" layer="95" rot="R180" xref="yes"/>
+</segment>
+</net>
+<net name="CSN" class="0">
+<segment>
+<pinref part="U1" gate="A" pin="(OC0A/OC1C/PCINT7)_PB7"/>
+<wire x1="17.78" y1="73.66" x2="15.24" y2="73.66" width="0.1524" layer="91"/>
+<label x="15.24" y="73.66" size="1.778" layer="95" rot="R180" xref="yes"/>
+</segment>
+</net>
+<net name="IRQ" class="0">
+<segment>
+<pinref part="U1" gate="A" pin="(OC1B/PCINT6)_PB6"/>
+<wire x1="17.78" y1="76.2" x2="15.24" y2="76.2" width="0.1524" layer="91"/>
+<label x="15.24" y="76.2" size="1.778" layer="95" rot="R180" xref="yes"/>
+</segment>
+</net>
+<net name="SS_RADIO" class="0">
+<segment>
+<pinref part="U1" gate="A" pin="(OC1A/PCINT5)_PB5"/>
+<wire x1="17.78" y1="78.74" x2="15.24" y2="78.74" width="0.1524" layer="91"/>
+<label x="15.24" y="78.74" size="1.778" layer="95" rot="R180" xref="yes"/>
+</segment>
+</net>
+<net name="ENCODER2_SENSE" class="0">
+<segment>
+<wire x1="17.78" y1="66.04" x2="12.7" y2="66.04" width="0.1524" layer="91"/>
+<label x="12.7" y="66.04" size="1.778" layer="95" rot="R180" xref="yes"/>
+<pinref part="U1" gate="A" pin="PC1_(A9)"/>
+</segment>
+</net>
+<net name="ENCODER1_SENSE" class="0">
+<segment>
+<wire x1="17.78" y1="68.58" x2="12.7" y2="68.58" width="0.1524" layer="91"/>
+<label x="12.7" y="68.58" size="1.778" layer="95" rot="R180" xref="yes"/>
+<pinref part="U1" gate="A" pin="PC0_(A8)"/>
+</segment>
+</net>
+<net name="MASTCONNECTED" class="0">
+<segment>
+<pinref part="U1" gate="A" pin="PK1_(ADC9/PCINT17)"/>
+<wire x1="109.22" y1="45.72" x2="111.76" y2="45.72" width="0.1524" layer="91"/>
+<label x="111.76" y="45.72" size="1.778" layer="95" xref="yes"/>
+</segment>
+</net>
+<net name="DIAG_TX" class="0">
 <segment>
 <wire x1="109.22" y1="68.58" x2="111.76" y2="68.58" width="0.1524" layer="91"/>
 <label x="111.76" y="68.58" size="1.778" layer="95" xref="yes"/>
 <pinref part="U1" gate="A" pin="PJ1_(TXD3/PCINT10)"/>
-</segment>
-</net>
-<net name="CAN_RX" class="0">
-<segment>
-<pinref part="U1" gate="A" pin="(RXD1/INT2)_PD2"/>
-<wire x1="17.78" y1="40.64" x2="15.24" y2="40.64" width="0.1524" layer="91"/>
-<label x="15.24" y="40.64" size="1.778" layer="95" rot="R180" xref="yes"/>
-</segment>
-</net>
-<net name="CAN_TX" class="0">
-<segment>
-<pinref part="U1" gate="A" pin="(TXD1/INT3)_PD3"/>
-<wire x1="17.78" y1="38.1" x2="15.24" y2="38.1" width="0.1524" layer="91"/>
-<label x="15.24" y="38.1" size="1.778" layer="95" rot="R180" xref="yes"/>
-</segment>
-</net>
-<net name="CSN" class="0">
-<segment>
-<pinref part="U1" gate="A" pin="(OC0A/OC1C/PCINT7)_PB7"/>
-<wire x1="17.78" y1="73.66" x2="15.24" y2="73.66" width="0.1524" layer="91"/>
-<label x="15.24" y="73.66" size="1.778" layer="95" rot="R180" xref="yes"/>
-</segment>
-</net>
-<net name="IRQ" class="0">
-<segment>
-<pinref part="U1" gate="A" pin="(OC1B/PCINT6)_PB6"/>
-<wire x1="17.78" y1="76.2" x2="15.24" y2="76.2" width="0.1524" layer="91"/>
-<label x="15.24" y="76.2" size="1.778" layer="95" rot="R180" xref="yes"/>
-</segment>
-</net>
-<net name="SS_RADIO" class="0">
-<segment>
-<pinref part="U1" gate="A" pin="(OC1A/PCINT5)_PB5"/>
-<wire x1="17.78" y1="78.74" x2="15.24" y2="78.74" width="0.1524" layer="91"/>
-<label x="15.24" y="78.74" size="1.778" layer="95" rot="R180" xref="yes"/>
-</segment>
-</net>
-<net name="ENCODER2_SENSE" class="0">
-<segment>
-<wire x1="17.78" y1="66.04" x2="12.7" y2="66.04" width="0.1524" layer="91"/>
-<label x="12.7" y="66.04" size="1.778" layer="95" rot="R180" xref="yes"/>
-<pinref part="U1" gate="A" pin="PC1_(A9)"/>
-</segment>
-</net>
-<net name="ENCODER1_SENSE" class="0">
-<segment>
-<wire x1="17.78" y1="68.58" x2="12.7" y2="68.58" width="0.1524" layer="91"/>
-<label x="12.7" y="68.58" size="1.778" layer="95" rot="R180" xref="yes"/>
-<pinref part="U1" gate="A" pin="PC0_(A8)"/>
-</segment>
-</net>
-<net name="MASTCONNECTED" class="0">
-<segment>
-<pinref part="U1" gate="A" pin="PK1_(ADC9/PCINT17)"/>
-<wire x1="109.22" y1="45.72" x2="111.76" y2="45.72" width="0.1524" layer="91"/>
-<label x="111.76" y="45.72" size="1.778" layer="95" xref="yes"/>
 </segment>
 </net>
@@
 <wire x1="345.44" y1="233.68" x2="345.44" y2="271.78" width="0.1524" layer="97" style="shortdash"/>
 <wire x1="345.44" y1="271.78" x2="266.7" y2="271.78" width="0.1524" layer="97" style="shortdash"/>
-<text x="271.78" y="266.7" size="1.778" layer="97">Voltage Regulator (12v -&gt; 3v3 @ 3A)</text>
+<text x="271.78" y="266.7" size="1.778" layer="97">Voltage Regulator (12v -&gt; 5v @ 3A)</text>
 <text x="381" y="269.24" size="1.778" layer="97" rot="R180">Voltage Regulator (5v -&gt; 3v3)</text>
 <wire x1="347.98" y1="271.78" x2="424.18" y2="271.78" width="0.1524" layer="97" style="shortdash"/>
@@
 <wire x1="58.42" y1="238.76" x2="58.42" y2="269.24" width="0.1524" layer="97" style="shortdash"/>
 <text x="60.96" y="266.7" size="1.778" layer="97">Mast Board Connnector</text>
+<text x="27.94" y="81.28" size="1.778" layer="91">ADD RADIO PART LABEL</text>
 </plain>
 <instances>
@@
 </segment>
 </net>
-<net name="CAN_TX" class="0">
+<net name="CAN_RX" class="0">
 <segment>
 <wire x1="35.56" y1="30.48" x2="25.4" y2="30.48" width="0.1524" layer="91"/>
@@
 </segment>
 </net>
-<net name="CAN_RX" class="0">
-<segment>
-<wire x1="35.56" y1="22.86" x2="25.4" y2="22.86" width="0.1524" layer="91"/>
-<label x="25.4" y="22.86" size="1.778" layer="95" rot="R180" xref="yes"/>
-<pinref part="U3" gate="A" pin="RXD"/>
-</segment>
-</net>
-<net name="LOGIC_RX" class="0">
-<segment>
-<pinref part="X2" gate="G$1" pin="X-4"/>
-<wire x1="27.94" y1="220.98" x2="33.02" y2="220.98" width="0.1524" layer="91"/>
-<label x="33.02" y="220.98" size="1.778" layer="95" xref="yes"/>
-</segment>
-</net>
 <net name="ENCODER2_SENSE" class="0">
 <segment>
@@
 <wire x1="27.94" y1="213.36" x2="33.02" y2="213.36" width="0.1524" layer="91"/>
 <label x="33.02" y="213.36" size="1.778" layer="95" xref="yes"/>
-</segment>
-</net>
-<net name="LOGIC_TX" class="0">
-<segment>
-<pinref part="X2" gate="G$1" pin="X-3"/>
-<wire x1="27.94" y1="218.44" x2="33.02" y2="218.44" width="0.1524" layer="91"/>
-<label x="33.02" y="218.44" size="1.778" layer="95" xref="yes"/>
 </segment>
 </net>
@@
 </segment>
 </net>
+<net name="CAN_TX" class="0">
+<segment>
+<wire x1="35.56" y1="22.86" x2="25.4" y2="22.86" width="0.1524" layer="91"/>
+<label x="25.4" y="22.86" size="1.778" layer="95" rot="R180" xref="yes"/>
+<pinref part="U3" gate="A" pin="RXD"/>
+</segment>
+</net>
+<net name="DIAG_RX" class="0">
+<segment>
+<pinref part="X2" gate="G$1" pin="X-4"/>
+<wire x1="27.94" y1="220.98" x2="33.02" y2="220.98" width="0.1524" layer="91"/>
+<label x="33.02" y="220.98" size="1.778" layer="95" xref="yes"/>
+</segment>
+</net>
+<net name="DIAG_TX" class="0">
+<segment>
+<pinref part="X2" gate="G$1" pin="X-3"/>
+<wire x1="27.94" y1="218.44" x2="33.02" y2="218.44" width="0.1524" layer="91"/>
+<label x="33.02" y="218.44" size="1.778" layer="95" xref="yes"/>
+</segment>
+</net>
