File: core-boards/diagnostics-main/Eagle Files/diagnostic-main.brd (EAGLE design)
At the start: 79.2 x 85 mm, 31 parts, among them J1 A118090TR-ND, J2 3M15451-ND, J3 B2PS-VH(LF)(SN), Q1 16 MHz, U1 ATMEGA2560-16AU, U2 296-38653-1-ND, U3 MCP2551T-I/SN, U4 LM1085ISX-5.0/NOPB, U5 LP2985IM5X-3.3/NOPB, U6 TXB0106PWR, X1 22-23-2031, X2 B6B-EH-A(LF)(SN), X5 22-23-2031, X8 WM4803-ND

Commit message: Internal Design Review Changes
Parts:
- removed C10, C9: 10uF, rcl:C0805
- removed C6: 2.2uF, rcl:C0603
- removed C7: .01uF, rcl:C0603
- removed C8: 1uF, rcl:C0603
- removed J3: B2PS-VH(LF)(SN), RoboJackets-Connectors:B2PS-CENTERED
- removed U4: LM1085ISX-5.0/NOPB, LM1085ISX:TS3B
- removed U5: LP2985IM5X-3.3/NOPB, LP2985IM5X:MF05A
- added C13: 2.2uF, rcl:C0603
- added C14: .01uF, rcl:C0603
- added C15: 1uF, rcl:C0603
- added C16, C17: 10uF, rcl:C0805
- added J4: B2PS-VH(LF)(SN), RoboJackets-Connectors:B2PS-CENTERED
- added U7: LM1085ISX-5.0/NOPB, LM1085ISX:TS3B
- added U8: LP2985IM5X-3.3/NOPB, LP2985IM5X:MF05A
- moved X3 2.79 mm to (54.4, 32.8)
- moved U6 1.52 mm to (39.6, 47.5)
- moved C12 0.76 mm to (34.8, 51.3)
Connections:
- removed net N$1: C7.1, U5.4
- new net N$2: C14.1, U8.4
- net +12V: now also C17.1, J4.2, U7.3; no longer C10.1, J3.2, U4.3
- net +3V3: now also C13.1, U8.5; no longer C6.1, U5.5
- net +5V: now also C15.1, C16.1, U7.2, U8.1, U8.3; no longer C8.1, C9.1, U4.2, U5.1, U5.3
- net CSN: now also U6.10; no longer U6.12
- net CSN3V3: now also U6.7; no longer U6.5
- net GND: now also C13.2, C14.2, C15.2, C16.2, C17.2, J4.1, U7.1, U8.2; no longer C10.2, C6.2, C7.2, C8.2, C9.2, J3.1, U4.1, U5.2
- net IRQ: now also U6.11; no longer U6.10
- net IRQ3V3: now also U6.6; no longer U6.7
- net MISO: now also U2.10; no longer U2.12
- net MISO3V3: now also U2.5; no longer U2.3
- net MOSI: now also U6.13; no longer U6.11
- net MOSI3V3: now also U6.4; no longer U6.6
- net SCK: now also U2.12, U6.12; no longer U2.10, U6.13
- net SCK3V3: now also U2.3, U6.5; no longer U2.5, U6.4
Routing:
- net GND: track 128.1 -> 104.8 mm, vias 22 -> 17
- net +12V: track 13.5 -> 0.00 mm
- net MISO: track 67.4 -> 74.9 mm
- net DIAG_TX: track 61.1 -> 68.1 mm
- net CAN_TX: track 4.46 -> 10.6 mm, vias 0 -> 2
- net +5V: track 0.00 -> 5.81 mm
- net MISO3V3: track 27.7 -> 33.3 mm
- net CSN: track 16.9 -> 22.0 mm
- net MOSI: track 73.3 -> 69.2 mm, vias 3 -> 2
- net DIAG_RX: track 57.5 -> 61.0 mm
- net N$1: track 3.30 -> 0.00 mm
- net SS_RADIO: track 16.1 -> 18.4 mm
- net MOSI3V3: track 29.7 -> 28.2 mm, vias 2 -> 0
- net SS2_3V3: track 11.9 -> 13.2 mm
- net IRQ: track 20.2 -> 21.5 mm
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Other:
- board size 79.2 x 85 mm -> 79.2 x 84.8 mm
- board text added: "ESTOP"
- board text added: "MAST"
- board text added: "MINIBOARDS"

Commit message: Final Changes for design review
Parts:
- added D3, D4, D5: GREEN, SparkFun-LED:LED-0603
- added R18: 2.2k, rcl:R0603
- added R19, R21: 1k, rcl:R0603
- added U$10: (no value), RoboJackets-Aesthetics:ROBOBUZZ_1.4X
- X3: value (none) -> CC1101
- moved C17 112.5 mm to (73.4, 84.8)
- moved C16 105.4 mm to (61.2, 81.0), turned to 90 degrees
- moved U7 104.0 mm to (63.8, 93.2)
- moved J4 101.1 mm to (74.4, 91.7), turned to 180 degrees
- moved C15 95.7 mm to (75.4, 55.4), turned to 270 degrees
- moved C14 93.5 mm to (74.4, 46.0), turned to 270 degrees
- moved U8 87.3 mm to (75.4, 50.3), turned to 270 degrees
- moved C13 82.8 mm to (76.5, 46.0), turned to 270 degrees
Connections:
- new net 12V_LED_R: D3.A, R18.1
- new net 3V3_LED_R: D5.A, R21.1
- new net 5V_LED_R: D4.A, R19.1
- net +12V: now also R18.2
- net +3V3: now also R21.2
- net +5V: now also R19.2
- net GND: now also D3.C, D4.C, D5.C
Routing:
- net +12V: track 0.00 -> 26.8 mm, vias 0 -> 2
- net +3V3: track 21.1 -> 41.6 mm
- net MASTCONNECTED: track 44.1 -> 41.0 mm, vias 0 -> 1
- net N$2: track 0.00 -> 2.28 mm
- net GND: track 104.8 -> 107.0 mm, vias 17 -> 25
- net 5V_LED_R: track 0.00 -> 2.08 mm
- net 3V3_LED_R: track 0.00 -> 2.08 mm
- net 12V_LED_R: track 0.00 -> 2.08 mm
- net CONNECTED: track 32.3 -> 33.2 mm, vias 0 -> 1
- net ESTOPCONNECTED: track 48.4 -> 48.9 mm, vias 0 -> 1
Other:
- outline, holes or cut-outs redrawn
- board text added: "12V"
- board text added: "3V3"
- board text added: "5V"
- board text added: "RoboJackets IGVC Central Diagnostics Board v0.1 BOARD #:"

Commit message: More small changes
Parts:
- removed D5: GREEN, SparkFun-LED:LED-0603
- added D1: GREEN, SparkFun-LED:LED-0603
- moved D3 5.08 mm to (72.1, 69.1)
- renumbered D4 to D2, R18 to R4, R19 to R5, R21 to R6
Connections:
- net 12V_LED_R: now also D1.A; no longer D3.A
- net 3V3_LED_R: now also D3.A; no longer D5.A
- net GND: now also D1.C; no longer D5.C
Routing:
- net CAN_P: track 194.5 -> 193.6 mm
- net CAN_N: track 193.5 -> 192.6 mm
Other:
- board text added: "1"

Commit message: Final Changes for Design Review
Parts:
- moved C16 0.92 mm to (61.7, 80.3)
- moved U7 0.57 mm to (64.3, 93.5)
- moved C5 0.25 mm to (15.7, 49.0)
Routing:
- net CAN_N: track 192.6 -> 150.1 mm, vias 0 -> 3
- net CAN_P: track 193.6 -> 151.4 mm, vias 0 -> 3
- net MISO: track 74.9 -> 72.9 mm
- net GND: track 107.0 -> 108.3 mm
- net +3V3: track 41.6 -> 40.8 mm

Commit message: Design Review Changes
Parts:
- added C10, C21, C25, C6: 1uF, rcl:C0402
- added C18, C22, C26, C7: 10uF, rcl:C0805
- added C19, C23, C8, C9: .1uF, rcl:C0603
- C2: value .01uF -> .1uF
- moved C2 38.2 mm to (8.38, 51.8)
- moved C1 7.47 mm to (38.9, 81.0)
- moved R2 7.44 mm to (23.9, 62.2)
- moved S1 6.65 mm to (21.6, 62.0)
Connections:
- net +3V3: now also C2.1
- net +5V: now also C10.1, C18.1, C19.1, C21.1, C22.1, C23.1, C25.1, C26.1, C6.1, C7.1, C8.1, C9.1; no longer C2.1
- net GND: now also C10.2, C18.2, C19.2, C21.2, C22.2, C23.2, C25.2, C26.2, C6.2, C7.2, C8.2, C9.2
Routing:
- net GND: track 108.3 -> 133.6 mm, vias 25 -> 28
- net !RESET: track 46.9 -> 49.9 mm
- net CSN: track 22.0 -> 24.5 mm
- net IRQ: track 21.5 -> 24.0 mm
- net +3V3: track 40.8 -> 42.0 mm

Commit message: More changes
Parts:
- moved C2 0.76 mm to (7.62, 51.8)
Routing:
- net +3V3: track 42.0 -> 42.8 mm
Changed lines of the file:
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@@
 <drawing>
 <settings>
-<setting alwaysvectorfont="no"/>
+<setting alwaysvectorfont="yes"/>
 <setting verticaltext="up"/>
 </settings>
@@
 <attribute name="SPICEPREFIX" value="C" x="30.988" y="46.736" size="1.778" layer="27" display="off"/>
 </element>
-<element name="C2" library="rcl" library_urn="urn:adsk.eagle:library:334" package="C0603" package3d_urn="urn:adsk.eagle:package:23616/2" value=".1uF" x="8.382" y="51.816" smashed="yes" rot="R180">
-<attribute name="NAME" x="6.731" y="52.197" size="1.27" layer="25" rot="R180"/>
-<attribute name="POPULARITY" value="73" x="8.382" y="51.816" size="1.778" layer="27" rot="R180" display="off"/>
-<attribute name="SPICEPREFIX" value="C" x="8.382" y="51.816" size="1.778" layer="27" rot="R180" display="off"/>
+<element name="C2" library="rcl" library_urn="urn:adsk.eagle:library:334" package="C0603" package3d_urn="urn:adsk.eagle:package:23616/2" value=".1uF" x="7.62" y="51.816" smashed="yes" rot="R180">
+<attribute name="NAME" x="5.969" y="52.197" size="1.27" layer="25" rot="R180"/>
+<attribute name="POPULARITY" value="73" x="7.62" y="51.816" size="1.778" layer="27" rot="R180" display="off"/>
+<attribute name="SPICEPREFIX" value="C" x="7.62" y="51.816" size="1.778" layer="27" rot="R180" display="off"/>
 </element>
 <element name="C9" library="rcl" library_urn="urn:adsk.eagle:library:334" package="C0603" package3d_urn="urn:adsk.eagle:package:23616/2" value=".1uF" x="10.668" y="60.452" smashed="yes" rot="R90">
@@
 <wire x1="10.668" y1="62.484" x2="11.049" y2="62.865" width="0.762" layer="1"/>
 <via x="11.049" y="62.865" extent="1-16" drill="0.35"/>
-<wire x1="7.532" y1="51.816" x2="6.096" y2="51.816" width="0.762" layer="1"/>
-<via x="6.096" y="51.816" extent="1-16" drill="0.35"/>
+<wire x1="6.77" y1="51.816" x2="5.334" y2="51.816" width="0.762" layer="1"/>
+<via x="5.334" y="51.816" extent="1-16" drill="0.35"/>
+<wire x1="76.708" y1="84.836" x2="76.402" y2="91.694" width="0" layer="19" extent="1-1"/>
+<wire x1="73.406" y1="76.2" x2="74.356" y2="84.836" width="0" layer="19" extent="1-1"/>
+<wire x1="64.516" y1="81.28" x2="73.406" y2="76.2" width="0" layer="19" extent="1-1"/>
+<wire x1="73.914" y1="54.356" x2="73.406" y2="67.056" width="0" layer="19" extent="1-1"/>
+<wire x1="76.454" y1="45.124" x2="75.438" y2="51.5112" width="0" layer="19" extent="1-1"/>
+<wire x1="54.422" y1="70.104" x2="61.722" y2="81.214" width="0" layer="19" extent="1-1"/>
+<wire x1="56.9722" y1="59.563" x2="54.722" y2="66.04" width="0" layer="19" extent="1-1"/>
+<wire x1="52.2478" y1="58.293" x2="56.9722" y2="59.563" width="0" layer="19" extent="1-1"/>
+<wire x1="45.974" y1="76.962" x2="48.768" y2="70.104" width="0" layer="19" extent="1-1"/>
+<wire x1="42.838" y1="59.69" x2="50.292" y2="58.42" width="0" layer="19" extent="1-1"/>
+<wire x1="33.274" y1="60.452" x2="36.156" y2="59.69" width="0" layer="19" extent="1-1"/>
+<wire x1="33.528" y1="61.976" x2="33.274" y2="60.452" width="0" layer="19" extent="1-1"/>
+<wire x1="32.258" y1="52.07" x2="31.638" y2="57.912" width="0" layer="19" extent="1-1"/>
+<wire x1="43.18" y1="52.07" x2="42.838" y2="59.69" width="0" layer="19" extent="1-1"/>
+<wire x1="45.808" y1="46.228" x2="41.899" y2="50.3174" width="0" layer="19" extent="1-1"/>
+<wire x1="38.012" y1="81.026" x2="45.9232" y2="78.232" width="0" layer="19" extent="1-1"/>
+<wire x1="31.938" y1="75.438" x2="36.9062" y2="78.232" width="0" layer="19" extent="1-1"/>
+<wire x1="20.828" y1="58.928" x2="31.638" y2="57.912" width="0" layer="19" extent="1-1"/>
+<wire x1="15.412" y1="52.298" x2="20.828" y2="58.928" width="0" layer="19" extent="1-1"/>
+<wire x1="9.398" y1="49.022" x2="15.412" y2="52.298" width="0" layer="19" extent="1-1"/>
+<wire x1="6.77" y1="51.816" x2="9.398" y2="49.022" width="0" layer="19" extent="1-1"/>
+<wire x1="11.049" y1="62.865" x2="20.79" y2="64.026" width="0" layer="19" extent="1-1"/>
+<wire x1="6.35" y1="68.834" x2="11.049" y2="62.865" width="0" layer="19" extent="1-1"/>
+<wire x1="32.766" y1="38.1" x2="33.948" y2="51.308" width="0" layer="19" extent="1-1"/>
+<wire x1="26.924" y1="96.012" x2="36.068" y2="83.566" width="0" layer="19" extent="1-1"/>
+<wire x1="27.584" y1="21.08" x2="32.766" y2="35.986" width="0" layer="19" extent="1-1"/>
 </signal>
 <signal name="!RESET">
@@
 <wire x1="67.564" y1="69" x2="67.564" y2="49.784" width="0.762" layer="1"/>
 <contactref element="C2" pad="1"/>
-<wire x1="9.232" y1="51.816" x2="10.414" y2="51.816" width="0.762" layer="1"/>
+<wire x1="8.47" y1="51.816" x2="10.414" y2="51.816" width="0.762" layer="1"/>
+<wire x1="76.454" y1="46.824" x2="76.3905" y2="49.0728" width="0" layer="19" extent="1-1"/>
+<wire x1="67.564" y1="49.784" x2="76.3905" y2="49.0728" width="0" layer="19" extent="1-1"/>
+<wire x1="44.108" y1="46.228" x2="67.564" y2="49.784" width="0" layer="19" extent="1-1"/>
+<wire x1="41.899" y1="44.6786" x2="44.108" y2="46.228" width="0" layer="19" extent="1-1"/>
+<wire x1="37.999" y1="44.6786" x2="41.899" y2="44.6786" width="0" layer="19" extent="1-1"/>
+<wire x1="43.434" y1="36.83" x2="41.899" y2="44.6786" width="0" layer="19" extent="1-1"/>
+<wire x1="14.898" y1="49.022" x2="37.999" y2="44.6786" width="0" layer="19" extent="1-1"/>
+<wire x1="14.249" y1="46.73" x2="14.898" y2="49.022" width="0" layer="19" extent="1-1"/>
+<wire x1="10.414" y1="49.276" x2="14.898" y2="49.022" width="0" layer="19" extent="1-1"/>
 </signal>
 <signal name="SCK3V3" airwireshidden="yes">
@@
 <contactref element="C17" pad="1"/>
 <contactref element="J4" pad="2"/>
-<wire x1="72.442" y1="91.694" x2="72.442" y2="84.85" width="0.762" layer="1"/>
+<wire x1="72.442" y1="91.694" x2="72.442" y2="89.916" width="0.762" layer="1"/>
+<wire x1="72.442" y1="89.916" x2="72.442" y2="84.85" width="0.762" layer="1"/>
 <wire x1="72.442" y1="84.85" x2="72.456" y2="84.836" width="0.762" layer="1"/>
 <wire x1="72.442" y1="84.85" x2="67.1436" y2="84.85" width="0.762" layer="1"/>

Commit message: More Design Review Changes
Parts:
- removed U$10: (no value), RoboJackets-Aesthetics:ROBOBUZZ_1.4X
- removed U7: LM1085ISX-5.0/NOPB, LM1085ISX:TS3B
- added C20: .1uF, rcl:C0603
- added U4: LM1085ISX-5.0/NOPB, LM1085ISX:TS3B
- moved C10 2.29 mm to (31.0, 69.1)
- moved C18 2.29 mm to (31.0, 73.2)
- moved C8 2.29 mm to (31.0, 70.9)
Connections:
- net CSN3V3 renamed RADIO_CSN_3V3
- net ESTOPCONNECTED renamed ESTOP_CONNECTED
- net IRQ3V3 renamed RADIO_IRQ_3V3
- net MASTCONNECTED renamed MAST_CONNECTED
- net SS1_3V3 renamed SD_SS_3V3
- net SS2_3V3 renamed RADIO_SS_3V3
- net SS_SDCARD renamed SD_SS
- removed net CSN: U1.26, U6.10
- removed net IRQ: U1.25, U6.11
- removed net MISO: J2.1, U1.22, U2.10, U6.14
- removed net MISO3V3: J1.7, U2.5, U6.3, X3.MISO
- removed net MOSI: J2.4, U1.21, U2.11, U6.13
- removed net MOSI3V3: J1.2, U2.4, U6.4, X3.MOSI
- removed net SCK: J2.3, U1.20, U2.12, U6.12
- removed net SCK3V3: J1.5, U2.3, U6.5, X3.SCK
- removed net SS_RADIO: U1.24, U6.16
- new net PROGRAM_MISO: J2.1, U1.2
- new net PROGRAM_MOSI: J2.4, U1.3
- new net PROGRAM_SCK: J2.3, U1.4
- new net RADIO_CSN: U1.17, U6.10
- new net RADIO_IRQ: U1.16, U6.11
- new net RADIO_MISO: U1.12, U6.14
- new net RADIO_MISO_3V3: U6.3, X3.MISO
- new net RADIO_MOSI: U1.13, U6.13
- new net RADIO_MOSI_3V3: U6.4, X3.MOSI
- new net RADIO_SCK: U1.14, U6.12
- new net RADIO_SCK_3V3: U6.5, X3.SCK
- new net RADIO_SS: U1.15, U6.16
- new net SD_MISO: U1.22, U2.10
- new net SD_MISO_3V3: J1.7, U2.5
- new net SD_MOSI: U1.21, U2.11
- new net SD_MOSI_3V3: J1.2, U2.4
- new net SD_SCK: U1.20, U2.12
- new net SD_SCK_3V3: J1.5, U2.3
- net +12V: now also U4.3; no longer U7.3
- net +5V: now also C20.1, U4.2; no longer U7.2
- net GND: now also C20.2, U4.1; no longer J1.SH1, J1.SH2, U7.1
Routing:
- net SCK: track 74.3 -> 0.00 mm, vias 2 -> 0
- net MISO: track 72.9 -> 0.00 mm, vias 2 -> 0
- net MOSI: track 69.2 -> 0.00 mm, vias 2 -> 0
- net SCK3V3: track 34.5 -> 0.00 mm
- net PROGRAM_SCK: track 0.00 -> 33.6 mm
- net MISO3V3: track 33.3 -> 0.00 mm
- net PROGRAM_MISO: track 0.00 -> 33.0 mm
- net PROGRAM_MOSI: track 0.00 -> 30.2 mm
- net RADIO_SCK_3V3: track 0.00 -> 28.5 mm
- net MOSI3V3: track 28.2 -> 0.00 mm
- net SD_SCK: track 0.00 -> 26.4 mm
- net SD_MOSI: track 0.00 -> 25.5 mm
- net RADIO_CSN: track 0.00 -> 25.3 mm, vias 0 -> 2
- net RADIO_IRQ: track 0.00 -> 25.2 mm, vias 0 -> 2
- net RADIO_SCK: track 0.00 -> 24.9 mm, vias 0 -> 2
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Other:
- board text added: "LOGIC BOARD"
- board text added: "Programming"
- board text removed: "1"
