File: core-boards/diagnostics-main/Eagle Files/diagnostic-main.sch (EAGLE design)
At the start: 31 parts, among them J1 A118090TR-ND, J2 3M15451-ND, J3 B2PS-VH(LF)(SN), Q1 16 MHz, U1 ATMEGA2560-16AU, U2 296-38653-1-ND, U3 MCP2551T-I/SN, U4 LM1085ISX-5.0/NOPB, U5 LP2985IM5X-3.3/NOPB, U6 TXB0106PWR, X1 22-23-2031, X2 B6B-EH-A(LF)(SN), X5 22-23-2031, X8 WM4803-ND

Commit message: Internal Design Review Changes
Parts:
- removed C10, C9: 10uF, rcl:C-EUC0805
- removed C6: 2.2uF, rcl:C-EUC0603
- removed C7: .01uF, rcl:C-EUC0603
- removed C8: 1uF, rcl:C-EUC0603
- removed J3: B2PS-VH(LF)(SN), RoboJackets-Connectors:B2PS-VH(LF)(SN)
- removed U4: LM1085ISX-5.0/NOPB, LM1085ISX:LM1085ISX-5.0/NOPB
- removed U5: LP2985IM5X-3.3/NOPB, LP2985IM5X:LP2985IM5X-3.3/NOPB
- added C13: 2.2uF, rcl:C-EUC0603
- added C14: .01uF, rcl:C-EUC0603
- added C15: 1uF, rcl:C-EUC0603
- added C16, C17: 10uF, rcl:C-EUC0805
- added J4: B2PS-VH(LF)(SN), RoboJackets-Connectors:B2PS-VH(LF)(SN)
- added U7: LM1085ISX-5.0/NOPB, LM1085ISX:LM1085ISX-5.0/NOPB
- added U8: LP2985IM5X-3.3/NOPB, LP2985IM5X:LP2985IM5X-3.3/NOPB
Connections:
- removed net N$1: C7.1, U5.BP
- new net N$2: C14.1, U8.BP
- net +12V: now also C17.1, J4.2, U7.VIN; no longer C10.1, J3.2, U4.VIN
- net +3V3: now also C13.1, U8.VOUT; no longer C6.1, U5.VOUT
- net +5V: now also C15.1, C16.1, U7.VOUT, U8.ON, U8.VIN; no longer C8.1, C9.1, U4.VOUT, U5.ON, U5.VIN
- net CSN: now also U6.B6; no longer U6.B4
- net CSN3V3: now also U6.A6; no longer U6.A4
- net GND: now also C13.2, C14.2, C15.2, C16.2, C17.2, J4.1, U7.ADJ/GND, U8.GND; no longer C10.2, C6.2, C7.2, C8.2, C9.2, J3.1, U4.ADJ/GND, U5.GND
- net IRQ: now also U6.B5; no longer U6.B6
- net IRQ3V3: now also U6.A5; no longer U6.A6
- net MISO: now also U2.B4; no longer U2.B2
- net MISO3V3: now also U2.A4; no longer U2.A2
- net MOSI: now also U6.B3; no longer U6.B5
- net MOSI3V3: now also U6.A3; no longer U6.A5
- net SCK: now also U2.B2, U6.B4; no longer U2.B4, U6.B3
- net SCK3V3: now also U2.A2, U6.A4; no longer U2.A4, U6.A3
Other:
- moved on the sheet: C11, C12, C5, J1, R1, R3, U1, U2, U3, U6, X1-1, X1-2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

Commit message: Final Changes for design review
Parts:
- added D3: GREEN, SparkFun-LED:LED-BLUE0603
- added D4, D5: GREEN, SparkFun-LED:LED-GREEN0603
- added R18: 2.2k, rcl:R-US_R0603
- added R19, R21: 1k, rcl:R-US_R0603
- X3: value (none) -> CC1101
Connections:
- new net 12V_LED_R: D3.A, R18.1
- new net 3V3_LED_R: D5.A, R21.1
- new net 5V_LED_R: D4.A, R19.1
- net +12V: now also R18.2
- net +3V3: now also R21.2
- net +5V: now also R19.2
- net GND: now also D3.C, D4.C, D5.C
Other:
- note added: "Status Indicator LEDs"
Changed lines of the file:
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@@
 <part name="C5" library="rcl" library_urn="urn:adsk.eagle:library:334" deviceset="C-EU" device="C0603" package3d_urn="urn:adsk.eagle:package:23616/2" value=".1uF"/>
 <part name="X8" library="con-molex" library_urn="urn:adsk.eagle:library:165" deviceset="22-23-2051" device="" package3d_urn="urn:adsk.eagle:package:8078636/1" value="WM4803-ND"/>
-<part name="R2" library="rcl" library_urn="urn:adsk.eagle:library:334" deviceset="R-US_" device="R0402" package3d_urn="urn:adsk.eagle:package:23547/2" value="10k"/>
+<part name="R2" library="rcl" library_urn="urn:adsk.eagle:library:334" deviceset="R-US_" device="R0402" package3d_urn="urn:adsk.eagle:package:23547/3" value="10k"/>
 <part name="P+7" library="supply1" library_urn="urn:adsk.eagle:library:371" deviceset="+5V" device=""/>
 <part name="GND8" library="supply1" library_urn="urn:adsk.eagle:library:371" deviceset="GND" device=""/>
-<part name="R1" library="rcl" library_urn="urn:adsk.eagle:library:334" deviceset="R-US_" device="R0402" package3d_urn="urn:adsk.eagle:package:23547/2" value="120"/>
-<part name="R3" library="rcl" library_urn="urn:adsk.eagle:library:334" deviceset="R-US_" device="R0402" package3d_urn="urn:adsk.eagle:package:23547/2" value="120"/>
+<part name="R1" library="rcl" library_urn="urn:adsk.eagle:library:334" deviceset="R-US_" device="R0402" package3d_urn="urn:adsk.eagle:package:23547/3" value="120"/>
+<part name="R3" library="rcl" library_urn="urn:adsk.eagle:library:334" deviceset="R-US_" device="R0402" package3d_urn="urn:adsk.eagle:package:23547/3" value="120"/>
 <part name="GND9" library="supply1" library_urn="urn:adsk.eagle:library:371" deviceset="GND" device=""/>
 <part name="P+8" library="supply1" library_urn="urn:adsk.eagle:library:371" deviceset="+5V" device=""/>
@@
 <part name="X2" library="IGVC-Connector" deviceset="B6B-EH-A(LF)(SN)" device=""/>
 <part name="X1" library="con-molex" library_urn="urn:adsk.eagle:library:165" deviceset="22-23-2031" device="" package3d_urn="urn:adsk.eagle:package:8078634/1"/>
-<part name="X3" library="IGVC-Connector" deviceset="NRF24L01+PA+LNA" device="" package3d_urn="urn:adsk.eagle:package:22461/2"/>
+<part name="X3" library="IGVC-Connector" deviceset="NRF24L01+PA+LNA" device="" package3d_urn="urn:adsk.eagle:package:22461/2" value="CC1101 "/>
 <part name="+3V5" library="supply1" library_urn="urn:adsk.eagle:library:371" deviceset="+3V3" device=""/>
 <part name="GND17" library="supply1" library_urn="urn:adsk.eagle:library:371" deviceset="GND" device=""/>
@@
 <part name="FRAME4" library="RoboJackets-Frames" deviceset="FRAME_A_L" device=""/>
 <part name="FRAME5" library="RoboJackets-Frames" deviceset="FRAME_A_L" device=""/>
+<part name="D4" library="SparkFun-LED" library_urn="urn:adsk.eagle:library:529" deviceset="LED-GREEN" device="0603" package3d_urn="urn:adsk.eagle:package:39354/1" value="GREEN"/>
+<part name="D5" library="SparkFun-LED" library_urn="urn:adsk.eagle:library:529" deviceset="LED-GREEN" device="0603" package3d_urn="urn:adsk.eagle:package:39354/1" value="GREEN"/>
+<part name="D3" library="SparkFun-LED" library_urn="urn:adsk.eagle:library:529" deviceset="LED-BLUE" device="0603" package3d_urn="urn:adsk.eagle:package:39354/1" value="GREEN"/>
+<part name="R21" library="rcl" library_urn="urn:adsk.eagle:library:334" deviceset="R-US_" device="R0603" package3d_urn="urn:adsk.eagle:package:23555/3" value="1k"/>
+<part name="R19" library="rcl" library_urn="urn:adsk.eagle:library:334" deviceset="R-US_" device="R0603" package3d_urn="urn:adsk.eagle:package:23555/3" value="1k"/>
+<part name="R18" library="rcl" library_urn="urn:adsk.eagle:library:334" deviceset="R-US_" device="R0603" package3d_urn="urn:adsk.eagle:package:23555/3" value="2.2k"/>
+<part name="P+6" library="supply1" library_urn="urn:adsk.eagle:library:371" deviceset="+5V" device=""/>
+<part name="+3V4" library="supply1" library_urn="urn:adsk.eagle:library:371" deviceset="+3V3" device=""/>
+<part name="SUPPLY3" library="supply2" library_urn="urn:adsk.eagle:library:372" deviceset="V+" device="" value="+12V"/>
+<part name="GND10" library="supply1" library_urn="urn:adsk.eagle:library:371" deviceset="GND" device=""/>
 </parts>
 <sheets>
@@
 <wire x1="-86.36" y1="160.02" x2="-86.36" y2="185.42" width="0.1524" layer="97" style="shortdash"/>
 <text x="-83.82" y="180.34" size="1.778" layer="97">ISP Connector</text>
+<wire x1="-73.66" y1="152.4" x2="-20.32" y2="152.4" width="0.1524" layer="97" style="shortdash"/>
+<wire x1="-20.32" y1="152.4" x2="-20.32" y2="96.52" width="0.1524" layer="97" style="shortdash"/>
+<wire x1="-20.32" y1="96.52" x2="-73.66" y2="96.52" width="0.1524" layer="97" style="shortdash"/>
+<wire x1="-73.66" y1="96.52" x2="-73.66" y2="152.4" width="0.1524" layer="97" style="shortdash"/>
+<text x="-71.12" y="147.32" size="1.778" layer="97">Status Indicator LEDs</text>
 </plain>
 <instances>
@@
 <attribute name="SHEET" x="-40.64" y="-19.05" size="2.54" layer="94" font="vector"/>
 <attribute name="DRAWING_NAME" x="-111.76" y="-1.27" size="2.54" layer="94" font="vector"/>
+</instance>
+<instance part="D4" gate="G$1" x="-45.72" y="116.84" smashed="yes">
+<attribute name="NAME" x="-49.149" y="112.268" size="1.778" layer="95" font="vector" rot="R90"/>
+<attribute name="VALUE" x="-43.815" y="112.268" size="1.778" layer="96" font="vector" rot="R90" align="top-left"/>
+</instance>
+<instance part="D5" gate="G$1" x="-35.56" y="116.84" smashed="yes">
+<attribute name="NAME" x="-38.989" y="112.268" size="1.778" layer="95" font="vector" rot="R90"/>
+<attribute name="VALUE" x="-33.655" y="112.268" size="1.778" layer="96" font="vector" rot="R90" align="top-left"/>
+</instance>
+<instance part="D3" gate="G$1" x="-55.88" y="116.84" smashed="yes">
+<attribute name="NAME" x="-59.309" y="112.268" size="1.778" layer="95" font="vector" rot="R90"/>
+<attribute name="VALUE" x="-53.975" y="112.268" size="1.778" layer="96" font="vector" rot="R90" align="top-left"/>
+</instance>
+<instance part="R21" gate="G$1" x="-35.56" y="129.54" smashed="yes" rot="R90">
+<attribute name="NAME" x="-37.0586" y="125.73" size="1.778" layer="95" rot="R90"/>
+<attribute name="VALUE" x="-32.258" y="125.73" size="1.778" layer="96" rot="R90"/>
+</instance>
+<instance part="R19" gate="G$1" x="-45.72" y="129.54" smashed="yes" rot="R90">
+<attribute name="NAME" x="-47.2186" y="125.73" size="1.778" layer="95" rot="R90"/>
+<attribute name="VALUE" x="-42.418" y="125.73" size="1.778" layer="96" rot="R90"/>
+</instance>
+<instance part="R18" gate="G$1" x="-55.88" y="129.54" smashed="yes" rot="R90">
+<attribute name="NAME" x="-57.3786" y="125.73" size="1.778" layer="95" rot="R90"/>
+<attribute name="VALUE" x="-52.578" y="125.73" size="1.778" layer="96" rot="R90"/>
+</instance>
+<instance part="P+6" gate="1" x="-45.72" y="142.24" smashed="yes">
+<attribute name="VALUE" x="-48.26" y="137.16" size="1.778" layer="96" rot="R90"/>
+</instance>
+<instance part="+3V4" gate="G$1" x="-35.56" y="142.24" smashed="yes">
+<attribute name="VALUE" x="-38.1" y="137.16" size="1.778" layer="96" rot="R90"/>
+</instance>
+<instance part="SUPPLY3" gate="1" x="-55.88" y="142.24" smashed="yes">
+<attribute name="VALUE" x="-59.182" y="138.176" size="1.778" layer="96" rot="R90"/>
+</instance>
+<instance part="GND10" gate="1" x="-45.72" y="101.6" smashed="yes">
+<attribute name="VALUE" x="-48.26" y="99.06" size="1.778" layer="96"/>
 </instance>
 </instances>
@@
 <pinref part="GND7" gate="1" pin="GND"/>
 </segment>
+<segment>
+<pinref part="D3" gate="G$1" pin="C"/>
+<wire x1="-55.88" y1="111.76" x2="-55.88" y2="109.22" width="0.1524" layer="91"/>
+<wire x1="-55.88" y1="109.22" x2="-45.72" y2="109.22" width="0.1524" layer="91"/>
+<pinref part="D4" gate="G$1" pin="C"/>
+<wire x1="-45.72" y1="109.22" x2="-45.72" y2="111.76" width="0.1524" layer="91"/>
+<wire x1="-45.72" y1="109.22" x2="-35.56" y2="109.22" width="0.1524" layer="91"/>
+<junction x="-45.72" y="109.22"/>
+<pinref part="D5" gate="G$1" pin="C"/>
+<wire x1="-35.56" y1="109.22" x2="-35.56" y2="111.76" width="0.1524" layer="91"/>
+<pinref part="GND10" gate="1" pin="GND"/>
+<wire x1="-45.72" y1="109.22" x2="-45.72" y2="104.14" width="0.1524" layer="91"/>
+</segment>
 </net>
 <net name="!RESET" class="0">
@@
 <pinref part="P+5" gate="1" pin="+5V"/>
 </segment>
+<segment>
+<wire x1="-45.72" y1="139.7" x2="-45.72" y2="134.62" width="0.1524" layer="91"/>
+<pinref part="R19" gate="G$1" pin="2"/>
+<pinref part="P+6" gate="1" pin="+5V"/>
+</segment>
 </net>
 <net name="SS_SDCARD" class="0">
@@
 </segment>
 </net>
+<net name="5V_LED_R" class="0">
+<segment>
+<pinref part="D4" gate="G$1" pin="A"/>
+<wire x1="-45.72" y1="124.46" x2="-45.72" y2="119.38" width="0.1524" layer="91"/>
+<pinref part="R19" gate="G$1" pin="1"/>
+</segment>
+</net>
+<net name="3V3_LED_R" class="0">
+<segment>
+<pinref part="D5" gate="G$1" pin="A"/>
+<wire x1="-35.56" y1="124.46" x2="-35.56" y2="119.38" width="0.1524" layer="91"/>
+<pinref part="R21" gate="G$1" pin="1"/>
+</segment>
+</net>
+<net name="12V_LED_R" class="0">
+<segment>
+<pinref part="D3" gate="G$1" pin="A"/>
+<wire x1="-55.88" y1="124.46" x2="-55.88" y2="119.38" width="0.1524" layer="91"/>
+<pinref part="R18" gate="G$1" pin="1"/>
+</segment>
+</net>
+<net name="+3V3" class="0">
+<segment>
+<wire x1="-35.56" y1="139.7" x2="-35.56" y2="134.62" width="0.1524" layer="91"/>
+<pinref part="R21" gate="G$1" pin="2"/>
+<pinref part="+3V4" gate="G$1" pin="+3V3"/>
+</segment>
+</net>
+<net name="+12V" class="0">
+<segment>
+<wire x1="-55.88" y1="134.62" x2="-55.88" y2="139.7" width="0.1524" layer="91"/>
+<pinref part="R18" gate="G$1" pin="2"/>
+<pinref part="SUPPLY3" gate="1" pin="V+"/>
+</segment>
+</net>

Commit message: More small changes
Parts:
- removed D5: GREEN, SparkFun-LED:LED-GREEN0603
- added D1: GREEN, SparkFun-LED:LED-BLUE0603
- D3: device SparkFun-LED:LED-BLUE0603 -> SparkFun-LED:LED-GREEN0603
- renumbered D4 to D2, R18 to R4, R19 to R5, R21 to R6
Connections:
- net 12V_LED_R: now also D1.A; no longer D3.A
- net 3V3_LED_R: now also D3.A; no longer D5.A
- net GND: now also D1.C; no longer D5.C
Other:
- moved on the sheet: D3
Changed lines of the file:
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@@
 <part name="FRAME4" library="RoboJackets-Frames" deviceset="FRAME_A_L" device=""/>
 <part name="FRAME5" library="RoboJackets-Frames" deviceset="FRAME_A_L" device=""/>
-<part name="D4" library="SparkFun-LED" library_urn="urn:adsk.eagle:library:529" deviceset="LED-GREEN" device="0603" package3d_urn="urn:adsk.eagle:package:39354/1" value="GREEN"/>
-<part name="D5" library="SparkFun-LED" library_urn="urn:adsk.eagle:library:529" deviceset="LED-GREEN" device="0603" package3d_urn="urn:adsk.eagle:package:39354/1" value="GREEN"/>
-<part name="D3" library="SparkFun-LED" library_urn="urn:adsk.eagle:library:529" deviceset="LED-BLUE" device="0603" package3d_urn="urn:adsk.eagle:package:39354/1" value="GREEN"/>
-<part name="R21" library="rcl" library_urn="urn:adsk.eagle:library:334" deviceset="R-US_" device="R0603" package3d_urn="urn:adsk.eagle:package:23555/3" value="1k"/>
-<part name="R19" library="rcl" library_urn="urn:adsk.eagle:library:334" deviceset="R-US_" device="R0603" package3d_urn="urn:adsk.eagle:package:23555/3" value="1k"/>
-<part name="R18" library="rcl" library_urn="urn:adsk.eagle:library:334" deviceset="R-US_" device="R0603" package3d_urn="urn:adsk.eagle:package:23555/3" value="2.2k"/>
+<part name="D2" library="SparkFun-LED" library_urn="urn:adsk.eagle:library:529" deviceset="LED-GREEN" device="0603" package3d_urn="urn:adsk.eagle:package:39354/1" value="GREEN"/>
+<part name="D3" library="SparkFun-LED" library_urn="urn:adsk.eagle:library:529" deviceset="LED-GREEN" device="0603" package3d_urn="urn:adsk.eagle:package:39354/1" value="GREEN"/>
+<part name="D1" library="SparkFun-LED" library_urn="urn:adsk.eagle:library:529" deviceset="LED-BLUE" device="0603" package3d_urn="urn:adsk.eagle:package:39354/1" value="GREEN"/>
+<part name="R6" library="rcl" library_urn="urn:adsk.eagle:library:334" deviceset="R-US_" device="R0603" package3d_urn="urn:adsk.eagle:package:23555/3" value="1k"/>
+<part name="R5" library="rcl" library_urn="urn:adsk.eagle:library:334" deviceset="R-US_" device="R0603" package3d_urn="urn:adsk.eagle:package:23555/3" value="1k"/>
+<part name="R4" library="rcl" library_urn="urn:adsk.eagle:library:334" deviceset="R-US_" device="R0603" package3d_urn="urn:adsk.eagle:package:23555/3" value="2.2k"/>
 <part name="P+6" library="supply1" library_urn="urn:adsk.eagle:library:371" deviceset="+5V" device=""/>
 <part name="+3V4" library="supply1" library_urn="urn:adsk.eagle:library:371" deviceset="+3V3" device=""/>
@@
 <attribute name="DRAWING_NAME" x="-111.76" y="-1.27" size="2.54" layer="94" font="vector"/>
 </instance>
-<instance part="D4" gate="G$1" x="-45.72" y="116.84" smashed="yes">
+<instance part="D2" gate="G$1" x="-45.72" y="116.84" smashed="yes">
 <attribute name="NAME" x="-49.149" y="112.268" size="1.778" layer="95" font="vector" rot="R90"/>
 <attribute name="VALUE" x="-43.815" y="112.268" size="1.778" layer="96" font="vector" rot="R90" align="top-left"/>
 </instance>
-<instance part="D5" gate="G$1" x="-35.56" y="116.84" smashed="yes">
+<instance part="D3" gate="G$1" x="-35.56" y="116.84" smashed="yes">
 <attribute name="NAME" x="-38.989" y="112.268" size="1.778" layer="95" font="vector" rot="R90"/>
 <attribute name="VALUE" x="-33.655" y="112.268" size="1.778" layer="96" font="vector" rot="R90" align="top-left"/>
 </instance>
-<instance part="D3" gate="G$1" x="-55.88" y="116.84" smashed="yes">
+<instance part="D1" gate="G$1" x="-55.88" y="116.84" smashed="yes">
 <attribute name="NAME" x="-59.309" y="112.268" size="1.778" layer="95" font="vector" rot="R90"/>
 <attribute name="VALUE" x="-53.975" y="112.268" size="1.778" layer="96" font="vector" rot="R90" align="top-left"/>
 </instance>
-<instance part="R21" gate="G$1" x="-35.56" y="129.54" smashed="yes" rot="R90">
+<instance part="R6" gate="G$1" x="-35.56" y="129.54" smashed="yes" rot="R90">
 <attribute name="NAME" x="-37.0586" y="125.73" size="1.778" layer="95" rot="R90"/>
 <attribute name="VALUE" x="-32.258" y="125.73" size="1.778" layer="96" rot="R90"/>
 </instance>
-<instance part="R19" gate="G$1" x="-45.72" y="129.54" smashed="yes" rot="R90">
+<instance part="R5" gate="G$1" x="-45.72" y="129.54" smashed="yes" rot="R90">
 <attribute name="NAME" x="-47.2186" y="125.73" size="1.778" layer="95" rot="R90"/>
 <attribute name="VALUE" x="-42.418" y="125.73" size="1.778" layer="96" rot="R90"/>
 </instance>
-<instance part="R18" gate="G$1" x="-55.88" y="129.54" smashed="yes" rot="R90">
+<instance part="R4" gate="G$1" x="-55.88" y="129.54" smashed="yes" rot="R90">
 <attribute name="NAME" x="-57.3786" y="125.73" size="1.778" layer="95" rot="R90"/>
 <attribute name="VALUE" x="-52.578" y="125.73" size="1.778" layer="96" rot="R90"/>
@@
 </segment>
 <segment>
-<pinref part="D3" gate="G$1" pin="C"/>
+<pinref part="D1" gate="G$1" pin="C"/>
 <wire x1="-55.88" y1="111.76" x2="-55.88" y2="109.22" width="0.1524" layer="91"/>
 <wire x1="-55.88" y1="109.22" x2="-45.72" y2="109.22" width="0.1524" layer="91"/>
-<pinref part="D4" gate="G$1" pin="C"/>
+<pinref part="D2" gate="G$1" pin="C"/>
 <wire x1="-45.72" y1="109.22" x2="-45.72" y2="111.76" width="0.1524" layer="91"/>
 <wire x1="-45.72" y1="109.22" x2="-35.56" y2="109.22" width="0.1524" layer="91"/>
 <junction x="-45.72" y="109.22"/>
-<pinref part="D5" gate="G$1" pin="C"/>
+<pinref part="D3" gate="G$1" pin="C"/>
 <wire x1="-35.56" y1="109.22" x2="-35.56" y2="111.76" width="0.1524" layer="91"/>
 <pinref part="GND10" gate="1" pin="GND"/>
@@
 <segment>
 <wire x1="-45.72" y1="139.7" x2="-45.72" y2="134.62" width="0.1524" layer="91"/>
-<pinref part="R19" gate="G$1" pin="2"/>
+<pinref part="R5" gate="G$1" pin="2"/>
 <pinref part="P+6" gate="1" pin="+5V"/>
 </segment>
@@
 <net name="5V_LED_R" class="0">
 <segment>
-<pinref part="D4" gate="G$1" pin="A"/>
+<pinref part="D2" gate="G$1" pin="A"/>
 <wire x1="-45.72" y1="124.46" x2="-45.72" y2="119.38" width="0.1524" layer="91"/>
-<pinref part="R19" gate="G$1" pin="1"/>
+<pinref part="R5" gate="G$1" pin="1"/>
 </segment>
 </net>
 <net name="3V3_LED_R" class="0">
 <segment>
-<pinref part="D5" gate="G$1" pin="A"/>
+<pinref part="D3" gate="G$1" pin="A"/>
 <wire x1="-35.56" y1="124.46" x2="-35.56" y2="119.38" width="0.1524" layer="91"/>
-<pinref part="R21" gate="G$1" pin="1"/>
+<pinref part="R6" gate="G$1" pin="1"/>
 </segment>
 </net>
 <net name="12V_LED_R" class="0">
 <segment>
-<pinref part="D3" gate="G$1" pin="A"/>
+<pinref part="D1" gate="G$1" pin="A"/>
 <wire x1="-55.88" y1="124.46" x2="-55.88" y2="119.38" width="0.1524" layer="91"/>
-<pinref part="R18" gate="G$1" pin="1"/>
+<pinref part="R4" gate="G$1" pin="1"/>
 </segment>
 </net>
@@
 <segment>
 <wire x1="-35.56" y1="139.7" x2="-35.56" y2="134.62" width="0.1524" layer="91"/>
-<pinref part="R21" gate="G$1" pin="2"/>
+<pinref part="R6" gate="G$1" pin="2"/>
 <pinref part="+3V4" gate="G$1" pin="+3V3"/>
 </segment>
@@
 <segment>
 <wire x1="-55.88" y1="134.62" x2="-55.88" y2="139.7" width="0.1524" layer="91"/>
-<pinref part="R18" gate="G$1" pin="2"/>
+<pinref part="R4" gate="G$1" pin="2"/>
 <pinref part="SUPPLY3" gate="1" pin="V+"/>
 </segment>

Commit message: Final Changes for Design Review
Other:
- note removed: "ADD RADIO PART LABEL"
Changed lines of the file:
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@@
 <?xml version="1.0" encoding="utf-8"?>
 <!DOCTYPE eagle SYSTEM "eagle.dtd">
-<eagle version="9.2.2">
+<eagle version="9.5.2">
 <drawing>
 <settings>
@@
 <wire x1="-127" y1="185.42" x2="-127" y2="129.54" width="0.1524" layer="97" style="shortdash"/>
 <text x="-124.46" y="180.34" size="1.778" layer="97">Reset Line</text>
-<text x="-124.46" y="86.36" size="1.778" layer="97">External Clock Circuit</text>
+<text x="-124.46" y="88.9" size="1.778" layer="97">External Clock Circuit</text>
 <wire x1="-127" y1="91.44" x2="-127" y2="48.26" width="0.1524" layer="97" style="shortdash"/>
 <wire x1="-127" y1="48.26" x2="-81.28" y2="48.26" width="0.1524" layer="97" style="shortdash"/>
@@
 <wire x1="50.8" y1="248.92" x2="50.8" y2="279.4" width="0.1524" layer="97" style="shortdash"/>
 <text x="53.34" y="276.86" size="1.778" layer="97">Mast Board Connnector</text>
-<text x="20.32" y="142.24" size="1.778" layer="91">ADD RADIO PART LABEL</text>
 <wire x1="73.66" y1="190.5" x2="73.66" y2="137.16" width="0.1524" layer="97" style="shortdash"/>
 <wire x1="73.66" y1="137.16" x2="190.5" y2="137.16" width="0.1524" layer="97" style="shortdash"/>

Commit message: Design Review Changes
Parts:
- added C10, C21, C25, C6: 1uF, rcl:C-EUC0402
- added C18, C22, C26, C7: 10uF, rcl:C-EUC0805
- added C19, C23, C8, C9: .1uF, rcl:C-EUC0603
- C2: value .01uF -> .1uF
Connections:
- net +3V3: now also C2.1
- net +5V: now also C10.1, C18.1, C19.1, C21.1, C22.1, C23.1, C25.1, C26.1, C6.1, C7.1, C8.1, C9.1; no longer C2.1
- net GND: now also C10.2, C18.2, C19.2, C21.2, C22.2, C23.2, C25.2, C26.2, C6.2, C7.2, C8.2, C9.2
Other:
- moved on the sheet: C1, C3, C4, D1, D2, D3, Q1, R1, R3, R4, R5, R6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
