File: core-boards/diagnostics-main/Eagle Files/diagnostic-main.sch (EAGLE design)
At the start: 49 parts, among them J1 A118090TR-ND, J2 3M15451-ND, J4 B2PS-VH(LF)(SN), Q1 16 MHz, U1 ATMEGA2560-16AU, U2 296-38653-1-ND, U3 MCP2551T-I/SN, U6 TXB0106PWR, U7 LM1085ISX-5.0/NOPB, U8 LP2985IM5X-3.3/NOPB, X1 22-23-2031, X2 B6B-EH-A(LF)(SN), X3 CC1101, X5 22-23-2031, X8 WM4803-ND

Commit message: More changes
Changed lines of the file:
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@@
 <parts>
 <part name="U1" library="ATMEGA2560-16AU" deviceset="ATMEGA2560-16AU" device=""/>
-<part name="FRAME1" library="RoboJackets-Frames" deviceset="FRAME_B_L" device=""/>
 <part name="S1" library="RoboJackets-Switches" deviceset="KMR2" device=""/>
 <part name="GND1" library="supply1" library_urn="urn:adsk.eagle:library:371" deviceset="GND" device=""/>
@@
 <part name="C9" library="rcl" library_urn="urn:adsk.eagle:library:334" deviceset="C-EU" device="C0603" package3d_urn="urn:adsk.eagle:package:23616/2" value=".1uF"/>
 <part name="GND16" library="supply1" library_urn="urn:adsk.eagle:library:371" deviceset="GND" device=""/>
+<part name="P+12" library="supply1" library_urn="urn:adsk.eagle:library:371" deviceset="+12V" device=""/>
+<part name="GND27" library="supply1" library_urn="urn:adsk.eagle:library:371" deviceset="GND" device=""/>
 </parts>
 <sheets>
@@
 <wire x1="-81.28" y1="83.82" x2="-81.28" y2="127" width="0.1524" layer="97" style="shortdash"/>
 <wire x1="-127" y1="127" x2="-81.28" y2="127" width="0.1524" layer="97" style="shortdash"/>
-<wire x1="-127" y1="81.28" x2="-15.24" y2="81.28" width="0.1524" layer="97" style="shortdash"/>
-<wire x1="-15.24" y1="81.28" x2="-15.24" y2="25.4" width="0.1524" layer="97" style="shortdash"/>
-<wire x1="-15.24" y1="25.4" x2="-127" y2="25.4" width="0.1524" layer="97" style="shortdash"/>
+<wire x1="-127" y1="81.28" x2="-7.62" y2="81.28" width="0.1524" layer="97" style="shortdash"/>
+<wire x1="-7.62" y1="81.28" x2="-7.62" y2="25.4" width="0.1524" layer="97" style="shortdash"/>
+<wire x1="-7.62" y1="25.4" x2="-127" y2="25.4" width="0.1524" layer="97" style="shortdash"/>
 <wire x1="-127" y1="25.4" x2="-127" y2="81.28" width="0.1524" layer="97" style="shortdash"/>
 <text x="-124.46" y="76.2" size="1.778" layer="97">Decoupling Capicaitors</text>
@@
 <attribute name="VALUE" x="58.212809375" y="8.5187" size="2.08436875" layer="96" ratio="10" rot="SR0"/>
 </instance>
-<instance part="FRAME1" gate="G$2" x="187.96" y="-86.36" smashed="yes">
-<attribute name="LAST_DATE_TIME" x="200.66" y="-85.09" size="2.54" layer="94" font="vector"/>
-<attribute name="SHEET" x="274.32" y="-85.09" size="2.54" layer="94" font="vector"/>
-<attribute name="DRAWING_NAME" x="203.2" y="-67.31" size="2.54" layer="94" font="vector"/>
-<attribute name="SCH_DESC" x="189.23" y="-80.01" size="2.54" layer="94"/>
-</instance>
 <instance part="S1" gate="G$1" x="-104.14" y="147.32" smashed="yes" rot="R90">
 <attribute name="NAME" x="-107.95" y="142.24" size="2.54" layer="95" font="vector" rot="R90"/>
@@
 <attribute name="NAME" x="-69.596" y="38.481" size="1.778" layer="95"/>
 <attribute name="VALUE" x="-69.596" y="33.401" size="1.778" layer="96"/>
+</instance>
+<instance part="P+12" gate="1" x="-17.78" y="66.04" smashed="yes">
+<attribute name="VALUE" x="-15.24" y="71.12" size="1.778" layer="96" rot="R180"/>
+</instance>
+<instance part="GND27" gate="1" x="-17.78" y="48.26" smashed="yes">
+<attribute name="VALUE" x="-20.32" y="45.72" size="1.778" layer="96"/>
 </instance>
 </instances>
@@
 <pinref part="C26" gate="G$1" pin="2"/>
 </segment>
+<segment>
+<wire x1="-17.78" y1="53.34" x2="-17.78" y2="50.8" width="0.1524" layer="91"/>
+<pinref part="GND27" gate="1" pin="GND"/>
+</segment>
 </net>
 <net name="!RESET" class="0">
@@
 <pinref part="R4" gate="G$1" pin="2"/>
 <pinref part="SUPPLY3" gate="1" pin="V+"/>
+</segment>
+<segment>
+<wire x1="-17.78" y1="63.5" x2="-17.78" y2="60.96" width="0.1524" layer="91"/>
+<pinref part="P+12" gate="1" pin="+12V"/>
 </segment>
 </net>
@@
 <instance part="X3" gate="A" x="35.56" y="165.1" smashed="yes">
 <attribute name="NAME" x="21.59" y="173.355" size="1.778" layer="95"/>
-<attribute name="VALUE" x="21.59" y="157.48" size="1.778" layer="96"/>
+<attribute name="VALUE" x="29.21" y="157.48" size="1.778" layer="96"/>
 </instance>
 <instance part="+3V5" gate="G$1" x="48.26" y="175.26" smashed="yes">

Commit message: More Design Review Changes
Parts:
- added C20: .1uF, rcl:C-EUC0603
- renumbered U7 to U4
Connections:
- net CSN3V3 renamed RADIO_CSN_3V3
- net ESTOPCONNECTED renamed ESTOP_CONNECTED
- net IRQ3V3 renamed RADIO_IRQ_3V3
- net MASTCONNECTED renamed MAST_CONNECTED
- net SS1_3V3 renamed SD_SS_3V3
- net SS2_3V3 renamed RADIO_SS_3V3
- net SS_SDCARD renamed SD_SS
- removed net CSN: U1.(OC0A/OC1C/PCINT7)_PB7, U6.B6
- removed net IRQ: U1.(OC1B/PCINT6)_PB6, U6.B5
- removed net MISO: J2.1, U1.(MISO/PCINT3)_PB3, U2.B4, U6.B2
- removed net MISO3V3: J1.DAT0, U2.A4, U6.A2, X3.MISO
- removed net MOSI: J2.4, U1.(MOSI/PCINT2)_PB2, U2.B3, U6.B3
- removed net MOSI3V3: J1.CMD, U2.A3, U6.A3, X3.MOSI
- removed net SCK: J2.3, U1.(SCK/PCINT1)_PB1, U2.B2, U6.B4
- removed net SCK3V3: J1.CLK, U2.A2, U6.A4, X3.SCK
- removed net SS_RADIO: U1.(OC1A/PCINT5)_PB5, U6.B1
- new net PROGRAM_MISO: J2.1, U1.(RXD0/PCINT8)_PE0
- new net PROGRAM_MOSI: J2.4, U1.(TXD0)_PE1
- new net PROGRAM_SCK: J2.3, U1.(XCK0/AIN0)_PE2
- new net RADIO_CSN: U1.(OC4C)_PH5, U6.B6
- new net RADIO_IRQ: U1.(OC4B)_PH4, U6.B5
- new net RADIO_MISO: U1.(RXD2)_PH0, U6.B2
- new net RADIO_MISO_3V3: U6.A2, X3.MISO
- new net RADIO_MOSI: U1.(TXD2)_PH1, U6.B3
- new net RADIO_MOSI_3V3: U6.A3, X3.MOSI
- new net RADIO_SCK: U1.(XCK2)_PH2, U6.B4
- new net RADIO_SCK_3V3: U6.A4, X3.SCK
- new net RADIO_SS: U1.(OC4A)_PH3, U6.B1
- new net SD_MISO: U1.(MISO/PCINT3)_PB3, U2.B4
- new net SD_MISO_3V3: J1.DAT0, U2.A4
- new net SD_MOSI: U1.(MOSI/PCINT2)_PB2, U2.B3
- new net SD_MOSI_3V3: J1.CMD, U2.A3
- new net SD_SCK: U1.(SCK/PCINT1)_PB1, U2.B2
- new net SD_SCK_3V3: J1.CLK, U2.A2
- net +5V: now also C20.1
- net GND: now also C20.2; no longer J1.SHIELD
Other:
- note added: "CAN BUS"
- note removed: "CAN BUS CONNECTOR"
- moved on the sheet: C12, C2, R2, S1, U6

Commit message: Cleaning Up Parts Names and Part List
Still need to decide on connectors
Parts:
- removed C26: 10uF, rcl:C-EUC0805
- removed U8: LP2985IM5X-3.3/NOPB, LP2985IM5X:LP2985IM5X-3.3/NOPB
- added C24: .01uF, rcl:C-EUC0603
- added U5: LM1085ISX-5.0/NOPB, LM1085ISX:LM1085ISX-5.0/NOPB
- C1, C11, C2: value .1uF -> 10uF; device rcl:C-EUC0603 -> rcl:C-EUC0805
- C10, C21: value 1uF -> 10uF; device rcl:C-EUC0402 -> rcl:C-EUC0805
- C12, C5: value .1uF -> 1uF; device rcl:C-EUC0603 -> rcl:C-EUC0402
- C13: value 2.2uF -> 1uF; device rcl:C-EUC0603 -> rcl:C-EUC0402
- C14: value .01uF -> .1uF
- C15: value 1uF -> .1uF
- C16, C17, C18, C7: value 10uF -> .1uF; device rcl:C-EUC0805 -> rcl:C-EUC0603
- C23: value .1uF -> 1uF
- C25: value 1uF -> 2.2uF; device rcl:C-EUC0402 -> rcl:C-EUC0603
- J1: value A118090TR-ND -> 3M15451-ND; device A118090TR-ND:1939870-1 -> 3M15451-ND:30306-6002HB
- J2: value 3M15451-ND -> A118090TR-ND; device 3M15451-ND:30306-6002HB -> A118090TR-ND:1939870-1
- R1: value 120 -> 10k
- R2: value 10k -> 2.2k
- R3: value 120 -> 1k
- R4: value 2.2k -> 1k; device rcl:R-US_R0603 -> rcl:R-US_R0402
- R5, R6: value 1k -> 120; device rcl:R-US_R0603 -> rcl:R-US_R0402
- U3: value MCP2551T-I/SN -> TXB0106PWR; device MCP2551T:MCP2551T-I/SN -> TXB0106PWR:TXB0106PWR
- U4: value LM1085ISX-5.0/NOPB -> MCP2551T-I/SN; device LM1085ISX:LM1085ISX-5.0/NOPB -> MCP2551T:MCP2551T-I/SN
- U6: value TXB0106PWR -> LP2985IM5X-3.3/NOPB; device TXB0106PWR:TXB0106PWR -> LP2985IM5X:LP2985IM5X-3.3/NOPB
- X2: value B6B-EH-A(LF)(SN) -> CC1101; device IGVC-Connector:B6B-EH-A(LF)(SN) -> IGVC-Connector:NRF24L01+PA+LNA
- X3: value CC1101 -> 22-23-2031; device IGVC-Connector:NRF24L01+PA+LNA -> con-molex:22-23-2031
- X5: value 22-23-2031 -> B6B-EH-A(LF)(SN); device con-molex:22-23-2031 -> IGVC-Connector:B6B-EH-A(LF)(SN)
- renumbered J4 to J3, X8 to X4
Connections:
- net !RESET: now also J1.5, R1.1; no longer J2.5, R2.1
- net +12V: now also C21.1, R2.2, U5.VIN; no longer C17.1, R4.2, U4.VIN
- net +3V3: now also C16.1, C17.1, C18.1, C25.1, J2.VDD, R4.2, U3.OE, U3.VCCA, U6.VOUT, X2.VCC; no longer C11.1, C13.1, C2.1, C5.1, J1.VDD, R6.2, U6.OE, U6.VCCA, U8.VOUT, X3.VCC
- net +5V: now also C11.1, C13.1, C14.1, C2.1, C5.1, J1.2, R1.2, R3.2, U3.VCCB, U4.VDD, U5.VOUT, U6.ON, U6.VIN; no longer C16.1, C18.1, C21.1, C25.1, C26.1, J2.2, R2.2, R5.2, U3.VDD, U4.VOUT, U6.VCCB, U8.ON, U8.VIN
- net 12V_LED_R: now also R2.1; no longer R4.1
- net 3V3_LED_R: now also R4.1; no longer R6.1
- net 5V_LED_R: now also R3.1; no longer R5.1
- net CAN_N: now also R5.1, R6.1, U4.CANL, X3-2.S, X5.X-5; no longer R1.1, R3.1, U3.CANL, X2.X-5, X5-2.S
- net CAN_P: now also R5.2, R6.2, U4.CANH, X3-3.S, X5.X-6; no longer R1.2, R3.2, U3.CANH, X2.X-6, X5-3.S
- net CAN_RX: now also U4.TXD; no longer U3.TXD
- net CAN_TX: now also U4.RXD; no longer U3.RXD
- net DIAG_RX: now also X5.X-4; no longer X2.X-4
- net DIAG_TX: now also X5.X-3; no longer X2.X-3
- net ENCODER1_SENSE: now also X5.X-1; no longer X2.X-1
- net ENCODER2_SENSE: now also X5.X-2; no longer X2.X-2
- net GND: now also C24.2, J1.6, J2.VSS, U3.GND, U4.RS, U4.VSS, U5.ADJ/GND, X2.GND; no longer C26.2, J1.VSS, J2.6, U3.RS, U3.VSS, U4.ADJ/GND, U8.GND, X3.GND
- net MAST_CONNECTED: now also X3-1.S; no longer X5-1.S
- net N$2: now also C24.1, U6.BP; no longer C14.1, U8.BP
- net PROGRAM_MISO: now also J1.1; no longer J2.1
- net PROGRAM_MOSI: now also J1.4; no longer J2.4
- net PROGRAM_SCK: now also J1.3; no longer J2.3
- net RADIO_CSN: now also U3.B6; no longer U6.B6
- net RADIO_CSN_3V3: now also U3.A6, X2.CSN; no longer U6.A6, X3.CSN
- net RADIO_IRQ: now also U3.B5; no longer U6.B5
- net RADIO_IRQ_3V3: now also U3.A5, X2.IRQ; no longer U6.A5, X3.IRQ
- net RADIO_MISO: now also U3.B2; no longer U6.B2
- net RADIO_MISO_3V3: now also U3.A2, X2.MISO; no longer U6.A2, X3.MISO
- net RADIO_MOSI: now also U3.B3; no longer U6.B3
- net RADIO_MOSI_3V3: now also U3.A3, X2.MOSI; no longer U6.A3, X3.MOSI
- net RADIO_SCK: now also U3.B4; no longer U6.B4
- net RADIO_SCK_3V3: now also U3.A4, X2.SCK; no longer U6.A4, X3.SCK
- net RADIO_SS: now also U3.B1; no longer U6.B1
- net RADIO_SS_3V3: now also U3.A1, X2.CE; no longer U6.A1, X3.CE
- net SD_MISO_3V3: now also J2.DAT0; no longer J1.DAT0
- net SD_MOSI_3V3: now also J2.CMD; no longer J1.CMD
- net SD_SCK_3V3: now also J2.CLK; no longer J1.CLK
- net SD_SS_3V3: now also J2.CD/DAT3; no longer J1.CD/DAT3
- net XTAL1: now also C3.2; no longer C4.2
- net XTAL2: now also C4.2; no longer C3.2
