File: core-boards/hotswap/hotswap.brd (EAGLE design)
At the start: 92.7 x 56.8 mm, 19 parts, among them Q1 SUP75P03_07, Q2 SUP75P03_07, Q3 SUP75P03_07, U1 LTC4416EMS#PBF

Commit message: Yes
Parts:
- moved VCC_BATT 2.00 mm to (8.00, 7.00)
- moved U$1 1.00 mm to (8.00, 34.0)
- moved U$2 1.00 mm to (8.00, 21.0)
Routing:
- net VCC_WALL: track 29.2 -> 28.4 mm
Changed lines of the file:
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@@
 <?xml version="1.0" encoding="utf-8"?>
 <!DOCTYPE eagle SYSTEM "eagle.dtd">
-<eagle version="9.5.0">
+<eagle version="9.5.2">
 <drawing>
 <settings>
@@
 <text x="51.02" y="51.07" size="1.778" layer="25">RoboJackets IGVC
 Hotswap Board v.1.0</text>
-<text x="12.51" y="27.53" size="1.778" layer="25">GND</text>
+<text x="13.51" y="26.53" size="1.778" layer="25">GND</text>
 </plain>
 <attributes>
@@
 <attribute name="SPICEPREFIX" value="C" x="44.67" y="24.4" size="1.778" layer="27" display="off"/>
 </element>
-<element name="U$1" library="IGVC-Connector" package="6T4AWGLUG" value="6T4AWGLUG" x="8" y="35" smashed="yes"/>
-<element name="U$2" library="IGVC-Connector" package="6T4AWGLUG" value="6T4AWGLUG" x="8" y="22" smashed="yes"/>
-<element name="VCC_BATT" library="IGVC-Connector" package="6T4AWGLUG" value="6T4AWGLUG" x="8" y="9" smashed="yes"/>
+<element name="U$1" library="IGVC-Connector" package="6T4AWGLUG" value="6T4AWGLUG" x="8" y="34" smashed="yes"/>
+<element name="U$2" library="IGVC-Connector" package="6T4AWGLUG" value="6T4AWGLUG" x="8" y="21" smashed="yes"/>
+<element name="VCC_BATT" library="IGVC-Connector" package="6T4AWGLUG" value="6T4AWGLUG" x="8" y="7" smashed="yes"/>
 <element name="VCC_WALL" library="IGVC-Connector" package="6T4AWGLUG" value="6T4AWGLUG" x="8" y="48" smashed="yes"/>
 <element name="VCC_COMP" library="IGVC-Connector" package="6T4AWGLUG" value="6T4AWGLUG" x="84" y="35" smashed="yes" rot="R180"/>
@@
 <via x="43.4" y="49.8" extent="1-16" drill="0.4"/>
 <contactref element="C3" pad="2"/>
-<wire x1="39.21" y1="43.61" x2="39.21" y2="40.02" width="0.3" layer="1"/>
-<wire x1="39.21" y1="40.02" x2="47.21" y2="32.02" width="0.3" layer="1"/>
 <via x="47.21" y="32.02" extent="1-16" drill="0.4"/>
 <contactref element="U$1" pad="P$2"/>
@@
 <contactref element="VCC_COMP" pad="P$1"/>
 <polygon width="0.1524" layer="1" thermals="no">
-<vertex x="2" y="41"/>
-<vertex x="2" y="16"/>
-<vertex x="31" y="16"/>
-<vertex x="31" y="41"/>
+<vertex x="2" y="40"/>
+<vertex x="2" y="15"/>
+<vertex x="31" y="15"/>
+<vertex x="31" y="40"/>
 </polygon>
 <wire x1="68.35" y1="35" x2="80.5" y2="35" width="0.254" layer="1"/>
+<wire x1="39.21" y1="43.61" x2="39.21" y2="40.02" width="0.254" layer="1"/>
+<wire x1="39.21" y1="40.02" x2="47.21" y2="32.02" width="0.254" layer="1"/>
+<wire x1="54.7" y1="25.67" x2="68.35" y2="35" width="0" layer="19" extent="1-1"/>
+<wire x1="51.02" y1="29.099" x2="52.29" y2="25.67" width="0" layer="19" extent="1-1"/>
+<wire x1="47.21" y1="32.02" x2="48.8356" y2="29.48" width="0" layer="19" extent="1-1"/>
+<wire x1="45.94" y1="27.36" x2="48.8356" y2="29.48" width="0" layer="19" extent="1-1"/>
+<wire x1="47.21" y1="25.0576" x2="45.94" y2="27.36" width="0" layer="19" extent="1-1"/>
+<wire x1="40.99" y1="49.8" x2="39.21" y2="43.61" width="0" layer="19" extent="1-1"/>
+<wire x1="43.4" y1="18.05" x2="45.62" y2="24.4" width="0" layer="19" extent="1-1"/>
+<wire x1="23.65" y1="21" x2="40.99" y2="18.05" width="0" layer="19" extent="1-1"/>
+<wire x1="11.5" y1="21" x2="23.65" y2="21" width="0" layer="19" extent="1-1"/>
+<wire x1="23.65" y1="34" x2="23.65" y2="21" width="0" layer="19" extent="1-1"/>
+<wire x1="11.5" y1="34" x2="23.65" y2="34" width="0" layer="19" extent="1-1"/>
 </signal>
 <signal name="N$4">
@@
 <contactref element="VCC_WALL" pad="P$1"/>
 <polygon width="0.1524" layer="1" thermals="no">
-<vertex x="2" y="54"/>
+<vertex x="2" y="55"/>
 <vertex x="2" y="42"/>
 <vertex x="49" y="42"/>
-<vertex x="49" y="54"/>
+<vertex x="49" y="55"/>
 </polygon>
 <wire x1="49" y1="29.98038125" x2="48.8356" y2="29.98038125" width="0.254" layer="1"/>
 <wire x1="34.67" y1="45.14" x2="36" y2="43.81" width="0.254" layer="1"/>
-<wire x1="36" y1="43.81" x2="36" y2="40" width="0.254" layer="1"/>
-<wire x1="36" y1="40" x2="46.01961875" y2="29.98038125" width="0.254" layer="1"/>
-<wire x1="46.01961875" y1="29.98038125" x2="49" y2="29.98038125" width="0.254" layer="1"/>
+<wire x1="36" y1="43.81" x2="36" y2="41" width="0.254" layer="1"/>
+<wire x1="36" y1="41" x2="47.01961875" y2="29.98038125" width="0.254" layer="1"/>
+<wire x1="47.01961875" y1="29.98038125" x2="48.8356" y2="29.98038125" width="0.254" layer="1"/>
 </signal>
 <signal name="N$1">
@@
 <vertex x="91" y="27"/>
 <vertex x="91" y="1.54"/>
-<vertex x="49.75" y="1.54"/>
-<vertex x="49.75" y="54.88"/>
+<vertex x="50.75" y="1.54"/>
+<vertex x="50.75" y="54.88"/>
 </polygon>
 <contactref element="C5" pad="1"/>
@@
 <contactref element="VCC_BATT" pad="P$1"/>
 <polygon width="0.1524" layer="1" thermals="no">
-<vertex x="2" y="15"/>
-<vertex x="2" y="3"/>
-<vertex x="49" y="3"/>
+<vertex x="2" y="13"/>
+<vertex x="2" y="1"/>
+<vertex x="49" y="1"/>
 <vertex x="49" y="39"/>
 <vertex x="33" y="39"/>
-<vertex x="33" y="15"/>
+<vertex x="33" y="13"/>
 </polygon>
 </signal>

Commit message: Finish Optisolators
Parts:
- added J1: 2-PIN_2MM-V, RoboJackets-Connectors:2MM-2-V
- added Z1: TLP2745, IGVC-Discrete:TLP2745
Connections:
- new net N$2: J1.1, Z1.5
- new net VCC: Z1.4
- net GND: now also Z1.3, Z1.6
- net VCC_WALL: now also Z1.1
Routing:
- net GND: track 39.9 -> 221.9 mm, vias 7 -> 8
- net N$2: track 0.00 -> 30.6 mm
- net VCC_WALL: track 28.4 -> 41.0 mm
Other:
- board size 92.7 x 56.8 mm -> 92.7 x 62.8 mm
Changed lines of the file:
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@@
 <layer number="115" name="ReferenceISLANDS" color="7" fill="1" visible="no" active="yes"/>
 <layer number="116" name="Patch_BOT" color="9" fill="4" visible="no" active="yes"/>
+<layer number="117" name="BACKMAAT1" color="7" fill="1" visible="yes" active="yes"/>
 <layer number="118" name="Rect_Pads" color="7" fill="1" visible="no" active="yes"/>
+<layer number="119" name="KAP_TEKEN" color="7" fill="1" visible="yes" active="yes"/>
+<layer number="120" name="KAP_MAAT1" color="7" fill="1" visible="yes" active="yes"/>
 <layer number="121" name="_tsilk" color="7" fill="1" visible="no" active="yes"/>
 <layer number="122" name="_bsilk" color="7" fill="1" visible="no" active="yes"/>
@@
 <layer number="128" name="_bValues" color="7" fill="1" visible="no" active="yes"/>
 <layer number="129" name="Mask" color="7" fill="1" visible="no" active="yes"/>
+<layer number="130" name="SMDSTROOK" color="7" fill="1" visible="yes" active="yes"/>
 <layer number="131" name="tAdjust" color="7" fill="1" visible="no" active="yes"/>
 <layer number="132" name="bAdjust" color="7" fill="1" visible="no" active="yes"/>
@@
 <layer number="230" name="230bmp" color="7" fill="1" visible="no" active="yes"/>
 <layer number="231" name="231bmp" color="7" fill="1" visible="no" active="yes"/>
+<layer number="232" name="Eagle3D_PG2" color="7" fill="1" visible="yes" active="yes"/>
+<layer number="233" name="Eagle3D_PG3" color="7" fill="1" visible="yes" active="yes"/>
 <layer number="248" name="Housing" color="7" fill="1" visible="no" active="yes"/>
 <layer number="249" name="Edge" color="7" fill="1" visible="no" active="yes"/>
@@
 <plain>
 <wire x1="0" y1="0.27" x2="92.67" y2="0.27" width="0" layer="20"/>
-<wire x1="92.67" y1="0.27" x2="92.67" y2="57.09" width="0" layer="20"/>
-<wire x1="92.67" y1="57.09" x2="0" y2="57.09" width="0" layer="20"/>
-<wire x1="0" y1="57.09" x2="0" y2="0.27" width="0" layer="20"/>
+<wire x1="92.67" y1="0.27" x2="92.67" y2="63.09" width="0" layer="20"/>
+<wire x1="92.67" y1="63.09" x2="0" y2="63.09" width="0" layer="20"/>
+<wire x1="0" y1="63.09" x2="0" y2="0.27" width="0" layer="20"/>
 <text x="30.51" y="51.53" size="1.778" layer="25" rot="R270">WALL</text>
 <text x="37.78" y="23.51" size="1.778" layer="25" rot="R90">BATTERY</text>
@@
 <element name="VCC_COMP" library="IGVC-Connector" package="6T4AWGLUG" value="6T4AWGLUG" x="84" y="35" smashed="yes" rot="R180"/>
 <element name="U$6" library="IGVC-Connector" package="6T4AWGLUG" value="6T4AWGLUG" x="84" y="20" smashed="yes" rot="R180"/>
+<element name="Z1" library="IGVC-Discrete" package="TLP2745" value="TLP2745" x="50" y="59" smashed="yes"/>
+<element name="J1" library="RoboJackets-Connectors" package="2MM-2-V" value="2-PIN_2MM-V" x="86" y="59" smashed="yes">
+<attribute name="NAME" x="82" y="62.5" size="1" layer="25" font="vector"/>
+<attribute name="PINS" value="2" x="86" y="59" size="1.778" layer="27" display="off"/>
+<attribute name="PIN_PITCH" value="2.0 mm" x="86" y="59" size="1.778" layer="27" display="off"/>
+</element>
 </elements>
 <signals>
 <signal name="GND">
 <polygon width="0.254" layer="16" thermals="no">
-<vertex x="-0.127" y="57.039"/>
-<vertex x="92.563" y="57.039"/>
+<vertex x="-0.127" y="63.039"/>
+<vertex x="92.563" y="63.039"/>
 <vertex x="92.563" y="-0.111"/>
 <vertex x="-0.127" y="-0.111"/>
@@
 <wire x1="39.21" y1="43.61" x2="39.21" y2="40.02" width="0.254" layer="1"/>
 <wire x1="39.21" y1="40.02" x2="47.21" y2="32.02" width="0.254" layer="1"/>
-<wire x1="54.7" y1="25.67" x2="68.35" y2="35" width="0" layer="19" extent="1-1"/>
-<wire x1="51.02" y1="29.099" x2="52.29" y2="25.67" width="0" layer="19" extent="1-1"/>
-<wire x1="47.21" y1="32.02" x2="48.8356" y2="29.48" width="0" layer="19" extent="1-1"/>
-<wire x1="45.94" y1="27.36" x2="48.8356" y2="29.48" width="0" layer="19" extent="1-1"/>
-<wire x1="47.21" y1="25.0576" x2="45.94" y2="27.36" width="0" layer="19" extent="1-1"/>
-<wire x1="40.99" y1="49.8" x2="39.21" y2="43.61" width="0" layer="19" extent="1-1"/>
-<wire x1="43.4" y1="18.05" x2="45.62" y2="24.4" width="0" layer="19" extent="1-1"/>
-<wire x1="23.65" y1="21" x2="40.99" y2="18.05" width="0" layer="19" extent="1-1"/>
-<wire x1="11.5" y1="21" x2="23.65" y2="21" width="0" layer="19" extent="1-1"/>
-<wire x1="23.65" y1="34" x2="23.65" y2="21" width="0" layer="19" extent="1-1"/>
-<wire x1="11.5" y1="34" x2="23.65" y2="34" width="0" layer="19" extent="1-1"/>
+<contactref element="Z1" pad="6"/>
+<contactref element="Z1" pad="3"/>
+<via x="42" y="57" extent="1-16" drill="0.381"/>
+<polygon width="0.1524" layer="16">
+<vertex x="0" y="63"/>
+<vertex x="0" y="0"/>
+<vertex x="92" y="0"/>
+<vertex x="92" y="63"/>
+</polygon>
+<wire x1="42" y1="57" x2="42.73" y2="57.73" width="0.254" layer="1"/>
+<wire x1="42.73" y1="57.73" x2="45.625" y2="57.73" width="0.254" layer="1"/>
+<wire x1="23.65" y1="34" x2="25.63" y2="32.02" width="0.254" layer="16"/>
+<wire x1="25.63" y1="32.02" x2="36" y2="32.02" width="0.254" layer="16"/>
+<wire x1="36" y1="32.02" x2="39" y2="32.02" width="0.254" layer="16"/>
+<wire x1="39" y1="32.02" x2="44" y2="32.02" width="0.254" layer="16"/>
+<wire x1="44" y1="32.02" x2="47.21" y2="32.02" width="0.254" layer="16"/>
+<wire x1="23.65" y1="21" x2="33" y2="21" width="0.254" layer="16"/>
+<wire x1="33" y1="21" x2="40.45" y2="21" width="0.254" layer="16"/>
+<wire x1="40.45" y1="21" x2="43.4" y2="18.05" width="0.254" layer="16"/>
+<wire x1="47.21" y1="25.0576" x2="37.0576" y2="25.0576" width="0.254" layer="16"/>
+<wire x1="37.0576" y1="25.0576" x2="33" y2="21" width="0.254" layer="16"/>
+<wire x1="39" y1="32.02" x2="43.4" y2="36.42" width="0.254" layer="16"/>
+<wire x1="43.4" y1="36.42" x2="43.4" y2="49.8" width="0.254" layer="16"/>
+<wire x1="42" y1="57" x2="36" y2="51" width="0.254" layer="16"/>
+<wire x1="36" y1="51" x2="36" y2="32.02" width="0.254" layer="16"/>
+<wire x1="52.29" y1="25.67" x2="59.02" y2="25.67" width="0.254" layer="16"/>
+<wire x1="59.02" y1="25.67" x2="62.175" y2="28.825" width="0.254" layer="16"/>
+<wire x1="62.175" y1="28.825" x2="62.449" y2="29.099" width="0.254" layer="16"/>
+<wire x1="62.449" y1="29.099" x2="68.35" y2="35" width="0.254" layer="16"/>
+<wire x1="51.02" y1="29.099" x2="62.449" y2="29.099" width="0.254" layer="16"/>
+<wire x1="44.67" y1="26.94" x2="44" y2="27.61" width="0.254" layer="16"/>
+<wire x1="44" y1="27.61" x2="44" y2="32.02" width="0.254" layer="16"/>
+<wire x1="23.65" y1="34" x2="11.5" y2="34" width="0.254" layer="1"/>
+<wire x1="23.65" y1="21" x2="11.5" y2="21" width="0.254" layer="1"/>
+<wire x1="45.625" y1="57.73" x2="54.375" y2="57.73" width="0.254" layer="1"/>
+<wire x1="62.175" y1="28.825" x2="62.175" y2="28.825" width="0.254" layer="16"/>
 </signal>
 <signal name="N$4">
@@
 <wire x1="54.06038125" y1="29.98038125" x2="54.83" y2="30.75" width="0.254" layer="1"/>
 <via x="54.83" y="30.75" extent="1-16" drill="0.4"/>
-<wire x1="53.2044" y1="29.98038125" x2="49" y2="29.98038125" width="0.254" layer="1"/>
+<wire x1="53.2044" y1="29.98038125" x2="48.8356" y2="29.98038125" width="0.254" layer="1"/>
 <contactref element="C1" pad="1"/>
 <contactref element="C4" pad="1"/>
@@
 <vertex x="49" y="55"/>
 </polygon>
-<wire x1="49" y1="29.98038125" x2="48.8356" y2="29.98038125" width="0.254" layer="1"/>
 <wire x1="34.67" y1="45.14" x2="36" y2="43.81" width="0.254" layer="1"/>
 <wire x1="36" y1="43.81" x2="36" y2="41" width="0.254" layer="1"/>
 <wire x1="36" y1="41" x2="47.01961875" y2="29.98038125" width="0.254" layer="1"/>
 <wire x1="47.01961875" y1="29.98038125" x2="48.8356" y2="29.98038125" width="0.254" layer="1"/>
+<contactref element="Z1" pad="1"/>
+<wire x1="45.625" y1="60.27" x2="43.27" y2="60.27" width="0.254" layer="1"/>
+<wire x1="43.27" y1="60.27" x2="36" y2="53" width="0.254" layer="1"/>
 </signal>
 <signal name="N$1">
@@
 <wire x1="34.67" y1="40.33" x2="34.67" y2="43.44" width="0.254" layer="1"/>
 </signal>
+<signal name="VCC">
+<contactref element="Z1" pad="4"/>
+</signal>
+<signal name="N$2">
+<contactref element="Z1" pad="5"/>
+<contactref element="J1" pad="1"/>
+<wire x1="54.375" y1="59" x2="85" y2="59" width="0.254" layer="1"/>
+</signal>
 </signals>

Commit message: Update hotswap.brd
Parts:
- moved J1 21.0 mm to (65.0, 59.0)
Routing:
- net N$2: track 30.6 -> 9.62 mm
Changed lines of the file:
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@@
 <element name="U$6" library="IGVC-Connector" package="6T4AWGLUG" value="6T4AWGLUG" x="84" y="20" smashed="yes" rot="R180"/>
 <element name="Z1" library="IGVC-Discrete" package="TLP2745" value="TLP2745" x="50" y="59" smashed="yes"/>
-<element name="J1" library="RoboJackets-Connectors" package="2MM-2-V" value="2-PIN_2MM-V" x="86" y="59" smashed="yes">
-<attribute name="NAME" x="82" y="62.5" size="1" layer="25" font="vector"/>
-<attribute name="PINS" value="2" x="86" y="59" size="1.778" layer="27" display="off"/>
-<attribute name="PIN_PITCH" value="2.0 mm" x="86" y="59" size="1.778" layer="27" display="off"/>
+<element name="J1" library="RoboJackets-Connectors" package="2MM-2-V" value="2-PIN_2MM-V" x="65" y="59" smashed="yes">
+<attribute name="NAME" x="61" y="62.5" size="1" layer="25" font="vector"/>
+<attribute name="PINS" value="2" x="65" y="59" size="1.778" layer="27" display="off"/>
+<attribute name="PIN_PITCH" value="2.0 mm" x="65" y="59" size="1.778" layer="27" display="off"/>
 </element>
 </elements>
@@
 <contactref element="Z1" pad="5"/>
 <contactref element="J1" pad="1"/>
-<wire x1="54.375" y1="59" x2="85" y2="59" width="0.254" layer="1"/>
+<wire x1="54.375" y1="59" x2="64" y2="59" width="0.254" layer="1"/>
 </signal>
 </signals>

Commit message: Finishing touches to the board
Routing:
- net GND: track 221.9 -> 99.3 mm, vias 8 -> 11
- net VCC_WALL: track 41.0 -> 43.0 mm
Changed lines of the file:
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@@
 Hotswap Board v.1.0</text>
 <text x="13.51" y="26.53" size="1.778" layer="25">GND</text>
+<dimension x1="93" y1="63" x2="90" y2="0" x3="97" y3="31.5" textsize="1.778" layer="1" dtype="vertical"/>
+<dimension x1="0" y1="63" x2="93" y2="61" x3="46.5" y3="67" textsize="1.778" layer="1" dtype="horizontal"/>
 </plain>
 <attributes>
@@
 <vertex x="0" y="63"/>
 <vertex x="0" y="0"/>
-<vertex x="92" y="0"/>
-<vertex x="92" y="63"/>
+<vertex x="93" y="0"/>
+<vertex x="93" y="63"/>
 </polygon>
 <wire x1="42" y1="57" x2="42.73" y2="57.73" width="0.254" layer="1"/>
 <wire x1="42.73" y1="57.73" x2="45.625" y2="57.73" width="0.254" layer="1"/>
-<wire x1="23.65" y1="34" x2="25.63" y2="32.02" width="0.254" layer="16"/>
-<wire x1="25.63" y1="32.02" x2="36" y2="32.02" width="0.254" layer="16"/>
-<wire x1="36" y1="32.02" x2="39" y2="32.02" width="0.254" layer="16"/>
-<wire x1="39" y1="32.02" x2="44" y2="32.02" width="0.254" layer="16"/>
-<wire x1="44" y1="32.02" x2="47.21" y2="32.02" width="0.254" layer="16"/>
-<wire x1="23.65" y1="21" x2="33" y2="21" width="0.254" layer="16"/>
-<wire x1="33" y1="21" x2="40.45" y2="21" width="0.254" layer="16"/>
-<wire x1="40.45" y1="21" x2="43.4" y2="18.05" width="0.254" layer="16"/>
-<wire x1="47.21" y1="25.0576" x2="37.0576" y2="25.0576" width="0.254" layer="16"/>
-<wire x1="37.0576" y1="25.0576" x2="33" y2="21" width="0.254" layer="16"/>
-<wire x1="39" y1="32.02" x2="43.4" y2="36.42" width="0.254" layer="16"/>
-<wire x1="43.4" y1="36.42" x2="43.4" y2="49.8" width="0.254" layer="16"/>
-<wire x1="42" y1="57" x2="36" y2="51" width="0.254" layer="16"/>
-<wire x1="36" y1="51" x2="36" y2="32.02" width="0.254" layer="16"/>
-<wire x1="52.29" y1="25.67" x2="59.02" y2="25.67" width="0.254" layer="16"/>
-<wire x1="59.02" y1="25.67" x2="62.175" y2="28.825" width="0.254" layer="16"/>
-<wire x1="62.175" y1="28.825" x2="62.449" y2="29.099" width="0.254" layer="16"/>
-<wire x1="62.449" y1="29.099" x2="68.35" y2="35" width="0.254" layer="16"/>
-<wire x1="51.02" y1="29.099" x2="62.449" y2="29.099" width="0.254" layer="16"/>
-<wire x1="44.67" y1="26.94" x2="44" y2="27.61" width="0.254" layer="16"/>
-<wire x1="44" y1="27.61" x2="44" y2="32.02" width="0.254" layer="16"/>
 <wire x1="23.65" y1="34" x2="11.5" y2="34" width="0.254" layer="1"/>
 <wire x1="23.65" y1="21" x2="11.5" y2="21" width="0.254" layer="1"/>
 <wire x1="45.625" y1="57.73" x2="54.375" y2="57.73" width="0.254" layer="1"/>
-<wire x1="62.175" y1="28.825" x2="62.175" y2="28.825" width="0.254" layer="16"/>
+<via x="26" y="28" extent="1-16" drill="0.381"/>
+<via x="21" y="27" extent="1-16" drill="0.381"/>
+<wire x1="23.65" y1="34" x2="26" y2="31.65" width="0.254" layer="1"/>
+<wire x1="26" y1="31.65" x2="26" y2="28" width="0.254" layer="1"/>
+<wire x1="23.65" y1="21" x2="23.65" y2="26.35" width="0.254" layer="1"/>
+<wire x1="23.65" y1="26.35" x2="23" y2="27" width="0.254" layer="1"/>
+<wire x1="23" y1="27" x2="21" y2="27" width="0.254" layer="1"/>
+<via x="68" y="28" extent="1-16" drill="0.381"/>
+<wire x1="68.35" y1="35" x2="68.35" y2="28.35" width="0.254" layer="1"/>
+<wire x1="68.35" y1="28.35" x2="68" y2="28" width="0.254" layer="1"/>
 </signal>
 <signal name="N$4">
@@
 <wire x1="47.01961875" y1="29.98038125" x2="48.8356" y2="29.98038125" width="0.254" layer="1"/>
 <contactref element="Z1" pad="1"/>
-<wire x1="45.625" y1="60.27" x2="43.27" y2="60.27" width="0.254" layer="1"/>
-<wire x1="43.27" y1="60.27" x2="36" y2="53" width="0.254" layer="1"/>
+<wire x1="41.27" y1="60.27" x2="34" y2="53" width="0.254" layer="1"/>
+<wire x1="45.625" y1="60.27" x2="41.27" y2="60.27" width="0.254" layer="1"/>
 </signal>
 <signal name="N$1">

Commit message: Minor tweaks
Connections:
- net VCC_COMP renamed VCC_ROBOT
Routing:
- net GND: track 99.3 -> 100.7 mm
Other:
- board text added: "ROBOT"
- board text removed: "COMPUTER"
Changed lines of the file:
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@@
 <text x="30.51" y="51.53" size="1.778" layer="25" rot="R270">WALL</text>
 <text x="37.78" y="23.51" size="1.778" layer="25" rot="R90">BATTERY</text>
-<text x="56.91" y="42.56" size="1.778" layer="25" rot="R270">COMPUTER
+<text x="56.91" y="39.56" size="1.778" layer="25" rot="R270">ROBOT
 </text>
 <text x="51.02" y="51.07" size="1.778" layer="25">RoboJackets IGVC
@@
 <wire x1="23.65" y1="26.35" x2="23" y2="27" width="0.254" layer="1"/>
 <wire x1="23" y1="27" x2="21" y2="27" width="0.254" layer="1"/>
-<via x="68" y="28" extent="1-16" drill="0.381"/>
-<wire x1="68.35" y1="35" x2="68.35" y2="28.35" width="0.254" layer="1"/>
-<wire x1="68.35" y1="28.35" x2="68" y2="28" width="0.254" layer="1"/>
+<via x="65" y="29" extent="1-16" drill="0.381"/>
+<wire x1="68.35" y1="35" x2="68.35" y2="30.35" width="0.254" layer="1"/>
+<wire x1="68.35" y1="30.35" x2="67" y2="29" width="0.254" layer="1"/>
+<wire x1="67" y1="29" x2="65" y2="29" width="0.254" layer="1"/>
 </signal>
 <signal name="N$4">
@@
 <wire x1="45.66" y1="14.679" x2="45.66" y2="10.17" width="0.254" layer="1"/>
 </signal>
-<signal name="VCC_COMP">
+<signal name="VCC_ROBOT">
 <contactref element="U1" pad="8"/>
 <polygon width="0.254" layer="1" thermals="no">
