File: core-boards/estop/Eagle Files/estop_tx.sch (EAGLE design)
At the start: 29 parts, among them J1 RFM95W-3072, J2 JST-XH-02-PIN-ROUND-PAD, J3 JST-XH-02-PIN-ROUND-PAD, J4 JST-XH-02-PIN-ROUND-PAD, J5 JST-XH-02-PIN-ROUND-PAD, J6 B2PS-VH(LF)(SN), U1 R-78E5.0-1.0CONV_R-78E5.0-1.0, U2 TXB0106PWR, U4 ATMEGA328P-AUR

Commit message: estop tx design review
Parts:
- added D4: Green, SparkFun-LED:LED-YELLOW0603
- added R7: 10k, rcl:R-US_R0603
- C6: device resistor:C-USC0603 -> rcl:C-USC0603
- R2: value 10k -> 1k
- R3: value 60k -> 10k
- R4, R5, R6: device resistor:R-US_R0603 -> rcl:R-US_R0603
Connections:
- new net BUTTON_LED_CONN: J5-1.S, U2.A2
- new net N$5: D4.C, R2.1
- new net WIRELESS_LED_CONN: J4-1.S, U2.A1
- net !RESET: now also R3.2; no longer R2.1
- net +3V3: now also D4.A, U2.OE
- net +5V: now also D1.A, R3.1; no longer D2.A, R2.2
- net BUTTON_LED: now also D3.A; no longer D1.A, J5-1.S, U2.A2
- net CE: now also U4.(PCINT2/SS/OC1B)_PB2; no longer U4.(PCINT6/XTAL1/TOSC1)_PB6
- net GND: now also R2.2, R4.2, R5.2, R6.2, R7.2; no longer J1.RST, R3.1, R4.1, R5.1, R6.1
- net N$2: now also D1.C, R4.1; no longer D2.C, R5.2
- net N$3: now also D3.C, R6.1; no longer D1.C, R4.2
- net N$4: now also D2.C, R5.1; no longer D3.C, R6.2
- net N$6: now also J1.RST, R7.1; no longer R3.2, U2.OE
- net WIRELESS_LED: now also D2.A; no longer D3.A, J4-1.S, U2.A1
Other:
- note added: "LED Connectors"
- note added: "Level Shifter (5V -> 3V3)"
- moved on the sheet: C1, C2, C3, C5, C6, C7, C8, D1, D2, D3, J3-1, J6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

Commit message: final tm edits for design review
Other:
- note added: "Button Input"
- note removed: "3.3V Button IN"
Changed lines of the file:
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@@
 <text x="421.64" y="289.56" size="3.81" layer="103" font="vector">Power LED</text>
 <text x="264.16" y="287.02" size="3.81" layer="103" font="vector">Microcontroller</text>
-<text x="345.44" y="350.52" size="5.08" layer="95" font="vector">Power</text>
+<text x="345.44" y="350.52" size="3.81" layer="99" font="vector">Power</text>
 <wire x1="424.18" y1="414.02" x2="424.18" y2="365.76" width="0.1524" layer="103" style="shortdash"/>
 <wire x1="424.18" y1="365.76" x2="502.92" y2="365.76" width="0.1524" layer="103" style="shortdash"/>
 <wire x1="502.92" y1="365.76" x2="502.92" y2="414.02" width="0.1524" layer="103" style="shortdash"/>
 <wire x1="502.92" y1="414.02" x2="424.18" y2="414.02" width="0.1524" layer="103" style="shortdash"/>
-<text x="429.26" y="406.4" size="5.08" layer="103" font="vector">3.3V Button IN</text>
-<text x="261.62" y="345.44" size="5.08" layer="103" font="vector">Reset Button</text>
+<text x="261.62" y="345.44" size="3.81" layer="103" font="vector">Reset Button</text>
 <wire x1="462.28" y1="254" x2="462.28" y2="215.9" width="0.1524" layer="103" style="shortdash"/>
 <wire x1="419.1" y1="215.9" x2="419.1" y2="254" width="0.1524" layer="103" style="shortdash"/>
@@
 <wire x1="467.36" y1="297.18" x2="510.54" y2="297.18" width="0.1524" layer="103" style="shortdash"/>
 <text x="469.9" y="289.56" size="3.81" layer="103" font="vector">Wireless LED</text>
-<text x="261.62" y="403.86" size="5.08" layer="97" font="vector">Radio Board</text>
+<text x="261.62" y="403.86" size="3.81" layer="97" font="vector">Radio Board</text>
 <wire x1="259.08" y1="411.48" x2="259.08" y2="355.6" width="0.1524" layer="97" style="shortdash"/>
 <wire x1="259.08" y1="411.48" x2="332.74" y2="411.48" width="0.1524" layer="97" style="shortdash"/>
@@
 <wire x1="419.1" y1="215.9" x2="462.28" y2="215.9" width="0.1524" layer="97" style="shortdash"/>
 <text x="510.54" y="411.48" size="3.81" layer="97">LED Connectors</text>
+<text x="426.72" y="406.4" size="3.81" layer="97">Button Input</text>
 </plain>
 <instances>

Commit message: almost order ready haha
Parts:
- removed J2: JST-XH-02-PIN-ROUND-PAD, IGVC-Connector:JST-XH-02-PIN-ROUND-PAD
- added J7: 2-PIN_2MM-V, RoboJackets-Connectors:2-PIN_2MM-V
- added R10, R8, R9: 200, rcl:R-US_R0603
- added R11: 10k, rcl:R-US_R0603
- J3, J4, J5: value JST-XH-02-PIN-ROUND-PAD -> 2-PIN_2MM-V; device IGVC-Connector:JST-XH-02-PIN-ROUND-PAD -> RoboJackets-Connectors:2-PIN_2MM-V
Connections:
- new net N$1: J3.1, R8.1
- new net N$10: J1.EN, R11.1
- new net N$7: J4.1, R9.1
- new net N$8: J5.1, R10.1
- net +3V3: now also R8.2; no longer J3-1.S
- net +5V: now also R11.2
- net BUTTON_LED_CONN: now also R10.2; no longer J5-1.S
- net GND: now also J3.2, J4.2, J5.2, J7.2, U2.A3, U2.A4, U2.A5, U2.A6, U2.B3, U2.B4, U2.B5, U2.B6; no longer J2-2.S, J3-2.S, J4-2.S, J5-2.S
- net IN: now also J7.1; no longer J2-1.S
- net WIRELESS_LED_CONN: now also R9.2; no longer J4-1.S

Commit message: things should be done tm
Parts:
- C1, C7: device rcl:C-USC0603 -> rcl:C-USC0805
Changed lines of the file:
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@@
 <part name="U1" library="IGVC-Regulator" deviceset="R-78E5.0-1.0" device="CONV_R-78E5.0-1.0"/>
 <part name="P+5" library="supply1" library_urn="urn:adsk.eagle:library:371" deviceset="+5V" device=""/>
-<part name="C1" library="rcl" library_urn="urn:adsk.eagle:library:334" deviceset="C-US" device="C0603" package3d_urn="urn:adsk.eagle:package:23616/2" value="10uF"/>
-<part name="C7" library="rcl" library_urn="urn:adsk.eagle:library:334" deviceset="C-US" device="C0603" package3d_urn="urn:adsk.eagle:package:23616/2" value="10uF"/>
+<part name="C1" library="rcl" library_urn="urn:adsk.eagle:library:334" deviceset="C-US" device="C0805" package3d_urn="urn:adsk.eagle:package:23617/2" value="10uF"/>
+<part name="C7" library="rcl" library_urn="urn:adsk.eagle:library:334" deviceset="C-US" device="C0805" package3d_urn="urn:adsk.eagle:package:23617/2" value="10uF"/>
 <part name="GND10" library="supply1" library_urn="urn:adsk.eagle:library:371" deviceset="GND" device=""/>
 <part name="GND11" library="supply1" library_urn="urn:adsk.eagle:library:371" deviceset="GND" device=""/>

Commit message: Fixed estop-tx
Parts:
- removed PROG: ICSP Connector, lcd-buzzer:2X3SHROUDED
- removed R7: 10k, rcl:R-US_R0603
- removed S3: SKQGADE010, rgb-led:SMD-SWITCH-TOP-260GF(4P-D5.2MM)
- added C10, C9: 1uF, rcl:C-EUC0603
- added C11: 0.1uF, rcl:C-USC0603
- added ICSP: ICSP Connector, lcd-buzzer:2X3SHROUDED
- added RESET: SKQGADE010, rgb-led:SMD-SWITCH-TOP-260GF(4P-D5.2MM)
- added U3: MIC550X, IGVC-Regulator:MIC550X
Connections:
- net IN renamed BUTTON-IN
- net N$10 renamed EN
- removed net N$6: J1.RST, R7.1
- new net RADIO_RST: J1.RST, U4.PD2_(INT0/PCINT18)
- net !RESET: now also ICSP.5, RESET.A0; no longer PROG.5, S3.A0
- net +3V3: now also C10.1, U3.OUT
- net +5V: now also C11.1, C9.1, ICSP.2, U3.EN, U3.IN; no longer PROG.2
- net GND: now also C10.2, C11.2, C9.2, ICSP.6, RESET.B0, U3.GND; no longer PROG.6, R7.2, S3.B0
- net MISO: now also ICSP.1; no longer PROG.1
- net MOSI: now also ICSP.4; no longer PROG.4
- net SCK: now also ICSP.3; no longer PROG.3
Other:
- note removed: "Button Input"
- note removed: "Button LED"
- note removed: "LED Connectors"
- note removed: "Level Shifter (5V -> 3V3)"
- note removed: "Microcontroller"
- note removed: "Power"
- note removed: "Power LED"
- note removed: "Programming Connector"
- note removed: "Radio Board"
- note removed: "Reset Button"
- note removed: "Wireless LED"
- moved on the sheet: C1, C2, C3, C4, C5, C6, C7, C8, D1, D2, D3, D4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
